File: cartes/Carte_RF_CAN/nrf_can.sch (EAGLE design)
At the start: 18 parts, among them Q1 16MHz, U1 MCP2551

Commit message: divers
Parts:
- removed C5, C6: (no value), SparkFun-Capacitors:CAP_POLPTH2
- removed JP1: end_lign, SparkFun-Passives:JUMPER-2PTH
- removed JP2, JP3, JP4, JP5: (no value), pinhead:PINHD-1X3/90
- removed SK3: (no value), jt-con-micromatch:MMATCH-8-SMT
- removed U$2: MCP2515SO, MCP2515_MT:MCP2515SO
- removed U$3: ARDUINO_PRO_MINI'SERVO, can_bus_servo:ARDUINO_PRO_MINI'SERVO
- removed U1: MCP2551, SparkFun-DigitalIC:MCP2551
- added 3.3V_REGULATOR: LM3480IM4, SparkFun-PowerIC:LM3480IM4
- added ARDUINO_MINI: (no value), nrf_can:ARDUINO_PRO_MININRF24L01
- added CAN_CONTROL: MCP2515SO, MCP2515_MT:MCP2515SO
- added CAN_MICROMATCH: (no value), jt-con-micromatch:MMATCH-8-PTH
- added JUMPER_CAN: JUMPER-3PTH, SparkFun-Passives:JUMPER-3PTH
- added NRF24L01: M04X2, SparkFun-Connectors:M04X2
- added TRANSCEIVER: MCP2551, SparkFun-DigitalIC:MCP2551
- C3: value (none) -> 100nF; device SparkFun-Capacitors:CAP_POLPTH2 -> SparkFun-Capacitors:CAP0805
- C4: value (none) -> 1uF; device SparkFun-Capacitors:CAP_POLPTH2 -> SparkFun-Capacitors:CAP0805
Connections:
- removed net A4: JP5.1
- removed net A5: JP4.1
- removed net A6: JP3.1
- removed net A7: JP2.1
- removed net RXI: U$3.RXI
- removed net TXO: U$3.TXO
- new net 3.3V: 3.3V_REGULATOR.OUT, C4.1, NRF24L01.2
- new net NRF_CE: ARDUINO_MINI.5, NRF24L01.3
- new net NRF_CSN: ARDUINO_MINI.4, NRF24L01.4
- new net NRF_IRQ: ARDUINO_MINI.*3
- net CANH: now also CAN_MICROMATCH.4, CAN_MICROMATCH.5, JUMPER_CAN.3, TRANSCEIVER.CANH; no longer JP1.2, SK3.4, SK3.5, U1.CANH
- net CANL: now also CAN_MICROMATCH.3, CAN_MICROMATCH.6, TRANSCEIVER.CANL; no longer SK3.3, SK3.6, U1.CANL
- net CAN_CS: now also ARDUINO_MINI.*10, CAN_CONTROL.CS/; no longer U$2.CS/, U$3.*10
- net CAN_INT: now also ARDUINO_MINI.2, CAN_CONTROL.INT/; no longer U$2.INT/, U$3.2
- net CAN_RXD: now also CAN_CONTROL.RXCAN, TRANSCEIVER.RXD; no longer U$2.RXCAN, U1.RXD
- net CAN_TXD: now also CAN_CONTROL.TXCAN, TRANSCEIVER.TXD; no longer U$2.TXCAN, U1.TXD
- net GND: now also 3.3V_REGULATOR.GND, ARDUINO_MINI.GND, C3.2, C4.2, CAN_CONTROL.GND, CAN_MICROMATCH.1, CAN_MICROMATCH.8, NRF24L01.1, TRANSCEIVER.VDD; no longer C3.-, C4.-, C5.-, C6.-, JP2.2, JP3.2, JP4.2, JP5.2, SK3.1, SK3.8, U$2.GND, U$3.GND, U1.VDD
- net MISO: now also ARDUINO_MINI.12, CAN_CONTROL.SO, NRF24L01.7; no longer U$2.SO, U$3.12
- net MOSI: now also ARDUINO_MINI.*11, CAN_CONTROL.SI, NRF24L01.6; no longer U$2.SI, U$3.*11
- net N$2: now also CAN_CONTROL.OSC2; no longer U$2.OSC2
- net N$3: now also CAN_CONTROL.OSC1; no longer U$2.OSC1
- net N$5: now also TRANSCEIVER.RS; no longer U1.RS
- net N$7: now also JUMPER_CAN.2; no longer JP1.1
- net RST: now also ARDUINO_MINI.RST, CAN_CONTROL.RESET/; no longer U$2.RESET/, U$3.RST
- net SCK: now also ARDUINO_MINI.13, CAN_CONTROL.SCK, NRF24L01.5; no longer U$2.SCK, U$3.13
- net VCC: now also 3.3V_REGULATOR.IN, ARDUINO_MINI.VCC, C3.1, CAN_CONTROL.VCC, CAN_MICROMATCH.2, CAN_MICROMATCH.7, TRANSCEIVER.VSS; no longer C3.+, C4.+, C5.+, C6.+, JP2.3, JP3.3, JP4.3, JP5.3, SK3.2, SK3.7, U$2.VCC, U$3.VCC, U1.VSS
Other:
- note added: "BUS CAN"
- moved on the sheet: C1, C2, Q1, R1, R2

Commit message: Ajout dru et finit carte
Parts:
- removed 3.3V_REGULATOR: LM3480IM4, SparkFun-PowerIC:LM3480IM4
- removed C3: 100nF, SparkFun-Capacitors:CAP0805
- removed C4: 1uF, SparkFun-Capacitors:CAP0805
- added 3.3V: 3.3V/150mA, SparkFun-PowerIC:V_REG_MIC52053.3V
- added C5: 1uF, SparkFun-Capacitors:CAP0805
- CAN: value (none) -> micromatch8p
- renumbered CAN_MICROMATCH to CAN, JUMPER_CAN to _CAN
Connections:
- new net N$4: 3.3V.OUT, C5.1
- net 3.3V: no longer 3.3V_REGULATOR.OUT, C4.1
- net GND: now also 3.3V.GND, C5.2; no longer 3.3V_REGULATOR.GND, C3.2, C4.2
- net VCC: now also 3.3V.EN, 3.3V.IN; no longer 3.3V_REGULATOR.IN, C3.1
Changed lines of the file:
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@@
 <part name="ARDUINO_MINI" library="nrf_can" deviceset="ARDUINO_PRO_MINI" device="NRF24L01"/>
 <part name="NRF24L01" library="SparkFun-Connectors" deviceset="M04X2" device=""/>
-<part name="C3" library="SparkFun-Capacitors" deviceset="CAP" device="0805" value="100nF"/>
-<part name="C4" library="SparkFun-Capacitors" deviceset="CAP" device="0805" value="1uF"/>
-<part name="3.3V_REGULATOR" library="SparkFun-PowerIC" deviceset="LM3480IM4" device="" value=""/>
-<part name="JUMPER_CAN" library="SparkFun-Passives" deviceset="JUMPER-3" device="PTH"/>
-<part name="CAN_MICROMATCH" library="jt-con-micromatch" deviceset="MMATCH-8-*" device="PTH"/>
+<part name="_CAN" library="SparkFun-Passives" deviceset="JUMPER-3" device="PTH"/>
+<part name="CAN" library="jt-con-micromatch" deviceset="MMATCH-8-*" device="PTH" value="micromatch8p"/>
+<part name="3.3V" library="SparkFun-PowerIC" deviceset="V_REG_MIC5205" device="3.3V" value="3.3V/150mA"/>
+<part name="C5" library="SparkFun-Capacitors" deviceset="CAP" device="0805" value="1uF"/>
+<part name="SUPPLY1" library="supply2" deviceset="GND" device=""/>
+<part name="SUPPLY2" library="supply2" deviceset="GND" device=""/>
 </parts>
 <sheets>
@@
 <instance part="ARDUINO_MINI" gate="G$1" x="-15.24" y="137.16"/>
 <instance part="NRF24L01" gate="G$1" x="55.88" y="106.68"/>
-<instance part="C3" gate="G$1" x="53.34" y="144.78"/>
-<instance part="C4" gate="G$1" x="81.28" y="144.78"/>
-<instance part="3.3V_REGULATOR" gate="G$1" x="68.58" y="149.86"/>
-<instance part="JUMPER_CAN" gate="G$1" x="15.24" y="12.7" rot="R90"/>
-<instance part="CAN_MICROMATCH" gate="G$1" x="-20.32" y="-15.24"/>
+<instance part="_CAN" gate="G$1" x="15.24" y="12.7" rot="R90"/>
+<instance part="CAN" gate="G$1" x="-20.32" y="-15.24"/>
+<instance part="3.3V" gate="G$1" x="71.12" y="175.26"/>
+<instance part="C5" gate="G$1" x="88.9" y="175.26"/>
+<instance part="SUPPLY1" gate="GND" x="88.9" y="170.18"/>
+<instance part="SUPPLY2" gate="GND" x="53.34" y="172.72"/>
 </instances>
 <busses>
@@
 <wire x1="-25.4" y1="-7.62" x2="-30.48" y2="-7.62" width="0.1524" layer="91"/>
 <label x="-33.02" y="-7.62" size="1.778" layer="95"/>
-<pinref part="CAN_MICROMATCH" gate="G$1" pin="7"/>
+<pinref part="CAN" gate="G$1" pin="7"/>
 </segment>
 <segment>
 <wire x1="-15.24" y1="-15.24" x2="-10.16" y2="-15.24" width="0.1524" layer="91"/>
 <label x="-10.16" y="-15.24" size="1.778" layer="95"/>
-<pinref part="CAN_MICROMATCH" gate="G$1" pin="2"/>
+<pinref part="CAN" gate="G$1" pin="2"/>
 </segment>
 <segment>
@@
 </segment>
 <segment>
-<label x="50.8" y="149.86" size="1.778" layer="95"/>
-<pinref part="C3" gate="G$1" pin="1"/>
-<wire x1="55.88" y1="149.86" x2="53.34" y2="149.86" width="0.1524" layer="91"/>
-<wire x1="53.34" y1="149.86" x2="50.8" y2="149.86" width="0.1524" layer="91"/>
-<junction x="53.34" y="149.86"/>
-<pinref part="3.3V_REGULATOR" gate="G$1" pin="IN"/>
+<pinref part="3.3V" gate="G$1" pin="IN"/>
+<wire x1="60.96" y1="180.34" x2="58.42" y2="180.34" width="0.1524" layer="91"/>
+<pinref part="3.3V" gate="G$1" pin="EN"/>
+<wire x1="58.42" y1="180.34" x2="53.34" y2="180.34" width="0.1524" layer="91"/>
+<wire x1="60.96" y1="170.18" x2="45.72" y2="170.18" width="0.1524" layer="91"/>
+<wire x1="45.72" y1="170.18" x2="45.72" y2="177.8" width="0.1524" layer="91"/>
+<wire x1="45.72" y1="177.8" x2="58.42" y2="177.8" width="0.1524" layer="91"/>
+<wire x1="58.42" y1="177.8" x2="58.42" y2="180.34" width="0.1524" layer="91"/>
+<junction x="58.42" y="180.34"/>
+<label x="50.8" y="180.34" size="1.778" layer="95"/>
 </segment>
 </net>
@@
 <wire x1="-25.4" y1="-15.24" x2="-30.48" y2="-15.24" width="0.1524" layer="91"/>
 <label x="-33.02" y="-15.24" size="1.778" layer="95"/>
-<pinref part="CAN_MICROMATCH" gate="G$1" pin="1"/>
+<pinref part="CAN" gate="G$1" pin="1"/>
 </segment>
 <segment>
 <wire x1="-15.24" y1="-7.62" x2="-10.16" y2="-7.62" width="0.1524" layer="91"/>
 <label x="-10.16" y="-7.62" size="1.778" layer="95"/>
-<pinref part="CAN_MICROMATCH" gate="G$1" pin="8"/>
+<pinref part="CAN" gate="G$1" pin="8"/>
 </segment>
 <segment>
@@
 </segment>
 <segment>
-<label x="68.58" y="139.7" size="1.778" layer="95" rot="R180"/>
-<pinref part="C3" gate="G$1" pin="2"/>
-<wire x1="68.58" y1="139.7" x2="68.58" y2="142.24" width="0.1524" layer="91"/>
-<wire x1="53.34" y1="142.24" x2="68.58" y2="142.24" width="0.1524" layer="91"/>
-<pinref part="C4" gate="G$1" pin="2"/>
-<wire x1="81.28" y1="142.24" x2="68.58" y2="142.24" width="0.1524" layer="91"/>
-<junction x="68.58" y="142.24"/>
-<pinref part="3.3V_REGULATOR" gate="G$1" pin="GND"/>
-<junction x="68.58" y="139.7"/>
-<wire x1="68.58" y1="139.7" x2="68.58" y2="134.62" width="0.1524" layer="91"/>
+<pinref part="C5" gate="G$1" pin="2"/>
+<pinref part="SUPPLY1" gate="GND" pin="GND"/>
+</segment>
+<segment>
+<pinref part="3.3V" gate="G$1" pin="GND"/>
+<wire x1="60.96" y1="175.26" x2="53.34" y2="175.26" width="0.1524" layer="91"/>
+<pinref part="SUPPLY2" gate="GND" pin="GND"/>
 </segment>
 </net>
@@
 <wire x1="22.86" y1="17.78" x2="22.86" y2="20.32" width="0.1524" layer="91"/>
 <label x="22.86" y="20.32" size="1.778" layer="95" rot="R90"/>
-<pinref part="JUMPER_CAN" gate="G$1" pin="3"/>
+<pinref part="_CAN" gate="G$1" pin="3"/>
 <wire x1="22.86" y1="17.78" x2="17.78" y2="17.78" width="0.1524" layer="91"/>
 </segment>
@@
 <wire x1="-25.4" y1="-10.16" x2="-30.48" y2="-10.16" width="0.1524" layer="91"/>
 <label x="-33.02" y="-10.16" size="1.778" layer="95"/>
-<pinref part="CAN_MICROMATCH" gate="G$1" pin="5"/>
+<pinref part="CAN" gate="G$1" pin="5"/>
 </segment>
 <segment>
 <wire x1="-15.24" y1="-12.7" x2="-10.16" y2="-12.7" width="0.1524" layer="91"/>
 <label x="-10.16" y="-12.7" size="1.778" layer="95"/>
-<pinref part="CAN_MICROMATCH" gate="G$1" pin="4"/>
+<pinref part="CAN" gate="G$1" pin="4"/>
 </segment>
 </net>
@@
 <wire x1="-25.4" y1="-12.7" x2="-30.48" y2="-12.7" width="0.1524" layer="91"/>
 <label x="-33.02" y="-12.7" size="1.778" layer="95"/>
-<pinref part="CAN_MICROMATCH" gate="G$1" pin="3"/>
+<pinref part="CAN" gate="G$1" pin="3"/>
 </segment>
 <segment>
 <wire x1="-15.24" y1="-10.16" x2="-10.16" y2="-10.16" width="0.1524" layer="91"/>
 <label x="-10.16" y="-10.16" size="1.778" layer="95"/>
-<pinref part="CAN_MICROMATCH" gate="G$1" pin="6"/>
+<pinref part="CAN" gate="G$1" pin="6"/>
 </segment>
 </net>
@@
 <segment>
 <pinref part="R2" gate="G$1" pin="2"/>
-<pinref part="JUMPER_CAN" gate="G$1" pin="2"/>
-<pinref part="JUMPER_CAN" gate="G$1" pin="2"/>
+<pinref part="_CAN" gate="G$1" pin="2"/>
+<pinref part="_CAN" gate="G$1" pin="2"/>
 <junction x="17.78" y="15.24"/>
 <wire x1="17.78" y1="15.24" x2="22.86" y2="15.24" width="0.1524" layer="91"/>
@@
 <junction x="63.5" y="111.76"/>
 </segment>
-<segment>
-<label x="83.82" y="149.86" size="1.778" layer="95"/>
-<pinref part="C4" gate="G$1" pin="1"/>
-<wire x1="81.28" y1="149.86" x2="86.36" y2="149.86" width="0.1524" layer="91"/>
-<junction x="81.28" y="149.86"/>
-<pinref part="3.3V_REGULATOR" gate="G$1" pin="OUT"/>
-</segment>
 </net>
 <net name="NRF_IRQ" class="0">
@@
 </segment>
 </net>
+<net name="N$4" class="0">
+<segment>
+<pinref part="3.3V" gate="G$1" pin="OUT"/>
+<wire x1="78.74" y1="180.34" x2="88.9" y2="180.34" width="0.1524" layer="91"/>
+<pinref part="C5" gate="G$1" pin="1"/>
+</segment>
+</net>

Commit message: ajout erreurs
Connections:
- removed net N$4: 3.3V.OUT, C5.1
- net 3.3V: now also 3.3V.OUT, C5.1
- net NRF_IRQ: now also NRF24L01.8
Other:
- moved on the sheet: 3.3V, ARDUINO_MINI, C5
Changed lines of the file:
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@@
 <instance part="CAN_CONTROL" gate="G$1" x="78.74" y="27.94"/>
 <instance part="FRAME1" gate="G$1" x="-53.34" y="-68.58"/>
-<instance part="ARDUINO_MINI" gate="G$1" x="-15.24" y="137.16"/>
+<instance part="ARDUINO_MINI" gate="G$1" x="-5.08" y="93.98"/>
 <instance part="NRF24L01" gate="G$1" x="55.88" y="106.68"/>
 <instance part="_CAN" gate="G$1" x="15.24" y="12.7" rot="R90"/>
 <instance part="CAN" gate="G$1" x="-20.32" y="-15.24"/>
-<instance part="3.3V" gate="G$1" x="71.12" y="175.26"/>
-<instance part="C5" gate="G$1" x="88.9" y="175.26"/>
-<instance part="SUPPLY1" gate="GND" x="88.9" y="170.18"/>
-<instance part="SUPPLY2" gate="GND" x="53.34" y="172.72"/>
+<instance part="3.3V" gate="G$1" x="60.96" y="83.82"/>
+<instance part="C5" gate="G$1" x="78.74" y="83.82"/>
+<instance part="SUPPLY1" gate="GND" x="78.74" y="78.74"/>
+<instance part="SUPPLY2" gate="GND" x="43.18" y="81.28"/>
 </instances>
 <busses>
@@
 <segment>
 <pinref part="ARDUINO_MINI" gate="G$1" pin="*11"/>
-<wire x1="-2.54" y1="127" x2="7.62" y2="127" width="0.1524" layer="91"/>
-<label x="5.08" y="127" size="1.778" layer="95"/>
+<wire x1="7.62" y1="83.82" x2="17.78" y2="83.82" width="0.1524" layer="91"/>
+<label x="15.24" y="83.82" size="1.778" layer="95"/>
 </segment>
 <segment>
@@
 <segment>
 <pinref part="ARDUINO_MINI" gate="G$1" pin="12"/>
-<wire x1="-2.54" y1="129.54" x2="7.62" y2="129.54" width="0.1524" layer="91"/>
-<label x="5.08" y="129.54" size="1.778" layer="95"/>
+<wire x1="7.62" y1="86.36" x2="17.78" y2="86.36" width="0.1524" layer="91"/>
+<label x="15.24" y="86.36" size="1.778" layer="95"/>
 </segment>
 <segment>
@@
 <segment>
 <pinref part="ARDUINO_MINI" gate="G$1" pin="13"/>
-<wire x1="-2.54" y1="132.08" x2="7.62" y2="132.08" width="0.1524" layer="91"/>
-<label x="5.08" y="132.08" size="1.778" layer="95"/>
+<wire x1="7.62" y1="88.9" x2="17.78" y2="88.9" width="0.1524" layer="91"/>
+<label x="15.24" y="88.9" size="1.778" layer="95"/>
 </segment>
 <segment>
@@
 <segment>
 <pinref part="ARDUINO_MINI" gate="G$1" pin="VCC"/>
-<wire x1="-2.54" y1="144.78" x2="7.62" y2="144.78" width="0.1524" layer="91"/>
-<label x="5.08" y="144.78" size="1.778" layer="95"/>
+<wire x1="7.62" y1="101.6" x2="17.78" y2="101.6" width="0.1524" layer="91"/>
+<label x="15.24" y="101.6" size="1.778" layer="95"/>
 </segment>
 <segment>
 <pinref part="3.3V" gate="G$1" pin="IN"/>
-<wire x1="60.96" y1="180.34" x2="58.42" y2="180.34" width="0.1524" layer="91"/>
+<wire x1="50.8" y1="88.9" x2="48.26" y2="88.9" width="0.1524" layer="91"/>
 <pinref part="3.3V" gate="G$1" pin="EN"/>
-<wire x1="58.42" y1="180.34" x2="53.34" y2="180.34" width="0.1524" layer="91"/>
-<wire x1="60.96" y1="170.18" x2="45.72" y2="170.18" width="0.1524" layer="91"/>
-<wire x1="45.72" y1="170.18" x2="45.72" y2="177.8" width="0.1524" layer="91"/>
-<wire x1="45.72" y1="177.8" x2="58.42" y2="177.8" width="0.1524" layer="91"/>
-<wire x1="58.42" y1="177.8" x2="58.42" y2="180.34" width="0.1524" layer="91"/>
-<junction x="58.42" y="180.34"/>
-<label x="50.8" y="180.34" size="1.778" layer="95"/>
+<wire x1="48.26" y1="88.9" x2="43.18" y2="88.9" width="0.1524" layer="91"/>
+<wire x1="50.8" y1="78.74" x2="35.56" y2="78.74" width="0.1524" layer="91"/>
+<wire x1="35.56" y1="78.74" x2="35.56" y2="86.36" width="0.1524" layer="91"/>
+<wire x1="35.56" y1="86.36" x2="48.26" y2="86.36" width="0.1524" layer="91"/>
+<wire x1="48.26" y1="86.36" x2="48.26" y2="88.9" width="0.1524" layer="91"/>
+<junction x="48.26" y="88.9"/>
+<label x="40.64" y="88.9" size="1.778" layer="95"/>
 </segment>
 </net>
@@
 </segment>
 <segment>
-<wire x1="-22.86" y1="144.78" x2="-25.4" y2="144.78" width="0.1524" layer="91"/>
-<label x="-40.64" y="144.78" size="1.778" layer="95"/>
+<wire x1="-12.7" y1="101.6" x2="-15.24" y2="101.6" width="0.1524" layer="91"/>
+<label x="-30.48" y="101.6" size="1.778" layer="95"/>
 <pinref part="ARDUINO_MINI" gate="G$1" pin="GND"/>
-<wire x1="-25.4" y1="144.78" x2="-40.64" y2="144.78" width="0.1524" layer="91"/>
-<junction x="-25.4" y="144.78"/>
+<wire x1="-15.24" y1="101.6" x2="-30.48" y2="101.6" width="0.1524" layer="91"/>
+<junction x="-15.24" y="101.6"/>
 </segment>
 <segment>
@@
 <segment>
 <pinref part="3.3V" gate="G$1" pin="GND"/>
-<wire x1="60.96" y1="175.26" x2="53.34" y2="175.26" width="0.1524" layer="91"/>
+<wire x1="50.8" y1="83.82" x2="43.18" y2="83.82" width="0.1524" layer="91"/>
 <pinref part="SUPPLY2" gate="GND" pin="GND"/>
 </segment>
@@
 <segment>
 <pinref part="ARDUINO_MINI" gate="G$1" pin="RST"/>
-<wire x1="-25.4" y1="147.32" x2="-38.1" y2="147.32" width="0.1524" layer="91"/>
-<label x="-40.64" y="147.32" size="1.778" layer="95"/>
+<wire x1="-15.24" y1="104.14" x2="-27.94" y2="104.14" width="0.1524" layer="91"/>
+<label x="-30.48" y="104.14" size="1.778" layer="95"/>
 </segment>
 </net>
@@
 <segment>
 <pinref part="ARDUINO_MINI" gate="G$1" pin="*10"/>
-<wire x1="-2.54" y1="124.46" x2="7.62" y2="124.46" width="0.1524" layer="91"/>
-<label x="5.08" y="124.46" size="1.778" layer="95"/>
+<wire x1="7.62" y1="81.28" x2="17.78" y2="81.28" width="0.1524" layer="91"/>
+<label x="15.24" y="81.28" size="1.778" layer="95"/>
 </segment>
 </net>
@@
 <segment>
 <pinref part="ARDUINO_MINI" gate="G$1" pin="2"/>
-<wire x1="-25.4" y1="142.24" x2="-38.1" y2="142.24" width="0.1524" layer="91"/>
-<label x="-40.64" y="142.24" size="1.778" layer="95"/>
+<wire x1="-15.24" y1="99.06" x2="-27.94" y2="99.06" width="0.1524" layer="91"/>
+<label x="-30.48" y="99.06" size="1.778" layer="95"/>
 </segment>
 </net>
@@
 <segment>
 <pinref part="ARDUINO_MINI" gate="G$1" pin="4"/>
-<wire x1="-25.4" y1="137.16" x2="-38.1" y2="137.16" width="0.1524" layer="91"/>
-<label x="-40.64" y="137.16" size="1.778" layer="95"/>
+<wire x1="-15.24" y1="93.98" x2="-27.94" y2="93.98" width="0.1524" layer="91"/>
+<label x="-30.48" y="93.98" size="1.778" layer="95"/>
 </segment>
 <segment>
@@
 <segment>
 <pinref part="ARDUINO_MINI" gate="G$1" pin="5"/>
-<wire x1="-25.4" y1="134.62" x2="-27.94" y2="134.62" width="0.1524" layer="91"/>
-<wire x1="-27.94" y1="134.62" x2="-30.48" y2="134.62" width="0.1524" layer="91"/>
-<wire x1="-30.48" y1="134.62" x2="-38.1" y2="134.62" width="0.1524" layer="91"/>
-<label x="-40.64" y="134.62" size="1.778" layer="95"/>
+<wire x1="-15.24" y1="91.44" x2="-27.94" y2="91.44" width="0.1524" layer="91"/>
+<label x="-30.48" y="91.44" size="1.778" layer="95"/>
 </segment>
 </net>
@@
 <junction x="63.5" y="111.76"/>
 </segment>
+<segment>
+<pinref part="3.3V" gate="G$1" pin="OUT"/>
+<wire x1="68.58" y1="88.9" x2="78.74" y2="88.9" width="0.1524" layer="91"/>
+<pinref part="C5" gate="G$1" pin="1"/>
+<label x="73.66" y="88.9" size="1.778" layer="95"/>
+</segment>
 </net>
 <net name="NRF_IRQ" class="0">
 <segment>
-<wire x1="-22.86" y1="139.7" x2="-25.4" y2="139.7" width="0.1524" layer="91"/>
-<label x="-40.64" y="139.7" size="1.778" layer="95"/>
+<wire x1="-12.7" y1="96.52" x2="-15.24" y2="96.52" width="0.1524" layer="91"/>
+<label x="-30.48" y="96.52" size="1.778" layer="95"/>
 <pinref part="ARDUINO_MINI" gate="G$1" pin="*3"/>
-<wire x1="-25.4" y1="139.7" x2="-38.1" y2="139.7" width="0.1524" layer="91"/>
-<junction x="-25.4" y="139.7"/>
-</segment>
-</net>
-<net name="N$4" class="0">
-<segment>
-<pinref part="3.3V" gate="G$1" pin="OUT"/>
-<wire x1="78.74" y1="180.34" x2="88.9" y2="180.34" width="0.1524" layer="91"/>
-<pinref part="C5" gate="G$1" pin="1"/>
-</segment>
-</net>
+<wire x1="-15.24" y1="96.52" x2="-27.94" y2="96.52" width="0.1524" layer="91"/>
+<junction x="-15.24" y="96.52"/>
+</segment>
+<segment>
+<wire x1="60.96" y1="104.14" x2="63.5" y2="104.14" width="0.1524" layer="91"/>
+<label x="68.58" y="104.14" size="1.778" layer="95"/>
+<pinref part="NRF24L01" gate="G$1" pin="8"/>
+<junction x="63.5" y="104.14"/>
+<wire x1="63.5" y1="104.14" x2="71.12" y2="104.14" width="0.1524" layer="91"/>
+</segment>
+</net>
