File: cartes/Carte_RF_CAN/nrf_can.brd (EAGLE design)
At the start: 44.1 x 37.5 mm, 10 parts, among them Q1 16MHz, U1 MCP2551

Commit message: divers
Parts:
- removed JP1: end_lign, SparkFun-Passives:1X02
- removed SK3: (no value), jt-con-micromatch:AMP-188275-8
- removed U$2: MCP2515SO, MCP2515_MT:SO18L
- removed U$3: ARDUINO_PRO_MINI'SERVO, can_bus_servo:ARDUINO_PRO_MINI
- removed U1: MCP2551, SparkFun-DigitalIC:SO08
- added 3.3V_REGULATOR: (no value), SparkFun-PowerIC:SOT23-3
- added ARDUINO_MINI: (no value), nrf_can:ARDUINO_PRO_MINI
- added C3: 100nF, SparkFun-Capacitors:0805
- added C4: 1uF, SparkFun-Capacitors:0805
- added CAN_CONTROL: MCP2515SO, MCP2515_MT:SO18L
- added CAN_MICROMATCH: (no value), jt-con-micromatch:AMP-215079-8
- added JUMPER_CAN: JUMPER-3PTH, SparkFun-Passives:1X03
- added NRF24L01: M04X2, SparkFun-Connectors:2X4
- added TRANSCEIVER: MCP2551, SparkFun-DigitalIC:SO08
- moved Q1 36.2 mm to (34.3, 43.2)
- moved C1 32.0 mm to (30.5, 47.0)
- moved R2 31.2 mm to (31.7, 19.1), flipped to the bottom, turned to 180 degrees
- moved C2 31.0 mm to (30.5, 40.6)
- moved R1 12.4 mm to (16.2, 18.1), flipped to the bottom, turned to 90 degrees
Connections:
- removed net RXI: U$3.RXI
- removed net TXO: U$3.TXO
- new net 3.3V: 3.3V_REGULATOR.1, C4.1, NRF24L01.2
- new net NRF_CE: ARDUINO_MINI.8, NRF24L01.3
- new net NRF_CSN: ARDUINO_MINI.7, NRF24L01.4
- new net NRF_IRQ: ARDUINO_MINI.6
- net CANH: now also CAN_MICROMATCH.4, CAN_MICROMATCH.5, JUMPER_CAN.3, TRANSCEIVER.7; no longer JP1.2, SK3.4, SK3.5, U1.7
- net CANL: now also CAN_MICROMATCH.3, CAN_MICROMATCH.6, TRANSCEIVER.6; no longer SK3.3, SK3.6, U1.6
- net CAN_CS: now also ARDUINO_MINI.13, CAN_CONTROL.16; no longer U$2.16, U$3.13
- net CAN_INT: now also ARDUINO_MINI.5, CAN_CONTROL.12; no longer U$2.12, U$3.5
- net CAN_RXD: now also CAN_CONTROL.2, TRANSCEIVER.4; no longer U$2.2, U1.4
- net CAN_TXD: now also CAN_CONTROL.1, TRANSCEIVER.1; no longer U$2.1, U1.1
- net GND: now also 3.3V_REGULATOR.3, ARDUINO_MINI.GND, C3.2, C4.2, CAN_CONTROL.9, CAN_MICROMATCH.1, CAN_MICROMATCH.8, NRF24L01.1, TRANSCEIVER.3; no longer SK3.1, SK3.8, U$2.9, U$3.GND, U1.3
- net MISO: now also ARDUINO_MINI.15, CAN_CONTROL.15, NRF24L01.7; no longer U$2.15, U$3.15
- net MOSI: now also ARDUINO_MINI.14, CAN_CONTROL.14, NRF24L01.6; no longer U$2.14, U$3.14
- net N$2: now also CAN_CONTROL.7; no longer U$2.7
- net N$3: now also CAN_CONTROL.8; no longer U$2.8
- net N$5: now also TRANSCEIVER.8; no longer U1.8
- net N$7: now also JUMPER_CAN.2; no longer JP1.1
- net RST: now also ARDUINO_MINI.3, CAN_CONTROL.17; no longer U$2.17, U$3.3
- net SCK: now also ARDUINO_MINI.16, CAN_CONTROL.13, NRF24L01.5; no longer U$2.13, U$3.16
- net VCC: now also 3.3V_REGULATOR.2, ARDUINO_MINI.VCC, C3.1, CAN_CONTROL.18, CAN_MICROMATCH.2, CAN_MICROMATCH.7, TRANSCEIVER.2; no longer SK3.2, SK3.7, U$2.18, U$3.VCC, U1.2
Routing:
- net VCC: track 54.6 -> 0.00 mm, vias 2 -> 0
- net CANH: track 46.0 -> 0.00 mm, vias 3 -> 0
- net CANL: track 42.6 -> 0.00 mm
- net SCK: track 25.6 -> 0.00 mm, vias 2 -> 0
- net RST: track 22.2 -> 0.00 mm
- net CAN_INT: track 19.7 -> 0.00 mm
- net CAN_RXD: track 13.9 -> 0.00 mm
- net CAN_CS: track 11.1 -> 0.00 mm
- net MISO: track 10.1 -> 0.00 mm, vias 1 -> 0
- net MOSI: track 9.26 -> 0.00 mm, vias 1 -> 0
- net N$2: track 8.73 -> 0.00 mm
- net GND: track 8.18 -> 0.00 mm, vias 2 -> 0
- net N$3: track 6.73 -> 0.00 mm
- net CAN_TXD: track 4.65 -> 0.00 mm
- net N$5: track 3.47 -> 0.00 mm
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- removed copper zone on layer 1, net GND
Other:
- board size 44.1 x 37.5 mm -> 32.7 x 41.9 mm
- board text removed: "sharp 2014"

Commit message: finit rf
Parts:
- moved JUMPER_CAN 3.69 mm to (35.9, 19.6)
- moved CAN_CONTROL 2.08 mm to (23.9, 19.5)
- moved C1 2.00 mm to (31.0, 45.1), turned to 90 degrees
- moved CAN_MICROMATCH 1.17 mm to (35.1, 34.8)
- moved C2 0.92 mm to (31.0, 41.4), turned to 270 degrees
Routing:
- net VCC: track 0.00 -> 64.5 mm, vias 0 -> 2
- net N$2: track 0.00 -> 33.6 mm
- net CANH: track 0.00 -> 31.5 mm
- net RST: track 0.00 -> 29.3 mm, vias 0 -> 1
- net CANL: track 0.00 -> 24.1 mm
- net N$3: track 0.00 -> 23.0 mm
- net MOSI: track 0.00 -> 22.7 mm, vias 0 -> 1
- net NRF_CE: track 0.00 -> 21.2 mm
- net MISO: track 0.00 -> 21.0 mm
- net SCK: track 0.00 -> 18.8 mm, vias 0 -> 1
- net CAN_INT: track 0.00 -> 17.6 mm, vias 0 -> 1
- net N$5: track 0.00 -> 14.4 mm
- net NRF_CSN: track 0.00 -> 14.0 mm
- net CAN_RXD: track 0.00 -> 13.4 mm, vias 0 -> 1
- net 3.3V: track 0.00 -> 10.2 mm
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- added copper zone on layer 1, net GND
Other:
- board size 32.7 x 41.9 mm -> 33.4 x 41.8 mm

Commit message: Ajout dru et finit carte
Parts:
- removed 3.3V_REGULATOR: (no value), SparkFun-PowerIC:SOT23-3
- removed C3: 100nF, SparkFun-Capacitors:0805
- removed C4: 1uF, SparkFun-Capacitors:0805
- added 3.3V: 3.3V/150mA, SparkFun-PowerIC:SOT23-5
- added C5: 1uF, SparkFun-Capacitors:0805
- CAN: value (none) -> micromatch8p
- renumbered CAN_MICROMATCH to CAN, JUMPER_CAN to _CAN
Connections:
- new net N$4: 3.3V.5, C5.1
- net 3.3V: no longer 3.3V_REGULATOR.1, C4.1
- net GND: now also 3.3V.2, C5.2; no longer 3.3V_REGULATOR.3, C3.2, C4.2
- net VCC: now also 3.3V.1, 3.3V.3; no longer 3.3V_REGULATOR.2, C3.1
Routing:
- net 3.3V: track 10.2 -> 0.00 mm
- net N$4: track 0.00 -> 1.72 mm
- net VCC: track 64.5 -> 66.2 mm
- net MOSI: track 22.7 -> 23.6 mm
- net N$2: track 33.6 -> 32.9 mm
- net CAN_INT: track 17.6 -> 18.2 mm
- net RST: track 29.3 -> 29.9 mm, vias 1 -> 0
Other:
- board size 33.4 x 41.8 mm -> 33.3 x 41.8 mm

Commit message: ajout erreurs
Parts:
- moved C5 0.72 mm to (21.3, 43.3)
Connections:
- removed net N$4: 3.3V.5, C5.1
- net 3.3V: now also 3.3V.5, C5.1
- net NRF_IRQ: now also NRF24L01.8
Routing:
- net NRF_IRQ: track 0.00 -> 21.6 mm
- net 3.3V: track 0.00 -> 9.70 mm
- net N$4: track 1.72 -> 0.00 mm, vias 0 -> 1
Other:
- board size 33.3 x 41.8 mm -> 34.2 x 39.4 mm
Changed lines of the file:
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@@
 <setting verticaltext="up"/>
 </settings>
-<grid distance="0.001" unitdist="inch" unit="inch" style="lines" multiple="1" display="no" altdistance="0.001" altunitdist="inch" altunit="inch"/>
+<grid distance="0.01" unitdist="inch" unit="inch" style="lines" multiple="1" display="no" altdistance="0.001" altunitdist="inch" altunit="inch"/>
 <layers>
 <layer number="1" name="Top" color="4" fill="1" visible="yes" active="yes"/>
@@
 <layer number="43" name="vRestrict" color="2" fill="10" visible="yes" active="yes"/>
 <layer number="44" name="Drills" color="7" fill="1" visible="no" active="yes"/>
-<layer number="45" name="Holes" color="7" fill="1" visible="no" active="yes"/>
+<layer number="45" name="Holes" color="7" fill="1" visible="yes" active="yes"/>
 <layer number="46" name="Milling" color="3" fill="1" visible="no" active="yes"/>
 <layer number="47" name="Measures" color="7" fill="1" visible="no" active="yes"/>
@@
 <board>
 <plain>
-<wire x1="7.6454" y1="10.2616" x2="40.945" y2="10.5156" width="0" layer="20"/>
-<wire x1="40.945" y1="10.5156" x2="40.31" y2="52.06" width="0" layer="20"/>
-<wire x1="40.31" y1="52.06" x2="7.62" y2="52.06" width="0" layer="20"/>
-<wire x1="7.62" y1="52.06" x2="7.6454" y2="10.2616" width="0" layer="20"/>
+<wire x1="7.3914" y1="11.6332" x2="41.453" y2="11.7094" width="0" layer="20"/>
+<wire x1="41.453" y1="11.7094" x2="41.58" y2="51.044" width="0" layer="20"/>
+<wire x1="41.58" y1="51.044" x2="7.62" y2="50.6884" width="0" layer="20"/>
+<wire x1="7.62" y1="50.6884" x2="7.3914" y2="11.6332" width="0" layer="20"/>
 <polygon width="0.3048" layer="43">
 <vertex x="20.4978" y="21.209"/>
@@
 <attribute name="PROD_ID" value="VREG-00822" x="23.368" y="40.0812" size="1.778" layer="27" display="off"/>
 </element>
-<element name="C5" library="SparkFun-Capacitors" package="0805" value="1uF" x="20.8026" y="42.799" rot="R180"/>
+<element name="C5" library="SparkFun-Capacitors" package="0805" value="1uF" x="21.3106" y="43.307" rot="R180"/>
 </elements>
 <signals>
@@
 <signal name="3.3V">
 <contactref element="NRF24L01" pad="2"/>
+<contactref element="3.3V" pad="5"/>
+<contactref element="C5" pad="1"/>
+<wire x1="22.4028" y1="43.0276" x2="22.4028" y2="41.4274" width="0.15" layer="1"/>
+<wire x1="22.225" y1="43.2054" x2="22.4028" y2="43.0276" width="0.15" layer="1"/>
+<wire x1="22.225" y1="43.2054" x2="22.2106" y2="43.307" width="0.15" layer="1"/>
+<wire x1="17.0688" y1="41.4274" x2="22.4028" y2="41.4274" width="0.15" layer="1"/>
+<wire x1="17.0688" y1="39.116" x2="17.0688" y2="41.4274" width="0.15" layer="1"/>
+<wire x1="22.4028" y1="41.4274" x2="22.418" y2="41.3813" width="0.15" layer="1"/>
+<wire x1="17.0688" y1="39.116" x2="17.018" y2="39.0906" width="0.15" layer="1"/>
 </signal>
 <signal name="NRF_IRQ">
 <contactref element="ARDUINO_MINI" pad="6"/>
+<contactref element="NRF24L01" pad="8"/>
+<wire x1="22.9362" y1="25.6032" x2="17.0688" y2="31.4706" width="0.15" layer="16"/>
+<wire x1="28.2702" y1="25.6032" x2="22.9362" y2="25.6032" width="0.15" layer="16"/>
+<wire x1="29.337" y1="26.67" x2="28.2702" y2="25.6032" width="0.15" layer="16"/>
+<wire x1="29.337" y1="31.6484" x2="29.337" y2="26.67" width="0.15" layer="16"/>
+<wire x1="28.0924" y1="31.6484" x2="29.337" y2="31.6484" width="0.15" layer="16"/>
+<wire x1="17.0688" y1="31.4706" x2="17.018" y2="31.4706" width="0.15" layer="16"/>
+<wire x1="28.0924" y1="31.6484" x2="27.94" y2="31.75" width="0.15" layer="16"/>
+</signal>
+<signal name="N$1">
+<via x="9.652" y="48.768" extent="1-16" drill="2.1"/>
 </signal>
 <signal name="N$4">
-<contactref element="3.3V" pad="5"/>
-<contactref element="C5" pad="1"/>
-<wire x1="22.0472" y1="42.4942" x2="21.8694" y2="42.672" width="0.15" layer="1"/>
-<wire x1="22.0472" y1="42.1386" x2="22.0472" y2="42.4942" width="0.15" layer="1"/>
-<wire x1="22.4028" y1="41.783" x2="22.0472" y2="42.1386" width="0.15" layer="1"/>
-<wire x1="22.4028" y1="41.4274" x2="22.4028" y2="41.783" width="0.15" layer="1"/>
-<wire x1="21.8694" y1="42.672" x2="21.7026" y2="42.799" width="0.15" layer="1"/>
-<wire x1="22.4028" y1="41.4274" x2="22.418" y2="41.3813" width="0.15" layer="1"/>
+<via x="9.906" y="13.97" extent="1-16" drill="2.1"/>
+</signal>
+<signal name="N$6">
+<via x="39.37" y="13.97" extent="1-16" drill="2.1"/>
+</signal>
+<signal name="N$8">
+<via x="39.37" y="49.022" extent="1-16" drill="2.1"/>
 </signal>
 </signals>

Commit message: a
Other:
- board size 34.2 x 39.4 mm -> 34 x 39.4 mm
- board text added: "/home/showok/.eagle/logo_ares_3.bmp"
- board text added: "RF-CAN ARES 2014"
- board text added: "aaa"

Commit message: Ajout carte RF avec bon fichier
Routing:
- net NRF_IRQ: track 21.6 -> 11.1 mm
- net NRF_CE: track 21.2 -> 24.9 mm
- net VCC: track 66.2 -> 67.2 mm
- net CAN_INT: track 18.2 -> 19.0 mm
- net MOSI: track 23.6 -> 24.2 mm
- net NRF_CSN: vias 0 -> 1
Other:
- board text added: "& Dipole"
- board text added: "ARES 2014"
- board text added: "Carte Nrf24l01-CAN"

Commit message: plein de trucs
Other:
- board text added: "/home/showok/Documents/Projets/Ares/Robot-2013-2014/cartes/logo_ares_3.bmp"
