File: cartes/sharp_shield/mini_board0.sch (EAGLE design)
At the start: 18 parts, among them Q1 16MHz, U1 MCP2551

Commit message: divers
Parts:
- U$1: value ARDUINO_PRO_MINISHARP_CAPE -> arduino_mini
Other:
- note added: "BUS CAN"
- note added: "SHARP"
- moved on the sheet: C1, C2, C3, C4, C5, C6, JP1, JP2, JP3, JP4, JP5, Q1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

Commit message: a
Parts:
- removed JP1: end_lign, SparkFun-Passives:JUMPER-2PTH
- removed SK3: (no value), jt-con-micromatch:MMATCH-8-SMT
- removed U$1: arduino_mini, custom_can_bus:ARDUINO_PRO_MINISHARP_CAPE
- added C7, C8: (no value), SparkFun-Capacitors:CAP_POLPTH2
- added JP6, JP7: (no value), pinhead:PINHD-1X3/90
- added JP8: JUMPER-3PTH, SparkFun-Passives:JUMPER-3PTH
- added SK1: (no value), jt-con-micromatch:MMATCH-8-PTH
- added U$3: ARDUINO_PRO_MINI, sharp_shield:ARDUINO_PRO_MINI
Connections:
- removed net A6: JP3.1, U$1.A6
- removed net A7: JP2.1, U$1.A7
- new net A0: JP2.1, U$3.A0
- new net A1: JP3.1, U$3.A1
- new net A2: JP6.1, U$3.A2
- new net A3: JP5.1, U$3.A3
- net A4: now also JP4.1, U$3.A4; no longer JP5.1, U$1.A4
- net A5: now also JP7.1, U$3.A5; no longer JP4.1, U$1.A5
- net CANH: now also JP8.3, SK1.4, SK1.5; no longer JP1.2, SK3.4, SK3.5
- net CANL: now also SK1.3, SK1.6; no longer SK3.3, SK3.6
- net CAN_CS: now also U$3.*10; no longer U$1.*10
- net CAN_INT: now also U$3.2; no longer U$1.2
- net GND: now also C7.-, C8.-, JP6.2, JP7.2, SK1.1, SK1.8, U$3.GND; no longer SK3.1, SK3.8, U$1.GND@2
- net MISO: now also U$3.12; no longer U$1.12
- net MOSI: now also U$3.*11; no longer U$1.*11
- net N$7: now also JP8.2; no longer JP1.1
- net RST: now also U$3.RST; no longer U$1.RST@2
- net SCK: now also U$3.13; no longer U$1.13
- net VCC: now also C7.+, C8.+, JP6.3, JP7.3, SK1.2, SK1.7, U$3.VCC; no longer SK3.2, SK3.7, U$1.RAW
Other:
- moved on the sheet: R2

Commit message: Ajout carte sharp v2
Parts:
- renumbered JP2 to A0, JP3 to A1, JP4 to A4, JP5 to A3, JP6 to A2, JP7 to A5, JP8 to CAN_S, Q1 to 16MHZ, SK1 to CAN, U$2 to CONTROLLER, U$3 to ARDUINO
