File: cartes/sharp_shield/mini_board0.brd (EAGLE design)
At the start: 44.9 x 37.5 mm, 22 parts, among them U1 MCP2551

Commit message: sharp
Parts:
- moved A0 2.80 mm to (44.4, 20.9)
- moved A3 2.01 mm to (44.2, 45.0)
- moved C1 1.69 mm to (28.6, 44.0), turned to 90 degrees
- moved A1 1.52 mm to (44.4, 28.8)
- moved C8 1.12 mm to (11.0, 46.6)
- moved C4 0.51 mm to (10.5, 39.5), turned to 270 degrees
Routing:
- net VCC: track 139.2 -> 147.5 mm, vias 1 -> 2
- net A5: track 15.6 -> 21.7 mm, vias 1 -> 0
- net A3: track 31.2 -> 30.1 mm
- net N$5: track 21.7 -> 22.1 mm, vias 0 -> 2
