File: cartes/sharp_shield/mini_board0.brd (EAGLE design)
At the start: 44.1 x 37.5 mm, 18 parts, among them Q1 16MHz, U1 MCP2551

Commit message: divers
Parts:
- U$1: value ARDUINO_PRO_MINISHARP_CAPE -> arduino_mini
Changed lines of the file:
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@@
 <element name="JP1" library="SparkFun-Passives" package="1X02" value="end_lign" x="3.81" y="27.94"/>
 <element name="SK3" library="jt-con-micromatch" package="AMP-188275-8" value="" x="9.525" y="38.735" rot="R90"/>
-<element name="U$1" library="custom_can_bus" package="ARDUINO_PRO_MINI" value="ARDUINO_PRO_MINISHARP_CAPE" x="22.86" y="33.655"/>
+<element name="U$1" library="custom_can_bus" package="ARDUINO_PRO_MINI" value="arduino_mini" x="22.86" y="33.655"/>
 <element name="U$2" library="MCP2515_MT" package="SO18L" value="MCP2515SO" x="17.145" y="22.225" rot="R270"/>
 <element name="JP5" library="pinhead" package="1X03/90" value="" x="43.815" y="45.72" rot="R270"/>

Commit message: a
Parts:
- removed JP1: end_lign, SparkFun-Passives:1X02
- removed SK3: (no value), jt-con-micromatch:AMP-188275-8
- removed U$1: arduino_mini, custom_can_bus:ARDUINO_PRO_MINI
- added C7, C8: (no value), SparkFun-Capacitors:CPOL-RADIAL-10UF-25V
- added JP6, JP7: (no value), pinhead:1X03/90
- added JP8: JUMPER-3PTH, SparkFun-Passives:1X03
- added SK1: (no value), jt-con-micromatch:AMP-215079-8
- added U$3: ARDUINO_PRO_MINI, sharp_shield:ARDUINO_PRO_MINI
Connections:
- removed net A6: JP3.1, U$1.A6
- removed net A7: JP2.1, U$1.A7
- new net A0: JP2.1, U$3.17
- new net A1: JP3.1, U$3.18
- new net A2: JP6.1, U$3.19
- new net A3: JP5.1, U$3.20
- net A4: now also JP4.1, U$3.A4; no longer JP5.1, U$1.A4
- net A5: now also JP7.1, U$3.A5; no longer JP4.1, U$1.A5
- net CANH: now also JP8.3, SK1.4, SK1.5; no longer JP1.2, SK3.4, SK3.5
- net CANL: now also SK1.3, SK1.6; no longer SK3.3, SK3.6
- net CAN_CS: now also U$3.13; no longer U$1.13
- net CAN_INT: now also U$3.5; no longer U$1.5
- net GND: now also C7.2, C8.2, JP6.2, JP7.2, SK1.1, SK1.8, U$3.GND; no longer SK3.1, SK3.8, U$1.23
- net MISO: now also U$3.15; no longer U$1.15
- net MOSI: now also U$3.14; no longer U$1.14
- net N$7: now also JP8.2; no longer JP1.1
- net RST: now also U$3.3; no longer U$1.22
- net SCK: now also U$3.16; no longer U$1.16
- net VCC: now also C7.1, C8.1, JP6.3, JP7.3, SK1.2, SK1.7, U$3.VCC; no longer SK3.2, SK3.7, U$1.24
Routing:
- net VCC: track 113.2 -> 0.00 mm, vias 2 -> 0
- net CANH: track 46.0 -> 0.00 mm, vias 3 -> 0
- net CANL: track 42.6 -> 0.00 mm
- net SCK: track 25.8 -> 0.00 mm, vias 2 -> 0
- net A4: track 25.6 -> 0.00 mm
- net RST: track 22.3 -> 0.00 mm
- net A6: track 20.5 -> 0.00 mm
- net CAN_INT: track 19.8 -> 0.00 mm
- net A7: track 15.4 -> 0.00 mm, vias 1 -> 0
- net A5: track 15.0 -> 0.00 mm
- net CAN_RXD: track 13.9 -> 0.00 mm
- net CAN_CS: track 11.5 -> 0.00 mm
- net MISO: track 10.3 -> 0.00 mm, vias 1 -> 0
- net MOSI: track 9.38 -> 0.00 mm, vias 1 -> 0
- net N$2: track 8.73 -> 0.00 mm
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
Commit message: Ajout carte sharp v2
Parts:
- removed JP2, JP3, JP4, JP5, JP6, JP7: (no value), pinhead:1X03/90
- removed JP8: JUMPER-3PTH, SparkFun-Passives:1X03
- removed Q1: 16MHz, adafruit:HC49/S
- removed SK1: (no value), jt-con-micromatch:AMP-215079-8
- removed U$2: MCP2515SO, MCP2515_MT:SO18L
- removed U$3: ARDUINO_PRO_MINI, sharp_shield:ARDUINO_PRO_MINI
- added 16MHZ: 16MHz, adafruit:HC49/S
- added A0, A1, A2, A3, A4, A5: (no value), pinhead:1X03/90
- added ARDUINO: ARDUINO_PRO_MINI, sharp_shield:ARDUINO_PRO_MINI
- added CAN: (no value), jt-con-micromatch:AMP-215079-8
- added CAN_S: JUMPER-3PTH, SparkFun-Passives:1X03
- added CONTROLLER: MCP2515SO, MCP2515_MT:SO18L
- moved C8 69.8 mm to (10.2, 48.3), turned to 90 degrees
- moved C7 56.7 mm to (36.2, 35.7), turned to 270 degrees
- moved C1 29.8 mm to (28.6, 45.7)
- moved C2 29.3 mm to (28.6, 40.0), turned to 270 degrees
- moved C4 25.9 mm to (9.72, 39.1), turned to 90 degrees
- moved U1 15.5 mm to (17.8, 45.1), turned to 270 degrees
- moved R2 12.5 mm to (12.6, 23.6), turned to 90 degrees
- moved R1 3.18 mm to (6.99, 30.5), turned to 270 degrees
- moved C6 2.34 mm to (36.2, 17.7)
- moved C5 1.42 mm to (36.2, 26.7)
- moved C3 0.63 mm to (36.2, 45.1)
Connections:
- net A0: now also A0.1, ARDUINO.17; no longer JP2.1, U$3.17
- net A1: now also A1.1, ARDUINO.18; no longer JP3.1, U$3.18
- net A2: now also A2.1, ARDUINO.19; no longer JP6.1, U$3.19
- net A3: now also A3.1, ARDUINO.20; no longer JP5.1, U$3.20
- net A4: now also A4.1, ARDUINO.A4; no longer JP4.1, U$3.A4
- net A5: now also A5.1, ARDUINO.A5; no longer JP7.1, U$3.A5
- net CANH: now also CAN.4, CAN.5, CAN_S.3; no longer JP8.3, SK1.4, SK1.5
- net CANL: now also CAN.3, CAN.6; no longer SK1.3, SK1.6
- net CAN_CS: now also ARDUINO.13, CONTROLLER.16; no longer U$2.16, U$3.13
- net CAN_INT: now also ARDUINO.5, CONTROLLER.12; no longer U$2.12, U$3.5
- net CAN_RXD: now also CONTROLLER.2; no longer U$2.2
- net CAN_TXD: now also CONTROLLER.1; no longer U$2.1
- net GND: now also A0.2, A1.2, A2.2, A3.2, A4.2, A5.2, ARDUINO.GND, CAN.1, CAN.8, CONTROLLER.9; no longer JP2.2, JP3.2, JP4.2, JP5.2, JP6.2, JP7.2, SK1.1, SK1.8, U$2.9, U$3.GND
- net MISO: now also ARDUINO.15, CONTROLLER.15; no longer U$2.15, U$3.15
- net MOSI: now also ARDUINO.14, CONTROLLER.14; no longer U$2.14, U$3.14
- net N$2: now also 16MHZ.2, CONTROLLER.7; no longer Q1.2, U$2.7
- net N$3: now also 16MHZ.1, CONTROLLER.8; no longer Q1.1, U$2.8
- net N$7: now also CAN_S.2; no longer JP8.2
- net RST: now also ARDUINO.3, CONTROLLER.17; no longer U$2.17, U$3.3
- net SCK: now also ARDUINO.16, CONTROLLER.13; no longer U$2.13, U$3.16
- net VCC: now also A0.3, A1.3, A2.3, A3.3, A4.3, A5.3, ARDUINO.VCC, CAN.2, CAN.7, CONTROLLER.18; no longer JP2.3, JP3.3, JP4.3, JP5.3, JP6.3, JP7.3, SK1.2, SK1.7, U$2.18, U$3.VCC
Routing:
- net VCC: track 0.00 -> 139.3 mm, vias 0 -> 1
- net CANL: track 0.00 -> 41.8 mm
- net CANH: track 0.00 -> 33.2 mm
- net A3: track 0.00 -> 31.2 mm, vias 0 -> 1
- net N$2: track 0.00 -> 30.0 mm
- net CAN_CS: track 0.00 -> 29.4 mm
- net A0: track 0.00 -> 28.9 mm
- net N$3: track 0.00 -> 28.7 mm
- net A2: track 0.00 -> 28.1 mm
- net CAN_TXD: track 0.00 -> 27.0 mm
- net A1: track 0.00 -> 25.7 mm
- net N$5: track 0.00 -> 21.7 mm
- net CAN_RXD: track 0.00 -> 21.2 mm, vias 0 -> 2
- net SCK: track 0.00 -> 20.0 mm, vias 0 -> 1
- net CAN_INT: track 0.00 -> 18.7 mm
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Other:
- board size 44.1 x 37.5 mm -> 43.5 x 37.4 mm
- board text added: "Ares Dipole 2014"
- board text added: "Carte Sharp-CAN"
- board text removed: "sharp 2014"

Commit message: end sharp
Parts:
- moved C4 1.42 mm to (11.0, 39.7)
- moved C8 1.08 mm to (11.1, 47.8)
Routing:
- net VCC: track 139.3 -> 153.2 mm
Other:
- board size 43.5 x 37.4 mm -> 44.9 x 37.3 mm

Commit message: ajout nvlle carte puissance
Other:
- board size 44.9 x 37.3 mm -> 44.9 x 37.5 mm
Changed lines of the file:
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@@
 <board>
 <plain>
-<wire x1="0.762" y1="14.0335" x2="45.39" y2="13.97" width="0" layer="20"/>
-<wire x1="45.39" y1="13.97" x2="45.644" y2="51.171" width="0" layer="20"/>
+<wire x1="0.762" y1="13.9065" x2="45.39" y2="13.843" width="0" layer="20"/>
+<wire x1="45.39" y1="13.843" x2="45.644" y2="51.171" width="0" layer="20"/>
 <wire x1="45.644" y1="51.171" x2="0.8255" y2="51.298" width="0" layer="20"/>
-<wire x1="0.8255" y1="51.298" x2="0.762" y2="14.0335" width="0" layer="20"/>
-<text x="3.7465" y="16.5735" size="1.27" layer="25" rot="R90">Carte Sharp-CAN</text>
+<wire x1="0.8255" y1="51.298" x2="0.762" y2="13.9065" width="0" layer="20"/>
+<text x="3.2385" y="18.415" size="1.27" layer="25" rot="R90">Carte Sharp-CAN</text>
 <text x="12.1285" y="14.859" size="1.4224" layer="25">Ares Dipole 2014</text>
 </plain>

Commit message: ajouts problemes
Parts:
- moved A5 2.15 mm to (2.52, 44.4)
- moved A4 0.69 mm to (2.54, 36.1)
Routing:
- net VCC: track 153.2 -> 139.2 mm
- net A5: track 13.9 -> 15.6 mm, vias 0 -> 1
Other:
- board text added: "& Dipole"
- board text added: "/home/showok/Documents/Projets/Ares/Robot-2013-2014/cartes/logo_ares_3.bmp"
- board text added: "ARES 2014"
- board text removed: "Ares Dipole 2014"

Commit message: nouvelles cartes à jour
Routing:
- net VCC: track 139.2 -> 138.4 mm
Changed lines of the file:
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@@
 <setting verticaltext="up"/>
 </settings>
-<grid distance="0.4" unitdist="mil" unit="mil" style="lines" multiple="1" display="yes" altdistance="0.0635" altunitdist="mm" altunit="mm"/>
+<grid distance="0.4" unitdist="mil" unit="mm" style="lines" multiple="1" display="yes" altdistance="0.0635" altunitdist="mm" altunit="mm"/>
 <layers>
 <layer number="1" name="Top" color="4" fill="1" visible="yes" active="yes"/>
@@
 <wire x1="12.2682" y1="45.8724" x2="12.2682" y2="42.3164" width="0.2" layer="1"/>
 <wire x1="11.0236" y1="41.0718" x2="10.9855" y2="40.9575" width="0.2" layer="1"/>
-<wire x1="4.445" y1="23.6474" x2="8.3566" y2="23.6474" width="0.2" layer="1"/>
-<wire x1="4.445" y1="36.8046" x2="4.445" y2="23.6474" width="0.2" layer="1"/>
+<wire x1="4.445" y1="36.8046" x2="4.445" y2="24.43599375" width="0.2" layer="1"/>
+<wire x1="4.445" y1="24.43599375" x2="5.23359375" y2="23.6474" width="0.2" layer="1"/>
+<wire x1="5.23359375" y1="23.6474" x2="8.3566" y2="23.6474" width="0.2" layer="1"/>
 <wire x1="6.223" y1="38.5826" x2="4.445" y2="36.8046" width="0.2" layer="1"/>
 <wire x1="6.223" y1="38.5826" x2="6.35" y2="38.679121875" width="0.2" layer="1"/>
 <wire x1="15.2908" y1="50.8508" x2="12.2682" y2="47.8282" width="0.2" layer="1"/>
-<wire x1="24.003" y1="50.8508" x2="15.2908" y2="50.8508" width="0.2" layer="1"/>
-<wire x1="24.003" y1="49.6062" x2="24.003" y2="50.8508" width="0.2" layer="1"/>
+<wire x1="24.003" y1="49.6062" x2="24.003" y2="50.31210625" width="0.2" layer="1"/>
+<wire x1="24.003" y1="50.31210625" x2="23.46430625" y2="50.8508" width="0.2" layer="1"/>
+<wire x1="23.46430625" y1="50.8508" x2="15.2908" y2="50.8508" width="0.2" layer="1"/>
 <wire x1="24.003" y1="49.6062" x2="24.13" y2="49.53" width="0.2" layer="1"/>
 </signal>
@@
 <contactref element="CAN" pad="1"/>
 <contactref element="CAN" pad="8"/>
-<wire x1="15.1638" y1="44.45" x2="11.1125" y2="46.482" width="0" layer="19" extent="1-1"/>
+<via x="13.49248125" y="42.204640625" extent="1-16" drill="0.3"/>
 </signal>
 <signal name="CAN_TXD">
@@
 <wire x1="9.9568" y1="24.5364" x2="7.2898" y2="24.5364" width="0.2" layer="16"/>
 <wire x1="11.557" y1="22.9362" x2="9.9568" y2="24.5364" width="0.2" layer="16"/>
-<wire x1="11.557" y1="20.9804" x2="11.557" y2="22.9362" width="0.2" layer="16"/>
-<wire x1="9.6012" y1="20.9804" x2="11.557" y2="20.9804" width="0.2" layer="16"/>
+<wire x1="9.6012" y1="20.9804" x2="11.238578125" y2="20.9804" width="0.2" layer="16"/>
+<wire x1="11.238578125" y1="20.9804" x2="11.557" y2="21.298821875" width="0.2" layer="16"/>
+<wire x1="11.557" y1="21.298821875" x2="11.557" y2="22.9362" width="0.2" layer="16"/>
 <wire x1="7.112" y1="24.7142" x2="6.985" y2="24.765" width="0.2" layer="16"/>
 <wire x1="9.6012" y1="20.9804" x2="9.525" y2="20.955" width="0.2" layer="16"/>
@@
 <contactref element="ARDUINO" pad="20"/>
 <contactref element="A3" pad="1"/>
-<wire x1="31.2928" y1="49.6062" x2="40.005" y2="49.6062" width="0.2" layer="1"/>
-<wire x1="31.2928" y1="48.006" x2="31.2928" y2="49.6062" width="0.2" layer="1"/>
+<wire x1="31.2928" y1="48.006" x2="31.2928" y2="49.098684375" width="0.2" layer="1"/>
+<wire x1="31.2928" y1="49.098684375" x2="31.800315625" y2="49.6062" width="0.2" layer="1"/>
+<wire x1="31.800315625" y1="49.6062" x2="40.005" y2="49.6062" width="0.2" layer="1"/>
 <wire x1="25.4254" y1="42.1386" x2="31.2928" y2="48.006" width="0.2" layer="16"/>
 <wire x1="24.1808" y1="42.1386" x2="25.4254" y2="42.1386" width="0.2" layer="16"/>
