File: cartes/Carte IA/bb2.brd (EAGLE design)
At the start: 139.4 x 118.1 mm, 26 parts, among them IC1 MIC5219BM5

Commit message: wait
Other:
- board size 139.4 x 118.1 mm -> 60 x 72.4 mm
Changed lines of the file:
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@@
 <board>
 <plain>
-<wire x1="0" y1="0" x2="139.37" y2="0" width="0" layer="20"/>
-<wire x1="139.37" y1="0" x2="139.37" y2="118.1" width="0" layer="20"/>
-<wire x1="139.37" y1="118.1" x2="0" y2="118.1" width="0" layer="20"/>
-<wire x1="0" y1="118.1" x2="0" y2="0" width="0" layer="20"/>
+<wire x1="25.4" y1="15.875" x2="85.395" y2="15.875" width="0" layer="20"/>
+<wire x1="85.395" y1="15.875" x2="85.395" y2="88.255" width="0" layer="20"/>
+<wire x1="85.395" y1="88.255" x2="25.4" y2="88.255" width="0" layer="20"/>
+<wire x1="25.4" y1="88.255" x2="25.4" y2="15.875" width="0" layer="20"/>
 <text x="57.15" y="76.2" size="6.4516" layer="37" font="vector" ratio="11">IA</text>
 <text x="48.26" y="58.42" size="2.54" layer="37" font="vector" ratio="11">ARES ENSEA</text>
