File: cartes/servo_shield/servo_1.brd (EAGLE design)
At the start: 53 x 55.2 mm, 32 parts, among them Q1 16MHz, U1 MCP2551, U2 ADUM1400ARWZ, U3 ADUM1250ARZ, U4 ADUM1400ARWZ, X1 5V_INPUT, X2 12V_INPUT

Commit message: servo
Parts:
- added INPUT: MMATCH-6-, jt-con-micromatch:AMP-215079-6
Connections:
- new net C_DIR1: INPUT.3
- new net C_DIR2: INPUT.5
- new net C_PWM1: INPUT.4
- new net C_PWM2: INPUT.6
- net GND: now also INPUT.2
- net VCC: now also INPUT.1
Changed lines of the file:
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@@
 <attribute name="OC_FARNELL" value="unknown" x="29.5275" y="46.355" size="1.778" layer="27" rot="R180" display="off"/>
 </element>
+<element name="INPUT" library="jt-con-micromatch" package="AMP-215079-6" value="MMATCH-6-" x="20.5105" y="16.7005"/>
 </elements>
 <signals>
@@
 <wire x1="63.246" y1="72.5805" x2="66.8274" y2="72.5805" width="0.6096" layer="1"/>
 <wire x1="66.8274" y1="72.5805" x2="66.8655" y2="72.5424" width="0.6096" layer="1"/>
+<contactref element="INPUT" pad="1"/>
+<wire x1="20.5105" y1="16.7005" x2="43.1038" y2="29.21" width="0" layer="19" extent="1-1"/>
 </signal>
 <signal name="GND">
@@
 <wire x1="64.008" y1="71.4756" x2="67.6021" y2="71.4756" width="0.3048" layer="16"/>
 <wire x1="67.6021" y1="71.4756" x2="67.7545" y2="71.628" width="0.3048" layer="16"/>
+<contactref element="INPUT" pad="2"/>
+<wire x1="63.8937" y1="71.4375" x2="61.987" y2="75.438" width="0" layer="19" extent="16-16"/>
+<wire x1="53.6575" y1="73.3425" x2="61.987" y2="75.438" width="0" layer="19" extent="16-16"/>
+<wire x1="55.88" y1="64.4525" x2="53.6575" y2="73.3425" width="0" layer="19" extent="1-1"/>
+<wire x1="44.7675" y1="70.8025" x2="53.6575" y2="73.3425" width="0" layer="19" extent="1-1"/>
+<wire x1="49.5935" y1="54.5465" x2="55.88" y2="64.4525" width="0" layer="19" extent="1-1"/>
+<wire x1="45.974" y1="53.34" x2="49.5935" y2="54.5465" width="0" layer="19" extent="16-16"/>
+<wire x1="45.974" y1="45.72" x2="45.974" y2="53.34" width="0" layer="19" extent="16-16"/>
+<wire x1="45.974" y1="43.18" x2="45.974" y2="45.72" width="0" layer="19" extent="16-16"/>
+<wire x1="48.7045" y1="43.434" x2="45.974" y2="43.18" width="0" layer="19" extent="16-16"/>
+<wire x1="45.974" y1="35.56" x2="45.974" y2="43.18" width="0" layer="19" extent="16-16"/>
+<wire x1="48.0695" y1="33.909" x2="45.974" y2="35.56" width="0" layer="19" extent="16-16"/>
+<wire x1="43.1038" y1="33.02" x2="45.974" y2="35.56" width="0" layer="19" extent="1-16"/>
+<wire x1="49.2125" y1="29.845" x2="48.0695" y2="33.909" width="0" layer="19" extent="1-1"/>
+<wire x1="64.5905" y1="26.924" x2="49.2125" y2="29.845" width="0" layer="19" extent="16-16"/>
+<wire x1="67.045" y1="26.8605" x2="64.5905" y2="26.924" width="0" layer="19" extent="16-16"/>
+<wire x1="66.4972" y1="47.3075" x2="48.7045" y2="43.434" width="0" layer="19" extent="16-16"/>
+<wire x1="21.7805" y1="19.2405" x2="43.1038" y2="33.02" width="0" layer="19" extent="1-1"/>
 </signal>
 <signal name="CAN_TXD">
@@
 <wire x1="28.0924" y1="47.8282" x2="28.0375" y2="47.9425" width="0.254" layer="1"/>
 </signal>
+<signal name="C_PWM2">
+<contactref element="INPUT" pad="6"/>
+</signal>
+<signal name="C_DIR2">
+<contactref element="INPUT" pad="5"/>
+</signal>
+<signal name="C_PWM1">
+<contactref element="INPUT" pad="4"/>
+</signal>
+<signal name="C_DIR1">
+<contactref element="INPUT" pad="3"/>
+</signal>
 </signals>

Commit message: ajouts carte puissance
Parts:
- removed CARTE_PUISSANCE: (no value), jt-con-micromatch:AMP-215079-8
- removed INPUT: MMATCH-6-, jt-con-micromatch:AMP-215079-6
- removed JP1: end_lign, SparkFun-Passives:1X02
- removed JP11: PWM3, SparkFun-Connectors:1X03
- removed JP13: PWM6, SparkFun-Connectors:1X03
- added CAN_LINE: JUMPER-3PTH, SparkFun-Passives:1X03
- added PUISSANCE: MMATCH-6-, jt-con-micromatch:AMP-215079-6
- added PWM3: PWM3, SparkFun-Connectors:1X03
- added PWM6: servo_option, SparkFun-Connectors:1X03
- added R5: 10k, SparkFun-Passives:0805
- moved C4 1.40 mm to (36.4, 62.0)
- moved C3 1.14 mm to (26.4, 62.0)
- moved X1 1.14 mm to (36.2, 73.2)
- moved X2 1.08 mm to (26.4, 73.2)
- moved JP6 0.44 mm to (63.2, 67.4)
- moved R2 0.06 mm to (43.8, 64.8)
- renumbered JP10 to OUT8, JP14 to OUT4, JP7 to OUT7, JP8 to PWM5, JP9 to PWM9, LED1 to LED_5V, LED3 to LED_12V, Q1 to 16MHZ, SK1 to CAN, U$2 to CONTROLLER, U$3 to ARDUINO, U1 to TRANSCEIVER, U2 to ADUM1400_, U3 to ADUM1250, U4 to ADUM1400
Connections:
- net PWM4 renamed OUT4
- removed net C_DIR1: INPUT.3
- removed net C_DIR2: INPUT.5
- removed net C_PWM1: INPUT.4
- removed net C_PWM2: INPUT.6
- removed net PWM7: ADUM1400.3, ARDUINO.10, CARTE_PUISSANCE.7
- removed net PWM8: ADUM1400.4, ARDUINO.11, CARTE_PUISSANCE.3
- new net OUT7: ADUM1400.3, ARDUINO.10, PUISSANCE.5
- new net OUT8: ADUM1400.4, ARDUINO.11, PUISSANCE.3
- net 12V_DIRTY: now also R5.1
- net 5V_DIRTY: now also PWM3.2, PWM6.2; no longer JP11.2, JP13.2
- net CANH: now also CAN_LINE.3; no longer JP1.2
- net GND: now also PUISSANCE.2; no longer CARTE_PUISSANCE.2, INPUT.2
- net GND_DIRTY: now also PWM3.3, PWM6.3; no longer JP11.3, JP13.3
- net N$7: now also CAN_LINE.2; no longer JP1.1
- net PWM3_OUT: now also PWM3.1; no longer JP11.1
- net PWM6: now also PUISSANCE.6; no longer CARTE_PUISSANCE.6
- net PWM6_OUT: now also PWM6.1; no longer JP13.1
- net PWM9: now also PUISSANCE.4; no longer CARTE_PUISSANCE.4
- net RXTX_OUT: now also R5.2
- net VCC: now also PUISSANCE.1; no longer CARTE_PUISSANCE.1, INPUT.1
Routing:
- net OUT8: track 0.00 -> 33.6 mm, vias 0 -> 1
- net PWM7: track 22.5 -> 0.00 mm
- net OUT7: track 0.00 -> 22.2 mm
- net PWM8: track 19.7 -> 0.00 mm
- net GND_DIRTY: track 2.25 -> 18.7 mm
- net CANL: track 29.2 -> 20.4 mm
- net VCC: track 98.5 -> 105.2 mm, vias 1 -> 3
- net 12V_DIRTY: track 57.0 -> 61.4 mm
- net 5V_DIRTY: track 89.9 -> 94.2 mm
- net RXTX_OUT: track 13.2 -> 16.2 mm
- net PWM6: track 23.0 -> 25.7 mm
- net PWM9: track 12.7 -> 15.1 mm
- net CANH: track 19.2 -> 20.3 mm
- net GND: track 5.03 -> 5.22 mm, vias 3 -> 2
Other:
- board size 53 x 55.2 mm -> 55.8 x 54.8 mm
- board text added: "+12V"
- board text added: "+5V"
- board text added: "12V"
- board text added: "2014"
- board text added: "AX-12"
- board text added: "Actionneurs"
- board text added: "Carte"
- board text added: "Controller CAN"
- board text added: "DATA"
- board text added: "GND"
- board text added: "RX TX switch"
- board text added: "avec Dipole"
