File: cartes/servo_shield/servo_1.brd (EAGLE design)
At the start: 55.8 x 54.8 mm, 33 parts, among them X1 5V_INPUT, X2 12V_INPUT

Commit message: plein de trucs
Other:
- board text added: "Carte actionneurs 2014"

Commit message: nouvelles cartes à jour
Routing:
- net SCK: track 33.9 -> 27.2 mm
- net VCC: track 105.3 -> 101.1 mm
- net CAN_RXD: track 18.9 -> 17.8 mm
- net CAN_TXD: track 23.3 -> 22.3 mm
Changed lines of the file:
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@@
 <wire x1="54.0512" y1="52.0954" x2="54.9402" y2="51.2064" width="0.254" layer="1"/>
 <wire x1="54.0512" y1="55.2958" x2="54.0512" y2="52.0954" width="0.254" layer="1"/>
-<wire x1="54.5846" y1="55.8292" x2="54.0512" y2="55.2958" width="0.254" layer="1"/>
-<wire x1="67.2084" y1="55.8292" x2="54.5846" y2="55.8292" width="0.254" layer="1"/>
-<wire x1="67.2084" y1="41.6052" x2="67.2084" y2="55.8292" width="0.254" layer="1"/>
+<wire x1="67.1728375" y1="44.45" x2="55.7453625" y2="55.80975625" width="0.254" layer="1"/>
+<wire x1="55.7453625" y1="55.80975625" x2="54.5898625" y2="55.817359375" width="0.254" layer="1"/>
+<wire x1="54.5898625" y1="55.817359375" x2="54.0512" y2="55.2958" width="0.254" layer="1"/>
+<wire x1="67.2084" y1="41.6052" x2="67.1728375" y2="44.45" width="0.254" layer="1"/>
 <wire x1="56.5404" y1="51.2064" x2="56.6928" y2="51.1175" width="0.254" layer="16"/>
 <wire x1="67.2084" y1="41.6052" x2="67.31" y2="41.5925" width="0.254" layer="1"/>
@@
 <wire x1="46.0502" y1="54.7624" x2="45.974" y2="54.61" width="0.254" layer="16"/>
 <wire x1="47.4726" y1="74.8538" x2="46.0502" y2="73.4314" width="0.254" layer="1"/>
-<wire x1="52.2732" y1="74.8538" x2="47.4726" y2="74.8538" width="0.254" layer="1"/>
-<wire x1="52.2732" y1="70.9422" x2="52.2732" y2="74.8538" width="0.254" layer="1"/>
+<wire x1="52.2732" y1="70.9422" x2="52.2732" y2="73.9737375" width="0.254" layer="1"/>
+<wire x1="52.2732" y1="73.9737375" x2="51.3931375" y2="74.8538" width="0.254" layer="1"/>
+<wire x1="51.3931375" y1="74.8538" x2="47.4726" y2="74.8538" width="0.254" layer="1"/>
 <wire x1="46.0502" y1="73.4314" x2="46.0375" y2="73.3425" width="0.254" layer="1"/>
 <wire x1="52.2732" y1="70.9422" x2="52.3875" y2="70.8025" width="0.254" layer="1"/>
 <wire x1="66.8655" y1="72.5424" x2="64.008" y2="72.5424" width="0.254" layer="16"/>
-<wire x1="57.2516" y1="66.1416" x2="57.2516" y2="72.5424" width="0.254" layer="1"/>
 <wire x1="64.008" y1="72.5424" x2="63.8937" y2="72.7075" width="0.254" layer="16"/>
 <wire x1="57.2516" y1="66.1416" x2="57.1627" y2="66.0527" width="0.254" layer="1"/>
 <via x="66.8655" y="72.5424" extent="1-16" drill="0.6096"/>
-<wire x1="57.2516" y1="72.5424" x2="63.2079" y2="72.5424" width="0.3048" layer="1"/>
-<wire x1="63.2079" y1="72.5424" x2="63.246" y2="72.5805" width="0.3048" layer="1"/>
-<wire x1="63.246" y1="72.5805" x2="66.8274" y2="72.5805" width="0.6096" layer="1"/>
 <wire x1="66.8274" y1="72.5805" x2="66.8655" y2="72.5424" width="0.6096" layer="1"/>
 <contactref element="PUISSANCE" pad="1"/>
@@
 <wire x1="50.3174" y1="25.6032" x2="50.4825" y2="25.5905" width="0.2" layer="1"/>
 <wire x1="43.2054" y1="29.1592" x2="43.1038" y2="29.21" width="0.2" layer="1"/>
+<wire x1="57.2516" y1="66.1416" x2="63.6524" y2="72.5424" width="0.4064" layer="1"/>
+<wire x1="63.6524" y1="72.5424" x2="66.8655" y2="72.5424" width="0.4064" layer="1"/>
 </signal>
 <signal name="GND">
@@
 <wire x1="66.675" y1="63.119" x2="66.4972" y2="63.119" width="0.254" layer="16"/>
 <wire x1="67.3862" y1="63.8302" x2="66.675" y2="63.119" width="0.254" layer="16"/>
-<wire x1="67.3862" y1="69.5198" x2="67.3862" y2="63.8302" width="0.254" layer="16"/>
-<wire x1="62.5856" y1="69.5198" x2="67.3862" y2="69.5198" width="0.254" layer="16"/>
+<wire x1="62.5856" y1="69.5198" x2="65.647303125" y2="69.5198" width="0.254" layer="16"/>
+<wire x1="65.647303125" y1="69.5198" x2="67.3862" y2="67.780903125" width="0.254" layer="16"/>
+<wire x1="67.3862" y1="67.780903125" x2="67.3862" y2="63.8302" width="0.254" layer="16"/>
 <wire x1="62.4078" y1="69.6976" x2="62.5856" y2="69.5198" width="0.254" layer="16"/>
 <wire x1="62.4078" y1="73.9648" x2="62.4078" y2="69.6976" width="0.254" layer="16"/>
@@
 <wire x1="67.564" y1="56.7182" x2="66.8528" y2="56.7182" width="0.254" layer="16"/>
 <wire x1="67.9196" y1="57.0738" x2="67.564" y2="56.7182" width="0.254" layer="16"/>
-<wire x1="67.9196" y1="70.0532" x2="67.9196" y2="57.0738" width="0.254" layer="16"/>
-<wire x1="64.008" y1="70.0532" x2="67.9196" y2="70.0532" width="0.254" layer="16"/>
+<wire x1="64.008" y1="70.0532" x2="65.909203125" y2="70.0532" width="0.254" layer="16"/>
+<wire x1="65.909203125" y1="70.0532" x2="67.9196" y2="68.042803125" width="0.254" layer="16"/>
+<wire x1="67.9196" y1="68.042803125" x2="67.9196" y2="57.0738" width="0.254" layer="16"/>
 <wire x1="66.4972" y1="56.3626" x2="66.4972" y2="56.1975" width="0.254" layer="16"/>
 <wire x1="64.008" y1="70.0532" x2="63.8937" y2="70.1675" width="0.254" layer="16"/>
@@
 <contactref element="CAN" pad="5"/>
 <wire x1="57.9628" y1="72.7456" x2="58.4962" y2="72.7202" width="0.254" layer="16"/>
-<wire x1="55.2958" y1="73.2536" x2="57.9628" y2="72.7456" width="0.254" layer="16"/>
-<wire x1="54.0512" y1="74.4982" x2="55.2958" y2="73.2536" width="0.254" layer="16"/>
+<wire x1="54.0512" y1="74.4982" x2="55.155528125" y2="73.393871875" width="0.254" layer="16"/>
+<wire x1="55.155528125" y1="73.393871875" x2="55.84626875" y2="72.7542" width="0.254" layer="16"/>
+<wire x1="55.84626875" y1="72.7542" x2="57.9628" y2="72.7456" width="0.254" layer="16"/>
 <wire x1="49.784" y1="74.4982" x2="54.0512" y2="74.4982" width="0.254" layer="16"/>
 <wire x1="48.7172" y1="73.4314" x2="49.784" y2="74.4982" width="0.254" layer="16"/>
@@
 <wire x1="50.3682" y1="31.8262" x2="43.2054" y2="31.8262" width="0.254" layer="1"/>
 <wire x1="61.1632" y1="63.119" x2="50.673" y2="52.6288" width="0.254" layer="1"/>
-<wire x1="63.4746" y1="63.119" x2="61.1632" y2="63.119" width="0.254" layer="1"/>
-<wire x1="63.4746" y1="64.3636" x2="63.4746" y2="63.119" width="0.254" layer="1"/>
+<wire x1="63.4746" y1="64.3636" x2="63.4746" y2="63.74104375" width="0.254" layer="1"/>
+<wire x1="63.4746" y1="63.74104375" x2="62.85255625" y2="63.119" width="0.254" layer="1"/>
+<wire x1="62.85255625" y1="63.119" x2="61.1632" y2="63.119" width="0.254" layer="1"/>
 <wire x1="43.2054" y1="31.8262" x2="43.1038" y2="31.75" width="0.254" layer="1"/>
 <wire x1="63.4746" y1="64.3636" x2="63.5" y2="64.4525" width="0.254" layer="1"/>
