File: cartes/servo_shield/servo_1.sch (EAGLE design)
At the start: 32 parts, among them Q1 16MHz, U1 MCP2551, U2 ADUM1400ARWZ, U3 ADUM1250ARZ, U4 ADUM1400ARWZ, X1 5V_INPUT, X2 12V_INPUT

Commit message: servo
Parts:
- added INPUT: MMATCH-6-, jt-con-micromatch:MMATCH-6-
Connections:
- new net C_DIR1: INPUT.5
- new net C_DIR2: INPUT.7
- new net C_PWM1: INPUT.6
- new net C_PWM2: INPUT.8
- net GND: now also INPUT.4
- net VCC: now also INPUT.3
Changed lines of the file:
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@@
 <attribute name="OC_FARNELL" value="unknown"/>
 </part>
+<part name="INPUT" library="jt-con-micromatch" deviceset="MMATCH-6-*" device=""/>
+<part name="P+3" library="supply1" deviceset="VCC" device=""/>
+<part name="GND1" library="supply1" deviceset="GND" device=""/>
 </parts>
 <sheets>
@@
 <attribute name="MPN" x="-15.24" y="-5.08" size="1.778" layer="96" rot="R90" display="off"/>
 </instance>
+<instance part="INPUT" gate="G$1" x="-48.26" y="26.67"/>
+<instance part="P+3" gate="VCC" x="-59.69" y="16.51" rot="R180"/>
+<instance part="GND1" gate="1" x="-38.1" y="16.51"/>
 </instances>
 <busses>
@@
 <wire x1="-15.24" y1="17.78" x2="-22.86" y2="17.78" width="0.1524" layer="91"/>
 <label x="-25.4" y="17.78" size="1.778" layer="95"/>
+</segment>
+<segment>
+<pinref part="INPUT" gate="G$1" pin="3"/>
+<wire x1="-53.34" y1="24.13" x2="-59.69" y2="24.13" width="0.1524" layer="91"/>
+<wire x1="-59.69" y1="24.13" x2="-59.69" y2="19.05" width="0.1524" layer="91"/>
+<pinref part="P+3" gate="VCC" pin="VCC"/>
 </segment>
 </net>
@@
 <label x="2.54" y="17.78" size="1.778" layer="95"/>
 </segment>
+<segment>
+<pinref part="INPUT" gate="G$1" pin="4"/>
+<wire x1="-43.18" y1="24.13" x2="-38.1" y2="24.13" width="0.1524" layer="91"/>
+<wire x1="-38.1" y1="24.13" x2="-38.1" y2="19.05" width="0.1524" layer="91"/>
+<pinref part="GND1" gate="1" pin="GND"/>
+</segment>
 </net>
 <net name="CAN_TXD" class="0">
@@
 <net name="PWM7" class="0">
 <segment>
-<wire x1="-22.86" y1="58.42" x2="-40.64" y2="58.42" width="0.1524" layer="91"/>
+<wire x1="-22.86" y1="58.42" x2="-35.56" y2="58.42" width="0.1524" layer="91"/>
 <label x="-35.56" y="58.42" size="1.778" layer="95"/>
 <pinref part="U$3" gate="G$1" pin="7"/>
@@
 </segment>
 </net>
+<net name="C_PWM2" class="0">
+<segment>
+<pinref part="INPUT" gate="G$1" pin="8"/>
+<wire x1="-43.18" y1="29.21" x2="-38.1" y2="29.21" width="0.1524" layer="91"/>
+<label x="-38.1" y="29.21" size="1.778" layer="95"/>
+</segment>
+</net>
+<net name="C_DIR2" class="0">
+<segment>
+<pinref part="INPUT" gate="G$1" pin="7"/>
+<wire x1="-53.34" y1="29.21" x2="-58.42" y2="29.21" width="0.1524" layer="91"/>
+<label x="-58.42" y="29.21" size="1.778" layer="95" rot="R180"/>
+</segment>
+</net>
+<net name="C_PWM1" class="0">
+<segment>
+<pinref part="INPUT" gate="G$1" pin="6"/>
+<wire x1="-43.18" y1="26.67" x2="-38.1" y2="26.67" width="0.1524" layer="91"/>
+<label x="-38.1" y="26.67" size="1.778" layer="95"/>
+</segment>
+</net>
+<net name="C_DIR1" class="0">
+<segment>
+<pinref part="INPUT" gate="G$1" pin="5"/>
+<wire x1="-53.34" y1="26.67" x2="-58.42" y2="26.67" width="0.1524" layer="91"/>
+<label x="-58.42" y="26.67" size="1.778" layer="95" rot="R180"/>
+</segment>
+</net>

Commit message: ajouts carte puissance
Parts:
- removed CARTE_PUISSANCE: (no value), jt-con-micromatch:MMATCH-8-PTH
- removed JP1: end_lign, SparkFun-Passives:JUMPER-2PTH
- added CAN_LINE: JUMPER-3PTH, SparkFun-Passives:JUMPER-3PTH
- added R5: 10k, SparkFun-Passives:RESISTOR0805-RES
- PWM6: value PWM6 -> servo_option
- renumbered INPUT to PUISSANCE, JP10 to OUT8, JP11 to PWM3, JP13 to PWM6, JP14 to OUT4, JP7 to OUT7, JP8 to PWM5, JP9 to PWM9, LED1 to LED_5V, LED3 to LED_12V, Q1 to 16MHZ, SK1 to CAN, U$2 to CONTROLLER, U$3 to ARDUINO, U1 to TRANSCEIVER, U2 to ADUM1400_, U3 to ADUM1250, U4 to ADUM1400
Connections:
- net PWM4 renamed OUT4
- removed net C_DIR1: PUISSANCE.5
- removed net C_DIR2: PUISSANCE.7
- removed net C_PWM1: PUISSANCE.6
- removed net C_PWM2: PUISSANCE.8
- removed net PWM7: ADUM1400.VIA, ARDUINO.7, CARTE_PUISSANCE.7
- removed net PWM8: ADUM1400.VIB, ARDUINO.8, CARTE_PUISSANCE.3
- new net OUT7: ADUM1400.VIA, ARDUINO.7, PUISSANCE.7
- new net OUT8: ADUM1400.VIB, ARDUINO.8, PUISSANCE.5
- net 12V_DIRTY: now also R5.1
- net CANH: now also CAN_LINE.3; no longer JP1.2
- net GND: no longer CARTE_PUISSANCE.2
- net N$7: now also CAN_LINE.2; no longer JP1.1
- net PWM6: now also PUISSANCE.8; no longer CARTE_PUISSANCE.6
- net PWM9: now also PUISSANCE.6; no longer CARTE_PUISSANCE.4
- net RXTX_OUT: now also R5.2
- net VCC: no longer CARTE_PUISSANCE.1
