File: cartes/Carte_puissance/schema_puissance.brd (EAGLE design)
At the start: 73.7 x 46.6 mm, 22 parts, among them X2 GMSTBA2

Commit message: servo
Parts:
- renumbered U$4 to INPUT
Changed lines of the file:
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@@
 <element name="C5" library="rcl" package="C0805" value="100nF" x="32.4" y="25" rot="R90"/>
 <element name="C7" library="rcl" package="C0805" value="100nF" x="17.5" y="18.7" rot="R270"/>
-<element name="U$4" library="jt-con-micromatch" package="AMP-215079-6" value="MMATCH-6-" x="20.7" y="10.2"/>
+<element name="INPUT" library="jt-con-micromatch" package="AMP-215079-6" value="MMATCH-6-" x="20.7" y="10.2"/>
 </elements>
 <signals>
@@
 <contactref element="U$3" pad="6"/>
 <contactref element="SV1" pad="1"/>
-<contactref element="U$4" pad="6"/>
+<contactref element="INPUT" pad="6"/>
 <wire x1="27.005" y1="17.4" x2="27.05" y2="17.4" width="0.4064" layer="1"/>
 <wire x1="27.05" y1="17.4" x2="27.05" y2="12.74" width="0.4064" layer="1"/>
@@
 <contactref element="U$3" pad="5"/>
 <contactref element="SV1" pad="2"/>
-<contactref element="U$4" pad="5"/>
+<contactref element="INPUT" pad="5"/>
 <wire x1="25.735" y1="17.4" x2="25.78" y2="17.4" width="0.4064" layer="1"/>
 <wire x1="25.78" y1="17.4" x2="25.78" y2="10.2" width="0.4064" layer="1"/>
@@
 <contactref element="U$3" pad="4"/>
 <contactref element="SV1" pad="3"/>
-<contactref element="U$4" pad="4"/>
+<contactref element="INPUT" pad="4"/>
 <wire x1="24.465" y1="17.4" x2="24.51" y2="17.4" width="0.4064" layer="1"/>
 <wire x1="24.51" y1="17.4" x2="24.51" y2="12.74" width="0.4064" layer="1"/>
@@
 <contactref element="U$3" pad="3"/>
 <contactref element="SV1" pad="4"/>
-<contactref element="U$4" pad="3"/>
+<contactref element="INPUT" pad="3"/>
 <wire x1="23.195" y1="17.4" x2="23.24" y2="17.4" width="0.4064" layer="1"/>
 <wire x1="23.24" y1="17.4" x2="23.24" y2="10.2" width="0.4064" layer="1"/>
@@
 <wire x1="67.64" y1="11.16" x2="71.53" y2="11.16" width="0.6096" layer="1"/>
 <wire x1="71.53" y1="11.16" x2="71.54" y2="11.15" width="0.6096" layer="1"/>
-<contactref element="U$4" pad="1"/>
+<contactref element="INPUT" pad="1"/>
 <wire x1="20.3" y1="17.045" x2="20.3" y2="10.6" width="0.6096" layer="1"/>
 <wire x1="20.3" y1="10.6" x2="20.7" y2="10.2" width="0.6096" layer="1"/>
@@
 <wire x1="21.9" y1="18.7" x2="21.9" y2="17.425" width="0.6096" layer="1"/>
 <wire x1="21.9" y1="17.425" x2="21.925" y2="17.4" width="0.6096" layer="1"/>
-<contactref element="U$4" pad="2"/>
+<contactref element="INPUT" pad="2"/>
 </signal>
 <signal name="N$2">

Commit message: plein de trucs
Parts:
- renumbered SV1 to HEADER
Other:
- board text added: "&"
- board text added: "2014"
