File: cartes/Carte_puissance/schema_puissance.sch (EAGLE design)
At the start: 22 parts, among them X2 GMSTBA2

Commit message: servo
Parts:
- renumbered U$4 to INPUT
Changed lines of the file:
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@@
 <part name="C5" library="rcl" deviceset="C-EU" device="C0805" value="100nF"/>
 <part name="C7" library="rcl" deviceset="C-EU" device="C0805" value="100nF"/>
-<part name="U$4" library="jt-con-micromatch" deviceset="MMATCH-6-*" device=""/>
+<part name="INPUT" library="jt-con-micromatch" deviceset="MMATCH-6-*" device=""/>
 <part name="P+3" library="supply1" deviceset="VCC" device=""/>
 <part name="GND2" library="supply1" deviceset="GND" device=""/>
@@
 <instance part="C5" gate="G$1" x="-71.755" y="-27.305" rot="R90"/>
 <instance part="C7" gate="G$1" x="-132.715" y="-29.845" rot="R90"/>
-<instance part="U$4" gate="G$1" x="-149.86" y="-74.93"/>
+<instance part="INPUT" gate="G$1" x="-149.86" y="-74.93"/>
 <instance part="P+3" gate="VCC" x="-161.29" y="-85.09" rot="R180"/>
 <instance part="GND2" gate="1" x="-139.7" y="-85.09"/>
@@
 </segment>
 <segment>
-<pinref part="U$4" gate="G$1" pin="8"/>
+<pinref part="INPUT" gate="G$1" pin="8"/>
 <wire x1="-144.78" y1="-72.39" x2="-139.7" y2="-72.39" width="0.1524" layer="91"/>
 <label x="-139.7" y="-72.39" size="1.778" layer="95"/>
@@
 </segment>
 <segment>
-<pinref part="U$4" gate="G$1" pin="7"/>
+<pinref part="INPUT" gate="G$1" pin="7"/>
 <wire x1="-154.94" y1="-72.39" x2="-160.02" y2="-72.39" width="0.1524" layer="91"/>
 <label x="-160.02" y="-72.39" size="1.778" layer="95" rot="R180"/>
@@
 </segment>
 <segment>
-<pinref part="U$4" gate="G$1" pin="6"/>
+<pinref part="INPUT" gate="G$1" pin="6"/>
 <wire x1="-144.78" y1="-74.93" x2="-139.7" y2="-74.93" width="0.1524" layer="91"/>
 <label x="-139.7" y="-74.93" size="1.778" layer="95"/>
@@
 </segment>
 <segment>
-<pinref part="U$4" gate="G$1" pin="5"/>
+<pinref part="INPUT" gate="G$1" pin="5"/>
 <wire x1="-154.94" y1="-74.93" x2="-160.02" y2="-74.93" width="0.1524" layer="91"/>
 <label x="-160.02" y="-74.93" size="1.778" layer="95" rot="R180"/>
@@
 </segment>
 <segment>
-<pinref part="U$4" gate="G$1" pin="3"/>
+<pinref part="INPUT" gate="G$1" pin="3"/>
 <wire x1="-154.94" y1="-77.47" x2="-161.29" y2="-77.47" width="0.1524" layer="91"/>
 <wire x1="-161.29" y1="-77.47" x2="-161.29" y2="-82.55" width="0.1524" layer="91"/>
@@
 </segment>
 <segment>
-<pinref part="U$4" gate="G$1" pin="4"/>
+<pinref part="INPUT" gate="G$1" pin="4"/>
 <wire x1="-144.78" y1="-77.47" x2="-139.7" y2="-77.47" width="0.1524" layer="91"/>
 <wire x1="-139.7" y1="-77.47" x2="-139.7" y2="-82.55" width="0.1524" layer="91"/>

Commit message: plein de trucs
Parts:
- renumbered SV1 to HEADER
Changed lines of the file:
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@@
 <part name="U$6" library="WEIDMULLER" deviceset="SL-3.5-2-90G" device=""/>
 <part name="U$7" library="WEIDMULLER" deviceset="SL-3.5-2-90G" device=""/>
-<part name="SV1" library="con-lsta" deviceset="FE06-1" device=""/>
+<part name="HEADER" library="con-lsta" deviceset="FE06-1" device=""/>
 <part name="P+13" library="supply1" deviceset="VCC" device=""/>
 <part name="GND12" library="supply1" deviceset="GND" device=""/>
@@
 <instance part="U$6" gate="G$1" x="83.82" y="58.42" rot="R180"/>
 <instance part="U$7" gate="G$1" x="81.28" y="2.54" rot="R180"/>
-<instance part="SV1" gate="G$1" x="-121.92" y="17.78"/>
+<instance part="HEADER" gate="G$1" x="-121.92" y="17.78"/>
 <instance part="P+13" gate="VCC" x="-106.68" y="33.02"/>
 <instance part="GND12" gate="1" x="-96.52" y="33.02" rot="R180"/>
@@
 </segment>
 <segment>
-<pinref part="SV1" gate="G$1" pin="1"/>
+<pinref part="HEADER" gate="G$1" pin="1"/>
 <wire x1="-114.3" y1="12.7" x2="-104.14" y2="12.7" width="0.1524" layer="91"/>
 <label x="-104.14" y="12.7" size="1.778" layer="95"/>
@@
 </segment>
 <segment>
-<pinref part="SV1" gate="G$1" pin="2"/>
+<pinref part="HEADER" gate="G$1" pin="2"/>
 <wire x1="-114.3" y1="15.24" x2="-104.14" y2="15.24" width="0.1524" layer="91"/>
 <label x="-104.14" y="15.24" size="1.778" layer="95"/>
@@
 </segment>
 <segment>
-<pinref part="SV1" gate="G$1" pin="3"/>
+<pinref part="HEADER" gate="G$1" pin="3"/>
 <wire x1="-114.3" y1="17.78" x2="-104.14" y2="17.78" width="0.1524" layer="91"/>
 <label x="-104.14" y="17.78" size="1.778" layer="95"/>
@@
 </segment>
 <segment>
-<pinref part="SV1" gate="G$1" pin="4"/>
+<pinref part="HEADER" gate="G$1" pin="4"/>
 <wire x1="-114.3" y1="20.32" x2="-104.14" y2="20.32" width="0.1524" layer="91"/>
 <label x="-104.14" y="20.32" size="1.778" layer="95"/>
@@
 </segment>
 <segment>
-<pinref part="SV1" gate="G$1" pin="6"/>
+<pinref part="HEADER" gate="G$1" pin="6"/>
 <pinref part="P+13" gate="VCC" pin="VCC"/>
 <wire x1="-114.3" y1="25.4" x2="-106.68" y2="25.4" width="0.1524" layer="91"/>
@@
 </segment>
 <segment>
-<pinref part="SV1" gate="G$1" pin="5"/>
+<pinref part="HEADER" gate="G$1" pin="5"/>
 <pinref part="GND12" gate="1" pin="GND"/>
 <wire x1="-114.3" y1="22.86" x2="-96.52" y2="22.86" width="0.1524" layer="91"/>
