File: cartes/Carte asserv/board.sch (EAGLE design)
At the start: 13 parts, among them X1 MICROMATCH-6, X2 MICROMATCH-6

Commit message: nouvelles cartes à jour
Parts:
- removed X1, X2: MICROMATCH-6, con-amp-micromatch:MICROMATCH-6
- added ADC0, ADC1: MMATCH-6-, jt-con-micromatch:MMATCH-6-
- added COULEUR: MMATCH-4-, jt-con-micromatch:MMATCH-4-
- added PWM: (no value), pinhead:PINHD-1X6/90
- added R10, R11: 10k, rcl:R-EU_R0805
- CAN: value MICROMATCH-8 -> (none); device con-amp-micromatch:MICROMATCH-8 -> jt-con-micromatch:MMATCH-8-PTH
- COMMAND: value MICROMATCH-8 -> MMATCH-6-; device con-amp-micromatch:MICROMATCH-8 -> jt-con-micromatch:MMATCH-6-
- renumbered JP1 to JUMPERCAN
Connections:
- removed net TF1: COMMAND-8.S
- removed net TF2: COMMAND-5.S
- new net COULEUR: COULEUR.8, R11.2, TIVA.PF0
- new net PWM1: PWM.3, TIVA.PB6
- new net PWM2: PWM.4, TIVA.PA6
- new net PWM3: PWM.5, TIVA.PA7
- new net PWM4: PWM.6, TIVA.PC4
- new net TIRETTE: COULEUR.6, R10.2, TIVA.PB7
- new net VDD_3V3: COULEUR.7, TIVA.3.3V
- net +5V: now also ADC0.8, ADC1.8, CAN.2, CAN.7, COMMAND.3, PWM.1; no longer CAN-2.S, CAN-7.S, COMMAND-1.S, X1-1.S, X2-1.S
- net ADC_0: now also ADC0.5; no longer X1-3.S
- net ADC_1: now also ADC0.3; no longer X1-4.S
- net ADC_2: now also ADC0.6; no longer X1-5.S
- net ADC_3: now also ADC0.4; no longer X1-6.S
- net ADC_4: now also ADC1.5; no longer X2-3.S
- net ADC_5: now also ADC1.3; no longer X2-4.S
- net ADC_6: now also ADC1.6; no longer X2-5.S
- net ADC_7: now also ADC1.4; no longer X2-6.S
- net CANH: now also CAN.4, CAN.5; no longer CAN-4.S, CAN-5.S
- net CANL: now also CAN.3, CAN.6; no longer CAN-3.S, CAN-6.S
- net DIR1: now also COMMAND.5; no longer COMMAND-7.S
- net DIR2: now also COMMAND.7; no longer COMMAND-4.S
- net GND: now also ADC0.7, ADC1.7, CAN.1, CAN.8, COMMAND.4, COULEUR.5, PWM.2, R10.1, R11.1; no longer CAN-1.S, CAN-8.S, COMMAND-2.S, X1-2.S, X2-2.S
- net PWM_MOT1: now also COMMAND.6; no longer COMMAND-6.S
- net PWM_MOT2: now also COMMAND.8; no longer COMMAND-3.S
Other:
- moved on the sheet: UART
