File: cartes/Carte plan B/board.sch (EAGLE design)
At the start: 20 parts

Commit message: nouvelle version nouveau jumper
Parts:
- removed JUMPERCAN: header-3, jumper:JP2W
- added JUMPER: (no value), pinhead:PINHD-1X3
Connections:
- net CANH: now also JUMPER.2; no longer JUMPERCAN.2
- net N$9: now also JUMPER.3; no longer JUMPERCAN.1
Changed lines of the file:
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@@
 <part name="P+1" library="supply1" deviceset="+5V" device=""/>
 <part name="R1" library="rcl" deviceset="R-EU_" device="R0805" value="21k"/>
-<part name="JUMPERCAN" library="jumper" deviceset="JP2W" device="" value="header-3"/>
 <part name="R5" library="rcl" deviceset="R-US_" device="M0805" value="120"/>
 <part name="I2C" library="con-molex" deviceset="22-23-2021" device="" value="header-2"/>
@@
 <part name="ISOLATEURGALVANIQUE" library="Analog Devices_By_element14_Batch_1" deviceset="ADUM1250ARZ" device=""/>
 <part name="C2" library="mbed-rlcq" deviceset="C" device="0805" value="100u"/>
+<part name="JUMPER" library="pinhead" deviceset="PINHD-1X3" device=""/>
 </parts>
 <sheets>
@@
 <instance part="P+1" gate="1" x="116.84" y="177.8"/>
 <instance part="R1" gate="G$1" x="73.66" y="167.64" rot="R90"/>
-<instance part="JUMPERCAN" gate="1" x="86.36" y="134.62" rot="R90"/>
 <instance part="R5" gate="G$1" x="96.52" y="132.08" rot="R180"/>
 <instance part="I2C" gate="-1" x="30.48" y="180.34"/>
@@
 <instance part="ISOLATEURGALVANIQUE" gate="A" x="71.12" y="63.5"/>
 <instance part="C2" gate="G$1" x="256.54" y="99.06"/>
+<instance part="JUMPER" gate="A" x="83.82" y="134.62" rot="MR0"/>
 </instances>
 <busses>
@@
 </segment>
 <segment>
-<wire x1="88.9" y1="134.62" x2="106.68" y2="134.62" width="0.1524" layer="91"/>
+<wire x1="86.36" y1="134.62" x2="106.68" y2="134.62" width="0.1524" layer="91"/>
 <label x="99.06" y="134.62" size="1.778" layer="95"/>
-<pinref part="JUMPERCAN" gate="1" pin="2"/>
+<pinref part="JUMPER" gate="A" pin="2"/>
 </segment>
 </net>
@@
 <net name="N$9" class="0">
 <segment>
-<pinref part="JUMPERCAN" gate="1" pin="1"/>
 <pinref part="R5" gate="G$1" pin="2"/>
-<wire x1="88.9" y1="132.08" x2="91.44" y2="132.08" width="0.1524" layer="91"/>
-</segment>
-</net>
+<wire x1="86.36" y1="132.08" x2="91.44" y2="132.08" width="0.1524" layer="91"/>
+<pinref part="JUMPER" gate="A" pin="3"/>
+</segment>
+</net>

Commit message: nouvelles cartes à jour
Parts:
- added R2: 120, rcl:R-US_M0805
- COMMAND: value micromatch-8 -> MMATCH-6-; device con-amp-micromatch:MICROMATCH-8 -> jt-con-micromatch:MMATCH-6-
Connections:
- removed net TF1: COMMAND-8.S
- removed net TF2: COMMAND-5.S
- net +12V_DIRTY: now also R2.1
- net +5V: now also COMMAND.3; no longer COMMAND-1.S
- net DATA_AX12_DIRTY: now also R2.2
- net DIR1: now also COMMAND.5; no longer COMMAND-7.S
- net DIR2: now also COMMAND.7; no longer COMMAND-4.S
- net GND: now also COMMAND.4; no longer COMMAND-2.S
- net PWM_MOT1: now also COMMAND.6; no longer COMMAND-6.S
- net PWM_MOT2: now also COMMAND.8; no longer COMMAND-3.S
Changed lines of the file:
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@@
 <layer number="54" name="bGND_GNDA" color="1" fill="9" visible="no" active="no"/>
 <layer number="56" name="wert" color="7" fill="1" visible="no" active="no"/>
+<layer number="57" name="tCAD" color="7" fill="1" visible="no" active="no"/>
 <layer number="59" name="tCarbon" color="7" fill="1" visible="no" active="no"/>
 <layer number="60" name="bCarbon" color="7" fill="1" visible="no" active="no"/>
@@
 <layer number="125" name="_tNames" color="7" fill="1" visible="yes" active="yes"/>
 <layer number="126" name="_bNames" color="7" fill="1" visible="yes" active="yes"/>
+<layer number="127" name="_tValues" color="7" fill="1" visible="yes" active="yes"/>
+<layer number="128" name="_bValues" color="7" fill="1" visible="yes" active="yes"/>
 <layer number="129" name="Mask" color="7" fill="1" visible="yes" active="yes"/>
 <layer number="131" name="tAdjust" color="7" fill="1" visible="yes" active="yes"/>
 <layer number="132" name="bAdjust" color="7" fill="1" visible="yes" active="yes"/>
 <layer number="144" name="Drill_legend" color="7" fill="1" visible="yes" active="yes"/>
+<layer number="150" name="Notes" color="7" fill="1" visible="no" active="yes"/>
 <layer number="151" name="HeatSink" color="7" fill="1" visible="yes" active="yes"/>
+<layer number="152" name="_bDocu" color="7" fill="1" visible="yes" active="yes"/>
+<layer number="153" name="FabDoc1" color="6" fill="1" visible="no" active="no"/>
+<layer number="154" name="FabDoc2" color="2" fill="1" visible="no" active="no"/>
+<layer number="155" name="FabDoc3" color="7" fill="15" visible="no" active="no"/>
 <layer number="199" name="Contour" color="7" fill="1" visible="yes" active="yes"/>
 <layer number="200" name="200bmp" color="1" fill="10" visible="yes" active="yes"/>
@@
 <layer number="223" name="223bmp" color="24" fill="1" visible="no" active="no"/>
 <layer number="224" name="224bmp" color="25" fill="1" visible="no" active="no"/>
+<layer number="248" name="Housing" color="7" fill="1" visible="yes" active="yes"/>
+<layer number="249" name="Edge" color="7" fill="1" visible="yes" active="yes"/>
 <layer number="250" name="Descript" color="3" fill="1" visible="no" active="no"/>
 <layer number="251" name="SMDround" color="12" fill="11" visible="no" active="no"/>
@@
 <classes>
 <class number="0" name="default" width="0" drill="0">
+</class>
+<class number="1" name="+5V" width="0.6" drill="0.2">
+<clearance class="1" value="0.4"/>
 </class>
 </classes>
@@
 <part name="AX12-1" library="con-molex" deviceset="22-23-2031" device="" value="molex-3"/>
 <part name="AX12-2" library="con-molex" deviceset="22-23-2031" device="" value="molex-3"/>
-<part name="COMMAND" library="con-amp-micromatch" deviceset="MICROMATCH-8" device="" value="micromatch-8"/>
 <part name="ODO_G" library="con-lstb" deviceset="MA04-1" device="" value="header-4"/>
 <part name="ODO_D" library="con-lstb" deviceset="MA04-1" device="" value="header-4"/>
@@
 <part name="C2" library="mbed-rlcq" deviceset="C" device="0805" value="100u"/>
 <part name="JUMPER" library="pinhead" deviceset="PINHD-1X3" device=""/>
+<part name="R2" library="rcl" deviceset="R-US_" device="M0805" value="120"/>
+<part name="COMMAND" library="jt-con-micromatch" deviceset="MMATCH-6-*" device=""/>
+<part name="+5V" library="supply1" deviceset="VCC" device="" value="+5v"/>
+<part name="GND2" library="supply1" deviceset="GND" device=""/>
 </parts>
 <sheets>
@@
 <instance part="AX12-2" gate="-2" x="281.94" y="73.66"/>
 <instance part="AX12-2" gate="-3" x="281.94" y="71.12"/>
-<instance part="COMMAND" gate="-1" x="317.5" y="88.9"/>
-<instance part="COMMAND" gate="-2" x="317.5" y="86.36"/>
-<instance part="COMMAND" gate="-3" x="317.5" y="83.82"/>
-<instance part="COMMAND" gate="-4" x="317.5" y="81.28"/>
-<instance part="COMMAND" gate="-5" x="317.5" y="78.74"/>
-<instance part="COMMAND" gate="-6" x="317.5" y="76.2"/>
-<instance part="COMMAND" gate="-7" x="317.5" y="73.66"/>
-<instance part="COMMAND" gate="-8" x="317.5" y="71.12"/>
 <instance part="ODO_G" gate="1" x="190.5" y="38.1" rot="R180"/>
 <instance part="ODO_D" gate="1" x="190.5" y="17.78" rot="R180"/>
@@
 <instance part="C2" gate="G$1" x="256.54" y="99.06"/>
 <instance part="JUMPER" gate="A" x="83.82" y="134.62" rot="MR0"/>
+<instance part="R2" gate="G$1" x="254" y="78.74" rot="R270"/>
+<instance part="COMMAND" gate="G$1" x="330.2" y="87.63"/>
+<instance part="+5V" gate="VCC" x="318.77" y="77.47" rot="R180"/>
+<instance part="GND2" gate="1" x="340.36" y="77.47"/>
 </instances>
 <busses>
@@
 </segment>
 <segment>
-<pinref part="COMMAND" gate="-2" pin="S"/>
-<wire x1="322.58" y1="86.36" x2="330.2" y2="86.36" width="0.1524" layer="91"/>
-<label x="335.28" y="86.36" size="1.778" layer="95"/>
-</segment>
-<segment>
 <pinref part="ODO_G" gate="1" pin="4"/>
 <wire x1="182.88" y1="35.56" x2="177.8" y2="35.56" width="0.1524" layer="91"/>
@@
 <wire x1="208.28" y1="71.12" x2="200.66" y2="71.12" width="0.1524" layer="91"/>
 <label x="187.96" y="71.12" size="1.778" layer="95"/>
+</segment>
+<segment>
+<pinref part="COMMAND" gate="G$1" pin="4"/>
+<wire x1="335.28" y1="85.09" x2="340.36" y2="85.09" width="0.1524" layer="91"/>
+<wire x1="340.36" y1="85.09" x2="340.36" y2="80.01" width="0.1524" layer="91"/>
+<pinref part="GND2" gate="1" pin="GND"/>
 </segment>
 </net>
@@
 </segment>
 <segment>
-<pinref part="COMMAND" gate="-1" pin="S"/>
-<wire x1="322.58" y1="88.9" x2="330.2" y2="88.9" width="0.1524" layer="91"/>
-<label x="335.28" y="88.9" size="1.778" layer="95"/>
-</segment>
-<segment>
 <pinref part="ODO_G" gate="1" pin="1"/>
 <wire x1="182.88" y1="43.18" x2="177.8" y2="43.18" width="0.1524" layer="91"/>
@@
 <label x="137.16" y="68.58" size="1.778" layer="95"/>
 </segment>
+<segment>
+<pinref part="COMMAND" gate="G$1" pin="3"/>
+<wire x1="325.12" y1="85.09" x2="318.77" y2="85.09" width="0.1524" layer="91"/>
+<wire x1="318.77" y1="85.09" x2="318.77" y2="80.01" width="0.1524" layer="91"/>
+<pinref part="+5V" gate="VCC" pin="VCC"/>
+</segment>
 </net>
 <net name="CANL" class="0">
@@
 <label x="251.46" y="106.68" size="1.9304" layer="95"/>
 </segment>
+<segment>
+<pinref part="R2" gate="G$1" pin="1"/>
+<wire x1="254" y1="83.82" x2="254" y2="86.36" width="0.1524" layer="91"/>
+<label x="259.08" y="83.82" size="1.778" layer="95"/>
+</segment>
 </net>
 <net name="DATA_AX12" class="0">
@@
 <net name="PWM_MOT2" class="0">
 <segment>
-<pinref part="COMMAND" gate="-3" pin="S"/>
-<wire x1="322.58" y1="83.82" x2="330.2" y2="83.82" width="0.1524" layer="91"/>
-<label x="335.28" y="83.82" size="1.778" layer="95"/>
-</segment>
-<segment>
 <pinref part="MBED" gate="KIT" pin="P24"/>
 <wire x1="274.32" y1="137.16" x2="279.4" y2="137.16" width="0.1524" layer="91"/>
 <label x="279.4" y="137.16" size="1.778" layer="95"/>
 </segment>
+<segment>
+<pinref part="COMMAND" gate="G$1" pin="8"/>
+<wire x1="335.28" y1="90.17" x2="340.36" y2="90.17" width="0.1524" layer="91"/>
+<label x="340.36" y="90.17" size="1.778" layer="95"/>
+</segment>
 </net>
 <net name="DIR2" class="0">
-<segment>
-<pinref part="COMMAND" gate="-4" pin="S"/>
-<wire x1="322.58" y1="81.28" x2="330.2" y2="81.28" width="0.1524" layer="91"/>
-<label x="335.28" y="81.28" size="1.778" layer="95"/>
-</segment>
 <segment>
 <pinref part="MBED" gate="KIT" pin="P23"/>
@@
 <label x="279.4" y="134.62" size="1.778" layer="95"/>
 </segment>
-</net>
-<net name="TF2" class="0">
-<segment>
-<pinref part="COMMAND" gate="-5" pin="S"/>
-<wire x1="322.58" y1="78.74" x2="330.2" y2="78.74" width="0.1524" layer="91"/>
-<label x="335.28" y="78.74" size="1.778" layer="95"/>
+<segment>
+<pinref part="COMMAND" gate="G$1" pin="7"/>
+<wire x1="325.12" y1="90.17" x2="320.04" y2="90.17" width="0.1524" layer="91"/>
+<label x="320.04" y="90.17" size="1.778" layer="95" rot="R180"/>
 </segment>
 </net>
 <net name="PWM_MOT1" class="0">
-<segment>
-<pinref part="COMMAND" gate="-6" pin="S"/>
-<wire x1="322.58" y1="76.2" x2="330.2" y2="76.2" width="0.1524" layer="91"/>
-<label x="335.28" y="76.2" size="1.778" layer="95"/>
-</segment>
 <segment>
 <pinref part="MBED" gate="KIT" pin="P22"/>
@@
 <label x="279.4" y="132.08" size="1.778" layer="95"/>
 </segment>
+<segment>
+<pinref part="COMMAND" gate="G$1" pin="6"/>
+<wire x1="335.28" y1="87.63" x2="340.36" y2="87.63" width="0.1524" layer="91"/>
+<label x="340.36" y="87.63" size="1.778" layer="95"/>
+</segment>
 </net>
 <net name="DIR1" class="0">
-<segment>
-<pinref part="COMMAND" gate="-7" pin="S"/>
-<wire x1="322.58" y1="73.66" x2="330.2" y2="73.66" width="0.1524" layer="91"/>
-<label x="335.28" y="73.66" size="1.778" layer="95"/>
-</segment>
 <segment>
 <pinref part="MBED" gate="KIT" pin="P21"/>
@@
 <label x="279.4" y="129.54" size="1.778" layer="95"/>
 </segment>
-</net>
-<net name="TF1" class="0">
-<segment>
-<pinref part="COMMAND" gate="-8" pin="S"/>
-<wire x1="322.58" y1="71.12" x2="330.2" y2="71.12" width="0.1524" layer="91"/>
-<label x="335.28" y="71.12" size="1.778" layer="95"/>
+<segment>
+<pinref part="COMMAND" gate="G$1" pin="5"/>
+<wire x1="325.12" y1="87.63" x2="320.04" y2="87.63" width="0.1524" layer="91"/>
+<label x="320.04" y="87.63" size="1.778" layer="95" rot="R180"/>
 </segment>
 </net>
@@
 <label x="259.08" y="86.36" size="1.778" layer="95"/>
 </segment>
-</net>
+<segment>
+<pinref part="R2" gate="G$1" pin="2"/>
+<wire x1="254" y1="73.66" x2="254" y2="68.58" width="0.1524" layer="91"/>
+<label x="251.46" y="63.5" size="1.778" layer="95"/>
+</segment>
+</net>
