File: cartes/Carte_IA_cédric/bb2.brd (EAGLE design)
At the start: 100 x 80 mm, 29 parts, among them IC1 MIC5219BM5

Commit message: nouvelles cartes à jour
Other:
- board size 100 x 80 mm -> 86.5 x 54.5 mm
Changed lines of the file:
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@@
 <setting verticaltext="up"/>
 </settings>
-<grid distance="0.1" unitdist="mm" unit="mm" style="lines" multiple="1" display="no" altdistance="0.025" altunitdist="inch" altunit="inch"/>
+<grid distance="0.5" unitdist="mm" unit="mm" style="lines" multiple="1" display="no" altdistance="0.025" altunitdist="inch" altunit="inch"/>
 <layers>
 <layer number="1" name="Top" color="4" fill="1" visible="yes" active="yes"/>
@@
 <board>
 <plain>
-<wire x1="0" y1="0" x2="100" y2="0" width="0" layer="20"/>
-<wire x1="100" y1="0" x2="100" y2="80" width="0" layer="20"/>
-<wire x1="100" y1="80" x2="0" y2="80" width="0" layer="20"/>
-<wire x1="0" y1="80" x2="0" y2="0" width="0" layer="20"/>
+<wire x1="0" y1="25.5" x2="86.5" y2="25.5" width="0" layer="20"/>
+<wire x1="86.5" y1="25.5" x2="86.5" y2="80" width="0" layer="20"/>
+<wire x1="86.5" y1="80" x2="0" y2="80" width="0" layer="20"/>
+<wire x1="0" y1="80" x2="0" y2="25.5" width="0" layer="20"/>
 <text x="82.65" y="32.57" size="1.778" layer="21" rot="R90">ARES 2014</text>
 <text x="78.17" y="31.95" size="5.08" layer="21" rot="R90">IA</text>
