File: cartes/Carte_bouton/carte_bouton.sch (EAGLE design)
At the start: 8 parts, among them X1 22-23-2021

Commit message: plein de trucs
Parts:
- renumbered S1 to COULEUR, U$3 to CARTE_IA
Changed lines of the file:
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@@
 <?xml version="1.0" encoding="utf-8"?>
 <!DOCTYPE eagle SYSTEM "eagle.dtd">
-<eagle version="6.4">
+<eagle version="6.5.0">
 <drawing>
 <settings>
@@
 <setting verticaltext="up"/>
 </settings>
-<grid distance="0.025" unitdist="inch" unit="inch" style="lines" multiple="1" display="no" altdistance="0.01" altunitdist="inch" altunit="inch"/>
+<grid distance="0.1" unitdist="inch" unit="inch" style="lines" multiple="1" display="no" altdistance="0.01" altunitdist="inch" altunit="inch"/>
 <layers>
 <layer number="1" name="Top" color="4" fill="1" visible="no" active="no"/>
@@
 </classes>
 <parts>
-<part name="U$3" library="jt-con-micromatch" deviceset="MMATCH-4-*" device=""/>
+<part name="CARTE_IA" library="jt-con-micromatch" deviceset="MMATCH-4-*" device=""/>
 <part name="+3V2" library="supply1" deviceset="+3V3" device=""/>
 <part name="GND9" library="supply1" deviceset="GND" device=""/>
 <part name="X1" library="con-molex" deviceset="22-23-2021" device=""/>
 <part name="+3V1" library="supply1" deviceset="+3V3" device=""/>
-<part name="S1" library="switch" deviceset="320-916" device=""/>
+<part name="COULEUR" library="switch" deviceset="320-916" device=""/>
 <part name="+3V3" library="supply1" deviceset="+3V3" device=""/>
 <part name="GND1" library="supply1" deviceset="GND" device=""/>
@@
 </plain>
 <instances>
-<instance part="U$3" gate="G$1" x="19.05" y="29.21"/>
+<instance part="CARTE_IA" gate="G$1" x="19.05" y="29.21"/>
 <instance part="+3V2" gate="G$1" x="9.525" y="36.195"/>
 <instance part="GND9" gate="1" x="9.525" y="24.765"/>
@@
 <instance part="X1" gate="-2" x="71.755" y="34.29" rot="R90"/>
 <instance part="+3V1" gate="G$1" x="78.105" y="34.925"/>
-<instance part="S1" gate="1" x="40.005" y="50.165"/>
+<instance part="COULEUR" gate="1" x="40.005" y="50.165"/>
 <instance part="+3V3" gate="G$1" x="45.085" y="73.66"/>
 <instance part="GND1" gate="1" x="40.005" y="75.565" rot="R180"/>
@@
 <net name="GND" class="0">
 <segment>
-<pinref part="U$3" gate="G$1" pin="5"/>
+<pinref part="CARTE_IA" gate="G$1" pin="5"/>
 <wire x1="13.97" y1="29.21" x2="9.525" y2="29.21" width="0.1524" layer="91"/>
 <wire x1="9.525" y1="29.21" x2="9.525" y2="27.305" width="0.1524" layer="91"/>
@@
 </segment>
 <segment>
-<pinref part="S1" gate="1" pin="O"/>
+<pinref part="COULEUR" gate="1" pin="O"/>
 <wire x1="40.005" y1="55.245" x2="40.005" y2="66.675" width="0.1524" layer="91"/>
 <pinref part="GND1" gate="1" pin="GND"/>
@@
 <net name="+3V3" class="0">
 <segment>
-<pinref part="U$3" gate="G$1" pin="7"/>
+<pinref part="CARTE_IA" gate="G$1" pin="7"/>
 <wire x1="13.97" y1="31.75" x2="9.525" y2="31.75" width="0.1524" layer="91"/>
 <wire x1="9.525" y1="31.75" x2="9.525" y2="33.655" width="0.1524" layer="91"/>
@@
 </segment>
 <segment>
-<pinref part="S1" gate="1" pin="S"/>
+<pinref part="COULEUR" gate="1" pin="S"/>
 <wire x1="45.085" y1="55.245" x2="45.085" y2="66.675" width="0.1524" layer="91"/>
 <pinref part="+3V3" gate="G$1" pin="+3V3"/>
@@
 <net name="TIRETTE" class="0">
 <segment>
-<pinref part="U$3" gate="G$1" pin="6"/>
+<pinref part="CARTE_IA" gate="G$1" pin="6"/>
 <pinref part="X1" gate="-1" pin="S"/>
 <wire x1="24.13" y1="29.21" x2="43.18" y2="29.21" width="0.1524" layer="91"/>
@@
 <net name="N$1" class="0">
 <segment>
-<pinref part="U$3" gate="G$1" pin="8"/>
-<pinref part="S1" gate="1" pin="P"/>
+<pinref part="CARTE_IA" gate="G$1" pin="8"/>
+<pinref part="COULEUR" gate="1" pin="P"/>
 <wire x1="24.13" y1="31.75" x2="27.94" y2="31.75" width="0.1524" layer="91"/>
 <wire x1="27.94" y1="31.75" x2="42.545" y2="31.75" width="0.1524" layer="91"/>

Commit message: nouvelles cartes à jour
Parts:
- renumbered X1 to TIRETTE
Changed lines of the file:
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@@
 <part name="+3V2" library="supply1" deviceset="+3V3" device=""/>
 <part name="GND9" library="supply1" deviceset="GND" device=""/>
-<part name="X1" library="con-molex" deviceset="22-23-2021" device=""/>
+<part name="TIRETTE" library="con-molex" deviceset="22-23-2021" device=""/>
 <part name="+3V1" library="supply1" deviceset="+3V3" device=""/>
 <part name="COULEUR" library="switch" deviceset="320-916" device=""/>
@@
 <instance part="+3V2" gate="G$1" x="9.525" y="36.195"/>
 <instance part="GND9" gate="1" x="9.525" y="24.765"/>
-<instance part="X1" gate="-1" x="68.58" y="34.29" rot="R90"/>
-<instance part="X1" gate="-2" x="71.755" y="34.29" rot="R90"/>
+<instance part="TIRETTE" gate="-1" x="68.58" y="34.29" rot="R90"/>
+<instance part="TIRETTE" gate="-2" x="71.755" y="34.29" rot="R90"/>
 <instance part="+3V1" gate="G$1" x="78.105" y="34.925"/>
 <instance part="COULEUR" gate="1" x="40.005" y="50.165"/>
@@
 </segment>
 <segment>
-<pinref part="X1" gate="-2" pin="S"/>
+<pinref part="TIRETTE" gate="-2" pin="S"/>
 <wire x1="71.755" y1="31.75" x2="71.755" y2="29.21" width="0.1524" layer="91"/>
 <wire x1="71.755" y1="29.21" x2="78.105" y2="29.21" width="0.1524" layer="91"/>
@@
 <segment>
 <pinref part="CARTE_IA" gate="G$1" pin="6"/>
-<pinref part="X1" gate="-1" pin="S"/>
+<pinref part="TIRETTE" gate="-1" pin="S"/>
 <wire x1="24.13" y1="29.21" x2="43.18" y2="29.21" width="0.1524" layer="91"/>
 <wire x1="43.18" y1="29.21" x2="68.58" y2="29.21" width="0.1524" layer="91"/>
