File: cartes/Carte_bouton/cartev1/carte_bouton.brd (EAGLE design)
At the start: 30 x 33.3 mm, 12 parts

Commit message: carte bouton v2
Parts:
- removed ALIM: (no value), led:SML0805
- removed CARTE_ALIM: (no value), SparkFun-Connectors:MOLEX-1X3
- removed ON/OFF: (no value), switch:320-916
- removed R4: 1k, rcl:M0805
- moved R1 18.9 mm to (21.4, 4.69)
- moved CARTE_IA 18.4 mm to (12.9, 6.52), turned to 180 degrees
- moved JAUNE 12.2 mm to (3.80, 14.6)
- moved COULEUR 12.2 mm to (15.1, 14.8)
- moved R2 12.2 mm to (26.3, 20.0)
- moved R3 12.2 mm to (3.80, 20.6)
- moved ROUGE 12.2 mm to (26.4, 14.6)
- moved TIRETTE 12.2 mm to (15.2, 22.6)
Connections:
- removed net 5V: CARTE_ALIM.3, ON/OFF.3
- removed net DATA_SWITCH: ALIM.C, CARTE_ALIM.2, ON/OFF.2
- removed net GND_DIRTY: CARTE_ALIM.1, ON/OFF.1, R4.1
- removed net N$9: ALIM.A, R4.2
Routing:
- net GND_DIRTY: track 68.8 -> 0.00 mm, vias 2 -> 0
- net +3V3: track 76.6 -> 38.9 mm, vias 1 -> 0
- net 5V: track 27.3 -> 0.00 mm, vias 1 -> 0
- net DATA_SWITCH: track 27.0 -> 0.00 mm
- net TIRETTE: track 63.6 -> 39.9 mm, vias 1 -> 0
- net N$1: track 58.4 -> 41.1 mm
- net GND: track 0.00 -> 9.96 mm
- net N$9: track 3.08 -> 0.00 mm
- net N$2: track 5.16 -> 3.47 mm
Other:
- board size 30 x 33.3 mm -> 30 x 30 mm
