File: cartes/Carte_bouton/cartev1/carte_bouton.sch (EAGLE design)
At the start: 12 parts

Commit message: carte bouton v2
Parts:
- removed ALIM: (no value), led:LEDSML0805
- removed CARTE_ALIM: (no value), SparkFun-Connectors:M03POLAR
- removed ON/OFF: (no value), switch:320-916
- removed R4: 1k, rcl:R-US_M0805
Connections:
- removed net 5V: CARTE_ALIM.3, ON/OFF.S
- removed net DATA_SWITCH: ALIM.C, CARTE_ALIM.2, ON/OFF.P
- removed net GND_DIRTY: CARTE_ALIM.1, ON/OFF.O, R4.1
- removed net N$9: ALIM.A, R4.2
Changed lines of the file:
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@@
 <layer number="106" name="bPlate" color="7" fill="1" visible="no" active="yes"/>
 <layer number="107" name="Crop" color="7" fill="1" visible="no" active="yes"/>
-<layer number="108" name="tplace-old" color="10" fill="1" visible="yes" active="yes"/>
-<layer number="109" name="ref-old" color="11" fill="1" visible="yes" active="yes"/>
 <layer number="116" name="Patch_BOT" color="9" fill="4" visible="no" active="yes"/>
 <layer number="121" name="_tsilk" color="7" fill="1" visible="no" active="yes"/>
@@
 <layer number="144" name="Drill_legend" color="7" fill="1" visible="no" active="yes"/>
 <layer number="151" name="HeatSink" color="7" fill="1" visible="no" active="yes"/>
-<layer number="199" name="Contour" color="7" fill="1" visible="yes" active="yes"/>
 <layer number="200" name="200bmp" color="1" fill="10" visible="no" active="yes"/>
 <layer number="201" name="201bmp" color="2" fill="10" visible="no" active="yes"/>
@@
 <part name="JAUNE" library="led" deviceset="LED" device="SML0805"/>
 <part name="R3" library="rcl" deviceset="R-US_" device="M0805" value="1k"/>
-<part name="CARTE_ALIM" library="SparkFun-Connectors" deviceset="M03" device="POLAR"/>
-<part name="ON/OFF" library="switch" deviceset="320-916" device=""/>
-<part name="R4" library="rcl" deviceset="R-US_" device="M0805" value="1k"/>
-<part name="ALIM" library="led" deviceset="LED" device="SML0805"/>
 </parts>
 <sheets>
@@
 <instance part="JAUNE" gate="G$1" x="56.515" y="45.72"/>
 <instance part="R3" gate="G$1" x="56.515" y="57.785" rot="R90"/>
-<instance part="CARTE_ALIM" gate="G$1" x="-20.32" y="63.5"/>
-<instance part="ON/OFF" gate="1" x="7.62" y="66.04" rot="R270"/>
-<instance part="R4" gate="G$1" x="-2.54" y="48.26" rot="R180"/>
-<instance part="ALIM" gate="G$1" x="-14.605" y="48.26" rot="R270"/>
 </instances>
 <busses>
@@
 </segment>
 </net>
-<net name="GND_DIRTY" class="0">
-<segment>
-<pinref part="CARTE_ALIM" gate="G$1" pin="1"/>
-<wire x1="-12.7" y1="60.96" x2="-5.08" y2="60.96" width="0.1524" layer="91"/>
-<wire x1="-5.08" y1="60.96" x2="-5.08" y2="76.2" width="0.1524" layer="91"/>
-<wire x1="-5.08" y1="76.2" x2="15.24" y2="76.2" width="0.1524" layer="91"/>
-<wire x1="15.24" y1="76.2" x2="15.24" y2="66.04" width="0.1524" layer="91"/>
-<pinref part="ON/OFF" gate="1" pin="O"/>
-<wire x1="15.24" y1="66.04" x2="12.7" y2="66.04" width="0.1524" layer="91"/>
-<label x="0" y="60.96" size="1.778" layer="95" rot="R180"/>
-</segment>
-<segment>
-<wire x1="11.43" y1="48.26" x2="2.54" y2="48.26" width="0.1524" layer="91"/>
-<pinref part="R4" gate="G$1" pin="1"/>
-<label x="17.78" y="50.8" size="1.778" layer="95" rot="R180"/>
-</segment>
-</net>
-<net name="DATA_SWITCH" class="0">
-<segment>
-<pinref part="CARTE_ALIM" gate="G$1" pin="2"/>
-<wire x1="-12.7" y1="63.5" x2="2.54" y2="63.5" width="0.1524" layer="91"/>
-<pinref part="ON/OFF" gate="1" pin="P"/>
-<label x="2.54" y="63.5" size="1.778" layer="95" rot="R180"/>
-</segment>
-<segment>
-<pinref part="ALIM" gate="G$1" pin="C"/>
-<wire x1="-19.685" y1="48.26" x2="-23.495" y2="48.26" width="0.1524" layer="91"/>
-<label x="-20.32" y="50.8" size="1.778" layer="95" rot="R180"/>
-</segment>
-</net>
-<net name="5V" class="0">
-<segment>
-<pinref part="CARTE_ALIM" gate="G$1" pin="3"/>
-<wire x1="-12.7" y1="66.04" x2="0" y2="66.04" width="0.1524" layer="91"/>
-<wire x1="0" y1="66.04" x2="0" y2="58.42" width="0.1524" layer="91"/>
-<pinref part="ON/OFF" gate="1" pin="S"/>
-<wire x1="0" y1="58.42" x2="12.7" y2="58.42" width="0.1524" layer="91"/>
-<wire x1="12.7" y1="58.42" x2="12.7" y2="60.96" width="0.1524" layer="91"/>
-<label x="-10.16" y="66.04" size="1.778" layer="95" rot="R180"/>
-</segment>
-</net>
-<net name="N$9" class="0">
-<segment>
-<pinref part="R4" gate="G$1" pin="2"/>
-<pinref part="ALIM" gate="G$1" pin="A"/>
-<wire x1="-12.065" y1="48.26" x2="-7.62" y2="48.26" width="0.1524" layer="91"/>
-</segment>
-</net>
