File: cartes/Envoyé à dipole/Carte_puissance/schema_puissance.sch (EAGLE design)
At the start: 22 parts, among them X2 GMSTBA2

Commit message: ajout gerber puissance + export wiki
Parts:
- added IN: SL-3.5-2-90G, WEIDMULLER:SL-3.5-2-90G
Connections:
- net +12V: now also IN.2
- net GNDA: now also IN.1
Changed lines of the file:
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@@
 <part name="P+3" library="supply1" deviceset="VCC" device=""/>
 <part name="GND2" library="supply1" deviceset="GND" device=""/>
+<part name="IN" library="WEIDMULLER" deviceset="SL-3.5-2-90G" device=""/>
+<part name="P+4" library="supply1" deviceset="+12V" device=""/>
+<part name="GND5" library="supply1" deviceset="GNDA" device=""/>
 </parts>
 <sheets>
@@
 <instance part="P+3" gate="VCC" x="-161.29" y="-85.09" rot="R180"/>
 <instance part="GND2" gate="1" x="-139.7" y="-85.09"/>
+<instance part="IN" gate="G$1" x="-172.72" y="43.18"/>
+<instance part="P+4" gate="1" x="-160.02" y="50.8"/>
+<instance part="GND5" gate="1" x="-160.02" y="30.48"/>
 </instances>
 <busses>
@@
 <junction x="-64.135" y="-27.305"/>
 </segment>
+<segment>
+<pinref part="IN" gate="G$1" pin="1"/>
+<wire x1="-167.64" y1="40.64" x2="-160.02" y2="40.64" width="0.1524" layer="91"/>
+<pinref part="GND5" gate="1" pin="GNDA"/>
+<wire x1="-160.02" y1="33.02" x2="-160.02" y2="40.64" width="0.1524" layer="91"/>
+</segment>
 </net>
 <net name="+12V" class="0">
@@
 <pinref part="P+15" gate="1" pin="+12V"/>
 </segment>
-</net>
+<segment>
+<pinref part="IN" gate="G$1" pin="2"/>
+<wire x1="-167.64" y1="45.72" x2="-160.02" y2="45.72" width="0.1524" layer="91"/>
+<wire x1="-160.02" y1="45.72" x2="-160.02" y2="48.26" width="0.1524" layer="91"/>
+<pinref part="P+4" gate="1" pin="+12V"/>
+</segment>
+</net>
