File: cartes/En dev/Carte asserv/board.brd (EAGLE design)
At the start: 73.3 x 66 mm, 21 parts

Commit message: nouveaux gerber
Routing:
- net +5V: track 250.5 -> 247.8 mm
- net GND: track 0.00 -> 1.79 mm, vias 0 -> 3
- net VDD_3V3: track 58.4 -> 59.1 mm
Changed lines of the file:
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@@
 <contactref element="R11" pad="1"/>
 <contactref element="COULEUR" pad="1"/>
-<polygon width="0.4064" layer="16">
+<polygon width="0.4064" layer="16" isolate="0.3048">
 <vertex x="0" y="66.04"/>
 <vertex x="73.66" y="66.04"/>
@@
 <vertex x="0" y="0"/>
 </polygon>
-<polygon width="0.4064" layer="1">
+<polygon width="0.4064" layer="1" isolate="0.3048">
 <vertex x="0" y="66.04"/>
 <vertex x="73.66" y="66.04"/>
@@
 </polygon>
 <contactref element="PWM" pad="2"/>
+<via x="31.26" y="37.4" extent="1-16" drill="0.4"/>
+<via x="37.87" y="23.27" extent="1-16" drill="0.4"/>
+<wire x1="13.97" y1="30.48" x2="14.81" y2="29.64" width="0.4064" layer="16"/>
+<wire x1="14.81" y1="29.64" x2="14.81" y2="29.04" width="0.4064" layer="16"/>
+<via x="10.63" y="33.18" extent="1-16" drill="0.4"/>
+<wire x1="57.15" y1="33.02" x2="68.58" y2="33.02" width="0" layer="19" extent="1-1"/>
 </signal>
 <signal name="+5V" class="1">
@@
 <wire x1="62.6" y1="30.4" x2="62.5" y2="30.2" width="0.6" layer="1"/>
 <wire x1="5.2" y1="38.1" x2="6.35" y2="38.1" width="0.6" layer="1"/>
-<wire x1="1.22" y1="42.17" x2="5.2" y2="38.1" width="0.6" layer="1"/>
-<wire x1="1.2" y1="45.6" x2="1.22" y2="42.17" width="0.6" layer="1"/>
-<wire x1="6.4" y1="50.8" x2="1.2" y2="45.6" width="0.6" layer="1"/>
+<wire x1="6.4" y1="50.8" x2="2.742803125" y2="47.142803125" width="0.6" layer="1"/>
+<wire x1="2.742803125" y1="47.142803125" x2="2.706509375" y2="40.649875" width="0.6" layer="1"/>
+<wire x1="2.706509375" y1="40.649875" x2="5.2" y2="38.1" width="0.6" layer="1"/>
 <wire x1="6.4" y1="50.8" x2="6.35" y2="50.8" width="0.6" layer="1"/>
 <wire x1="25.6" y1="30.4" x2="28" y2="30.4" width="0.6" layer="16"/>
@@
 <wire x1="7.7" y1="59.9" x2="12.7" y2="54.9" width="0.6" layer="16"/>
 <wire x1="4.9" y1="59.9" x2="7.7" y2="59.9" width="0.6" layer="16"/>
-<wire x1="0.9" y1="55.9" x2="4.9" y2="59.9" width="0.6" layer="16"/>
-<wire x1="5" y1="51.8" x2="0.9" y2="55.9" width="0.6" layer="16"/>
+<wire x1="5" y1="51.8" x2="2.631184375" y2="54.168815625" width="0.6" layer="16"/>
+<wire x1="2.631184375" y1="54.168815625" x2="2.631184375" y2="57.631184375" width="0.6" layer="16"/>
+<wire x1="2.631184375" y1="57.631184375" x2="4.9" y2="59.9" width="0.6" layer="16"/>
 <wire x1="5.3" y1="51.8" x2="5" y2="51.8" width="0.6" layer="16"/>
 <wire x1="6.3" y1="50.8" x2="5.3" y2="51.8" width="0.6" layer="16"/>
@@
 <wire x1="11.2" y1="29.2" x2="6.4" y2="29.2" width="0.2" layer="1"/>
 <wire x1="12.6" y1="27.8" x2="11.2" y2="29.2" width="0.2" layer="1"/>
-<wire x1="15.4" y1="27.8" x2="12.6" y2="27.8" width="0.2" layer="1"/>
-<wire x1="15.5" y1="27.9" x2="15.4" y2="27.8" width="0.2" layer="1"/>
-<wire x1="20.2" y1="27.9" x2="15.5" y2="27.9" width="0.2" layer="16"/>
+<wire x1="15.11" y1="27.8" x2="12.6" y2="27.8" width="0.2" layer="1"/>
+<wire x1="15.97" y1="28.7" x2="15.11" y2="27.8" width="0.2" layer="1"/>
+<wire x1="20.2" y1="27.9" x2="16.75" y2="27.9" width="0.2" layer="16"/>
+<wire x1="16.75" y1="27.9" x2="15.97" y2="28.68" width="0.2" layer="16"/>
+<wire x1="15.97" y1="28.68" x2="15.97" y2="28.7" width="0.2" layer="16"/>
 <wire x1="26.9" y1="34.6" x2="20.2" y2="27.9" width="0.2" layer="16"/>
 <wire x1="53.6" y1="34.6" x2="26.9" y2="34.6" width="0.2" layer="16"/>
@@
 <wire x1="6.4" y1="29.2" x2="6.35" y2="29.21" width="0.2" layer="1"/>
 <wire x1="59.6" y1="30.5" x2="59.69" y2="30.48" width="0.2" layer="16"/>
-<via x="15.5" y="27.9" extent="1-16" drill="0.3"/>
+<via x="15.97" y="28.7" extent="1-16" drill="0.3"/>
 </signal>
 <signal name="TIRETTE">
