File: cartes/En dev/Carte plan B/board.brd (EAGLE design)
At the start: 49.9 x 73 mm, 21 parts

Commit message: nouveaux gerber
Parts:
- added R3, R4, R6, R7: 2,7k, rcl:R0805
Connections:
- net +5V: now also R3.2, R4.2, R6.2, R7.2
- net CHA_D: now also R6.1
- net CHA_G: now also R3.1
- net CHB_D: now also R7.1
- net CHB_G: now also R4.1
Routing:
- net CHA_G: track 16.2 -> 41.4 mm, vias 0 -> 1
- net +5V: track 229.7 -> 250.7 mm
- net CHB_G: track 16.2 -> 27.4 mm
- net CHB_D: track 52.1 -> 60.4 mm
- net CHA_D: track 43.2 -> 47.8 mm
Changed lines of the file:
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@@
 <element name="R2" library="rcl" package="M0805" value="120" x="6.16" y="6.97" rot="R270"/>
 <element name="COMMAND" library="jt-con-micromatch" package="AMP-215079-6" value="MMATCH-6-" x="34.28" y="3.1"/>
+<element name="R3" library="rcl" package="R0805" value="2,7k" x="37.01" y="39.55" rot="MR0"/>
+<element name="R4" library="rcl" package="R0805" value="2,7k" x="46.91" y="29.02" rot="MR0"/>
+<element name="R6" library="rcl" package="R0805" value="2,7k" x="36.22" y="51.09" rot="MR180"/>
+<element name="R7" library="rcl" package="R0805" value="2,7k" x="45.17" y="58.1" rot="MR0"/>
 </elements>
 <signals>
@@
 <wire x1="45.2" y1="47.5" x2="46.4" y2="47.5" width="0.4" layer="16"/>
 <wire x1="41.8" y1="50.9" x2="45.2" y2="47.5" width="0.4" layer="16"/>
-<wire x1="41.8" y1="63.7" x2="41.8" y2="50.9" width="0.4" layer="16"/>
+<wire x1="41.8" y1="63.7" x2="41.8" y2="60.51" width="0.4" layer="16"/>
+<wire x1="41.8" y1="60.51" x2="41.8" y2="51" width="0.4" layer="16"/>
+<wire x1="41.8" y1="51" x2="41.8" y2="50.9" width="0.4" layer="16"/>
 <wire x1="39.1" y1="66.4" x2="41.8" y2="63.7" width="0.4" layer="16"/>
 <wire x1="46.4" y1="47.5" x2="46.42" y2="47.45" width="0.4" layer="16"/>
@@
 <wire x1="2.6" y1="25.3" x2="2.54" y2="25.385" width="0.4" layer="1"/>
 <wire x1="34.2" y1="3.1" x2="34.28" y2="3.1" width="0.4" layer="1"/>
+<contactref element="R3" pad="2"/>
+<contactref element="R4" pad="2"/>
+<contactref element="R6" pad="2"/>
+<contactref element="R7" pad="2"/>
+<wire x1="36.06" y1="39.55" x2="35.71" y2="39.55" width="0.4064" layer="16"/>
+<wire x1="35.71" y1="39.55" x2="35.71" y2="42.35" width="0.4064" layer="16"/>
+<wire x1="35.71" y1="42.35" x2="34.71" y2="43.35" width="0.4064" layer="16"/>
+<wire x1="34.71" y1="43.35" x2="32.89" y2="43.35" width="0.4064" layer="16"/>
+<wire x1="32.89" y1="43.35" x2="31.59" y2="42.05" width="0.4064" layer="16"/>
+<wire x1="45.96" y1="29.02" x2="46.42" y2="29.48" width="0.4064" layer="16"/>
+<wire x1="46.42" y1="29.48" x2="46.42" y2="32.75" width="0.4064" layer="16"/>
+<wire x1="44.22" y1="58.1" x2="41.81" y2="60.51" width="0.4064" layer="16"/>
+<wire x1="41.81" y1="60.51" x2="41.8" y2="60.51" width="0.4064" layer="16"/>
+<wire x1="37.17" y1="51.09" x2="37.26" y2="51" width="0.4064" layer="16"/>
+<wire x1="37.26" y1="51" x2="38.36" y2="51.92" width="0.4064" layer="16"/>
+<wire x1="38.36" y1="51.92" x2="40.87" y2="51.92" width="0.4064" layer="16"/>
+<wire x1="40.87" y1="51.92" x2="41.52" y2="51.29" width="0.4064" layer="16"/>
+<wire x1="41.52" y1="51.29" x2="41.8" y2="51" width="0.4064" layer="16"/>
 </signal>
 <signal name="CANL">
@@
 <wire x1="39.1" y1="30.3" x2="39.8" y2="30.3" width="0.4" layer="16"/>
 <wire x1="34.5" y1="34.9" x2="39.1" y2="30.3" width="0.4" layer="16"/>
-<wire x1="34.5" y1="45.7" x2="34.5" y2="34.9" width="0.4" layer="16"/>
-<wire x1="18.7" y1="61.5" x2="34.5" y2="45.7" width="0.4" layer="1"/>
+<wire x1="34.5" y1="41.47" x2="34.5" y2="34.9" width="0.4" layer="16"/>
+<wire x1="18.7" y1="61.5" x2="32.92" y2="47.13" width="0.4" layer="1"/>
+<wire x1="32.92" y1="47.13" x2="34.5" y2="45.55" width="0.4" layer="1"/>
+<wire x1="34.5" y1="45.55" x2="34.5" y2="41.47" width="0.4" layer="1"/>
 <wire x1="17.6" y1="62.6" x2="18.7" y2="61.5" width="0.4" layer="16"/>
 <wire x1="14.3" y1="62.6" x2="17.6" y2="62.6" width="0.4" layer="16"/>
@@
 <wire x1="39.8" y1="30.3" x2="39.8" y2="30.29" width="0.4" layer="16"/>
 <wire x1="3.9" y1="53.3" x2="3.81" y2="53.23" width="0.4" layer="16"/>
-<via x="34.5" y="45.7" extent="1-16" drill="0.4"/>
+<via x="34.5" y="41.47" extent="1-16" drill="0.4"/>
 <via x="18.7" y="61.5" extent="1-16" drill="0.4"/>
 </signal>
@@
 <wire x1="39.8" y1="22.7" x2="39.8" y2="22.67" width="0.4" layer="16"/>
 <wire x1="46.4" y1="35.2" x2="46.42" y2="35.29" width="0.4" layer="16"/>
+<contactref element="R3" pad="1"/>
+<wire x1="37.96" y1="39.55" x2="38.94" y2="39.55" width="0.4064" layer="16"/>
+<wire x1="38.94" y1="39.55" x2="39.21" y2="39.28" width="0.4064" layer="16"/>
+<wire x1="39.21" y1="39.28" x2="42.04" y2="39.28" width="0.4064" layer="16"/>
+<wire x1="42.04" y1="39.28" x2="42.53" y2="38.79" width="0.4064" layer="16"/>
+<via x="42.53" y="38.79" extent="1-16" drill="0.4"/>
+<wire x1="42.53" y1="38.79" x2="42.5" y2="31.96" width="0.4064" layer="1"/>
+<wire x1="42.5" y1="31.96" x2="45.13" y2="29.43" width="0.4064" layer="1"/>
+<wire x1="45.13" y1="29.43" x2="47.51" y2="29.43" width="0.4064" layer="1"/>
+<wire x1="47.51" y1="29.43" x2="49.02" y2="31.08" width="0.4064" layer="1"/>
+<wire x1="49.02" y1="31.08" x2="49.02" y2="32.69" width="0.4064" layer="1"/>
+<wire x1="49.02" y1="32.69" x2="46.42" y2="35.29" width="0.4064" layer="1"/>
 </signal>
 <signal name="CHB_G">
@@
 <wire x1="39.8" y1="25.3" x2="39.8" y2="25.21" width="0.4" layer="16"/>
 <wire x1="46.4" y1="37.8" x2="46.42" y2="37.83" width="0.4" layer="16"/>
+<contactref element="R4" pad="1"/>
+<wire x1="47.86" y1="29.02" x2="49.17" y2="30.33" width="0.4064" layer="16"/>
+<wire x1="49.17" y1="30.33" x2="49.17" y2="36.39" width="0.4064" layer="16"/>
+<wire x1="49.17" y1="36.39" x2="47.73" y2="37.83" width="0.4064" layer="16"/>
+<wire x1="47.73" y1="37.83" x2="46.42" y2="37.83" width="0.4064" layer="16"/>
 </signal>
 <signal name="CHA_D">
@@
 <wire x1="28.7" y1="42.5" x2="28.7" y2="36.6" width="0.4" layer="16"/>
 <wire x1="33" y1="46.8" x2="28.7" y2="42.5" width="0.4" layer="16"/>
-<wire x1="40.7" y1="46.8" x2="33" y2="46.8" width="0.4" layer="16"/>
+<wire x1="40.7" y1="46.8" x2="34.52" y2="46.8" width="0.4" layer="16"/>
+<wire x1="34.52" y1="46.8" x2="33" y2="46.8" width="0.4" layer="16"/>
 <wire x1="43.9" y1="50" x2="40.7" y2="46.8" width="0.4" layer="1"/>
 <wire x1="46.4" y1="50" x2="43.9" y2="50" width="0.4" layer="1"/>
@@
 <wire x1="46.4" y1="50" x2="46.42" y2="49.99" width="0.4" layer="1"/>
 <via x="40.7" y="46.8" extent="1-16" drill="0.4"/>
+<contactref element="R6" pad="1"/>
+<wire x1="35.27" y1="51.09" x2="34.52" y2="50.34" width="0.4064" layer="16"/>
+<wire x1="34.52" y1="50.34" x2="34.52" y2="46.8" width="0.4064" layer="16"/>
 </signal>
 <signal name="CHB_D">
@@
 <wire x1="46.5" y1="52.5" x2="46.42" y2="52.53" width="0.4" layer="16"/>
 <via x="37.9" y="33" extent="1-16" drill="0.4"/>
+<contactref element="R7" pad="1"/>
+<wire x1="46.12" y1="58.1" x2="48.77" y2="55.45" width="0.4064" layer="16"/>
+<wire x1="48.77" y1="55.45" x2="48.77" y2="53.69" width="0.4064" layer="16"/>
+<wire x1="48.77" y1="53.69" x2="47.61" y2="52.53" width="0.4064" layer="16"/>
+<wire x1="47.61" y1="52.53" x2="46.42" y2="52.53" width="0.4064" layer="16"/>
 </signal>
 <signal name="DATA_SHARP_1">

Commit message: a envoyer
Parts:
- added M1, M2: SMALL_SERVO, SparkFun-Electromechanical:1X03
Connections:
- new net PWM1: M1.1, MBED.P$11
- new net PWM2: M2.1, MBED.P$12
- net +5V: now also M1.2, M2.2
- net GND: now also M1.3, M2.3
Routing:
- net PWM1: track 0.00 -> 94.2 mm, vias 0 -> 6
- net PWM2: track 0.00 -> 36.6 mm, vias 0 -> 6
- net +5V: track 250.7 -> 268.4 mm
- net GND: track 0.09 -> 14.3 mm, vias 10 -> 11
Other:
- board text added: "GND VCC PWM"
Changed lines of the file:
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@@
 <wire x1="49.9" y1="73" x2="0" y2="73" width="0" layer="20"/>
 <wire x1="0" y1="73" x2="0" y2="0" width="0" layer="20"/>
-<text x="48" y="11" size="1.778" layer="1" rot="R90">Carte_PLAN_B
+<text x="19.74" y="14.38" size="1.778" layer="22" rot="MR90">Carte_PLAN_B
 ARES_13-14</text>
 <text x="9.27" y="22.98" size="1.778" layer="21" rot="R90">BUS CAN</text>
@@
 <text x="28.15" y="50.68" size="1.4224" layer="22" rot="MR270">TRANSCEIVER CAN</text>
 <text x="37.37" y="36.18" size="1.4224" layer="22" rot="MR270">ISOLATEUR GALVANIQUE</text>
+<text x="44.52" y="5.57" size="1.27" layer="21" rot="R90">GND VCC PWM</text>
+<text x="44.47" y="19.85" size="1.27" layer="21" rot="R90">GND VCC PWM</text>
 </plain>
 <attributes>
@@
 <element name="R6" library="rcl" package="R0805" value="2,7k" x="36.22" y="51.09" rot="MR180"/>
 <element name="R7" library="rcl" package="R0805" value="2,7k" x="45.17" y="58.1" rot="MR0"/>
+<element name="M1" library="SparkFun-Electromechanical" package="1X03" value="SMALL_SERVO" x="46.53" y="25.5" rot="R270"/>
+<element name="M2" library="SparkFun-Electromechanical" package="1X03" value="SMALL_SERVO" x="46.43" y="16.69" rot="R270"/>
 </elements>
 <signals>
@@
 <via x="22.82" y="13.12" extent="1-16" drill="0.4"/>
 <contactref element="COMMAND" pad="2"/>
+<contactref element="M1" pad="3"/>
+<contactref element="M2" pad="3"/>
+<wire x1="37" y1="42" x2="38.59" y2="42" width="0.254" layer="1"/>
+<wire x1="38.59" y1="42" x2="38.59" y2="41.64" width="0.254" layer="1"/>
+<wire x1="38.59" y1="41.64" x2="40.98" y2="41.64" width="0.254" layer="1"/>
+<wire x1="40.98" y1="41.64" x2="40.98" y2="31.74" width="0.254" layer="1"/>
+<via x="37.91" y="28.45" extent="1-16" drill="0.4"/>
 </signal>
 <signal name="+5V">
@@
 <wire x1="40.87" y1="51.92" x2="41.52" y2="51.29" width="0.4064" layer="16"/>
 <wire x1="41.52" y1="51.29" x2="41.8" y2="51" width="0.4064" layer="16"/>
+<contactref element="M1" pad="2"/>
+<contactref element="M2" pad="2"/>
+<wire x1="46.5" y1="14.5" x2="46.5" y2="14.2" width="0.4" layer="16"/>
+<wire x1="48.1" y1="16.1" x2="46.5" y2="14.5" width="0.4" layer="16"/>
+<wire x1="48.1" y1="21.4" x2="48.1" y2="16.1" width="0.4" layer="16"/>
+<wire x1="46.6" y1="22.9" x2="48.1" y2="21.4" width="0.4" layer="16"/>
+<wire x1="46.5" y1="14.2" x2="46.43" y2="14.15" width="0.4" layer="16"/>
+<wire x1="46.6" y1="22.9" x2="46.53" y2="22.96" width="0.4" layer="16"/>
+<wire x1="46.6" y1="23.3" x2="46.6" y2="23.1" width="0.4" layer="16"/>
+<wire x1="48.1" y1="24.8" x2="46.6" y2="23.3" width="0.4" layer="16"/>
+<wire x1="48.1" y1="26.5" x2="48.1" y2="24.8" width="0.4" layer="16"/>
+<wire x1="46.1" y1="28.5" x2="48.1" y2="26.5" width="0.4" layer="16"/>
+<wire x1="46.1" y1="28.9" x2="46.1" y2="28.5" width="0.4" layer="16"/>
+<wire x1="46.6" y1="23.1" x2="46.53" y2="22.96" width="0.4" layer="16"/>
+<wire x1="46.1" y1="28.9" x2="45.96" y2="29.02" width="0.4" layer="16"/>
 </signal>
 <signal name="CANL">
@@
 <contactref element="C2" pad="2"/>
 <wire x1="14.24" y1="6.48" x2="14.3" y2="6.6" width="0.4" layer="1"/>
-<wire x1="14.3" y1="6.6" x2="14.3" y2="3.9" width="0.4" layer="1"/>
-<wire x1="10.34" y1="10.38" x2="14.24" y2="6.48" width="0.4" layer="1"/>
+<wire x1="14.3" y1="6.6" x2="14.3" y2="3.9" width="0.8128" layer="1"/>
+<wire x1="10.34" y1="10.38" x2="14.24" y2="6.48" width="0.8128" layer="1"/>
 <wire x1="14.3" y1="3.9" x2="14.32" y2="3.81" width="0.4" layer="1"/>
-<wire x1="10.34" y1="10.38" x2="10.33" y2="12.57" width="0.4" layer="1"/>
+<wire x1="10.34" y1="10.38" x2="10.33" y2="12.57" width="0.8128" layer="1"/>
 <wire x1="26" y1="5.9" x2="26" y2="16.4" width="0.4" layer="16"/>
 <wire x1="26" y1="16.4" x2="26" y2="18.4" width="0.4" layer="16"/>
@@
 <wire x1="26" y1="16.4" x2="28.9" y2="16.4" width="0.4" layer="16"/>
 <wire x1="35.1" y1="26.3" x2="35.195" y2="26.3262" width="0.4" layer="16"/>
-<wire x1="15.5" y1="6.6" x2="14.3" y2="6.6" width="0.4" layer="1"/>
-<wire x1="17" y1="5.1" x2="15.5" y2="6.6" width="0.4" layer="1"/>
-<wire x1="17.8" y1="5.1" x2="17" y2="5.1" width="0.4" layer="1"/>
-<wire x1="19.3" y1="6.6" x2="17.8" y2="5.1" width="0.4" layer="1"/>
-<wire x1="23.5" y1="6.6" x2="19.3" y2="6.6" width="0.4" layer="1"/>
-<wire x1="25.2" y1="4.9" x2="23.5" y2="6.6" width="0.4" layer="1"/>
-<wire x1="25.2" y1="3.9" x2="25.2" y2="4.9" width="0.4" layer="1"/>
+<wire x1="15.5" y1="6.6" x2="14.3" y2="6.6" width="0.8128" layer="1"/>
+<wire x1="17" y1="5.1" x2="15.5" y2="6.6" width="0.8128" layer="1"/>
+<wire x1="17.8" y1="5.1" x2="17" y2="5.1" width="0.8128" layer="1"/>
+<wire x1="19.3" y1="6.6" x2="17.8" y2="5.1" width="0.8128" layer="1"/>
+<wire x1="23.5" y1="6.6" x2="19.3" y2="6.6" width="0.8128" layer="1"/>
+<wire x1="25.2" y1="4.9" x2="23.5" y2="6.6" width="0.8128" layer="1"/>
+<wire x1="25.2" y1="3.9" x2="25.2" y2="4.9" width="0.8128" layer="1"/>
 <wire x1="25.2" y1="3.9" x2="25.21" y2="3.81" width="0.4" layer="1"/>
 </signal>
@@
 <wire x1="28.9" y1="20.4" x2="33.9" y2="25.4" width="0.4" layer="16"/>
 <wire x1="28.9" y1="17.7" x2="28.9" y2="20.4" width="0.4" layer="1"/>
-<wire x1="17.4" y1="6.2" x2="28.9" y2="17.7" width="0.4" layer="1"/>
+<wire x1="17.46" y1="6.32" x2="28.9" y2="17.7" width="0.4" layer="1"/>
 <wire x1="19.7" y1="3.9" x2="18.9" y2="4.7" width="0.4" layer="16"/>
-<wire x1="18.9" y1="4.7" x2="17.4" y2="6.2" width="0.4" layer="16"/>
+<wire x1="18.9" y1="4.7" x2="17.46" y2="6.32" width="0.4" layer="16"/>
 <wire x1="20.1" y1="3.9" x2="19.7" y2="3.9" width="0.4" layer="16"/>
 <wire x1="33.9" y1="26.3" x2="33.925" y2="26.3262" width="0.4" layer="16"/>
@@
 <wire x1="9.3" y1="3.8" x2="9.24" y2="3.81" width="0.4" layer="16"/>
 <via x="28.9" y="20.4" extent="1-16" drill="0.4"/>
-<via x="17.4" y="6.2" extent="1-16" drill="0.4"/>
+<via x="17.46" y="6.32" extent="1-16" drill="0.4"/>
 <contactref element="R2" pad="2"/>
 <wire x1="7.1" y1="6" x2="6.2" y2="6" width="0.4" layer="1"/>
@@
 <via x="25" y="9" extent="1-16" drill="0.4"/>
 </signal>
+<signal name="PWM1">
+<contactref element="MBED" pad="P$11"/>
+<contactref element="M1" pad="1"/>
+<wire x1="16.9" y1="36.1" x2="16.9" y2="35.4" width="0.4" layer="16"/>
+<wire x1="15.3" y1="37.7" x2="16.9" y2="36.1" width="0.4" layer="16"/>
+<wire x1="15.3" y1="38.8" x2="15.3" y2="37.7" width="0.4" layer="16"/>
+<wire x1="14.6" y1="39.5" x2="15.3" y2="38.8" width="0.4" layer="16"/>
+<wire x1="13.8" y1="39.5" x2="14.6" y2="39.5" width="0.4" layer="16"/>
+<wire x1="11.9" y1="37.6" x2="13.8" y2="39.5" width="0.4" layer="16"/>
+<wire x1="11.9" y1="27.4" x2="11.9" y2="37.6" width="0.4" layer="16"/>
+<wire x1="8.5" y1="24" x2="11.9" y2="27.4" width="0.4" layer="1"/>
+<wire x1="8.5" y1="21.4" x2="8.5" y2="24" width="0.4" layer="16"/>
+<wire x1="15.6" y1="14.3" x2="8.5" y2="21.4" width="0.4" layer="16"/>
+<wire x1="15.6" y1="12" x2="15.6" y2="14.3" width="0.4" layer="16"/>
+<wire x1="16.4" y1="11.2" x2="15.6" y2="12" width="0.4" layer="16"/>
+<wire x1="17.8" y1="11.2" x2="16.4" y2="11.2" width="0.4" layer="16"/>
+<wire x1="18.1" y1="10.9" x2="17.8" y2="11.2" width="0.4" layer="1"/>
+<wire x1="20" y1="10.9" x2="18.1" y2="10.9" width="0.4" layer="1"/>
+<wire x1="24.9" y1="10.9" x2="20" y2="10.9" width="0.4" layer="16"/>
+<wire x1="25.5" y1="10.9" x2="24.9" y2="10.9" width="0.4" layer="1"/>
+<wire x1="27.2" y1="9.2" x2="25.5" y2="10.9" width="0.4" layer="1"/>
+<wire x1="27.2" y1="8.3" x2="27.2" y2="9.2" width="0.4" layer="16"/>
+<wire x1="33.8" y1="1.7" x2="27.2" y2="8.3" width="0.4" layer="16"/>
+<wire x1="39.9" y1="1.7" x2="33.8" y2="1.7" width="0.4" layer="16"/>
+<wire x1="42.8" y1="4.6" x2="39.9" y2="1.7" width="0.4" layer="16"/>
+<wire x1="42.8" y1="21.8" x2="42.8" y2="4.6" width="0.4" layer="16"/>
+<wire x1="46.5" y1="25.5" x2="42.8" y2="21.8" width="0.4" layer="16"/>
+<wire x1="16.9" y1="35.4" x2="16.94" y2="35.37" width="0.4" layer="16"/>
+<wire x1="46.5" y1="25.5" x2="46.53" y2="25.5" width="0.4" layer="16"/>
+<via x="11.9" y="27.4" extent="1-16" drill="0.4"/>
+<via x="8.5" y="24" extent="1-16" drill="0.4"/>
+<via x="17.8" y="11.2" extent="1-16" drill="0.4"/>
+<via x="20" y="10.9" extent="1-16" drill="0.4"/>
+<via x="24.9" y="10.9" extent="1-16" drill="0.4"/>
+<via x="27.2" y="9.2" extent="1-16" drill="0.4"/>
+</signal>
+<signal name="PWM2">
+<contactref element="MBED" pad="P$12"/>
+<contactref element="M2" pad="1"/>
+<wire x1="20.2" y1="29.6" x2="17" y2="32.8" width="0.4" layer="16"/>
+<wire x1="21.7" y1="28.1" x2="20.2" y2="29.6" width="0.4" layer="1"/>
+<wire x1="33.2" y1="28.1" x2="21.7" y2="28.1" width="0.4" layer="16"/>
+<wire x1="37.7" y1="23.6" x2="33.2" y2="28.1" width="0.4" layer="1"/>
+<wire x1="37.7" y1="22.9" x2="37.7" y2="23.6" width="0.4" layer="16"/>
+<wire x1="39.2" y1="21.4" x2="37.7" y2="22.9" width="0.4" layer="16"/>
+<wire x1="41.7" y1="21.4" x2="39.2" y2="21.4" width="0.4" layer="16"/>
+<wire x1="43.9" y1="19.2" x2="41.7" y2="21.4" width="0.4" layer="1"/>
+<wire x1="46.4" y1="16.7" x2="43.9" y2="19.2" width="0.4" layer="16"/>
+<wire x1="17" y1="32.8" x2="16.94" y2="32.83" width="0.4" layer="16"/>
+<wire x1="46.4" y1="16.7" x2="46.43" y2="16.69" width="0.4" layer="16"/>
+<via x="20.2" y="29.6" extent="1-16" drill="0.4"/>
+<via x="21.7" y="28.1" extent="1-16" drill="0.4"/>
+<via x="33.2" y="28.1" extent="1-16" drill="0.4"/>
+<via x="37.7" y="23.6" extent="1-16" drill="0.4"/>
+<via x="41.7" y="21.4" extent="1-16" drill="0.4"/>
+<via x="43.9" y="19.2" extent="1-16" drill="0.4"/>
+</signal>
 </signals>
