File: cartes/En dev/Carte plan B/board.sch (EAGLE design)
At the start: 21 parts

Commit message: nouveaux gerber
Parts:
- added R3, R4, R6, R7: 2,7k, rcl:R-EU_R0805
Connections:
- net +5V: now also R3.2, R4.2, R6.2, R7.2
- net CHA_D: now also R6.1
- net CHA_G: now also R3.1
- net CHB_D: now also R7.1
- net CHB_G: now also R4.1
Changed lines of the file:
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@@
 <part name="+5V" library="supply1" deviceset="VCC" device="" value="+5v"/>
 <part name="GND2" library="supply1" deviceset="GND" device=""/>
+<part name="R3" library="rcl" deviceset="R-EU_" device="R0805" value="2,7k"/>
+<part name="R4" library="rcl" deviceset="R-EU_" device="R0805" value="2,7k"/>
+<part name="R6" library="rcl" deviceset="R-EU_" device="R0805" value="2,7k"/>
+<part name="R7" library="rcl" deviceset="R-EU_" device="R0805" value="2,7k"/>
 </parts>
 <sheets>
@@
 <instance part="+5V" gate="VCC" x="318.77" y="77.47" rot="R180"/>
 <instance part="GND2" gate="1" x="340.36" y="77.47"/>
+<instance part="R3" gate="G$1" x="147.32" y="43.18" rot="R90"/>
+<instance part="R4" gate="G$1" x="152.4" y="43.18" rot="R90"/>
+<instance part="R6" gate="G$1" x="144.78" y="22.86" rot="R90"/>
+<instance part="R7" gate="G$1" x="149.86" y="22.86" rot="R90"/>
 </instances>
 <busses>
@@
 <pinref part="+5V" gate="VCC" pin="VCC"/>
 </segment>
+<segment>
+<pinref part="R3" gate="G$1" pin="2"/>
+<wire x1="147.32" y1="48.26" x2="147.32" y2="50.8" width="0.1524" layer="91"/>
+<pinref part="R4" gate="G$1" pin="2"/>
+<wire x1="152.4" y1="48.26" x2="152.4" y2="50.8" width="0.1524" layer="91"/>
+<wire x1="147.32" y1="50.8" x2="152.4" y2="50.8" width="0.1524" layer="91"/>
+<label x="149.86" y="50.8" size="1.778" layer="95"/>
+</segment>
+<segment>
+<pinref part="R6" gate="G$1" pin="2"/>
+<wire x1="144.78" y1="27.94" x2="144.78" y2="30.48" width="0.1524" layer="91"/>
+<pinref part="R7" gate="G$1" pin="2"/>
+<wire x1="149.86" y1="27.94" x2="149.86" y2="30.48" width="0.1524" layer="91"/>
+<wire x1="144.78" y1="30.48" x2="149.86" y2="30.48" width="0.1524" layer="91"/>
+<label x="147.32" y="30.48" size="1.778" layer="95"/>
+</segment>
 </net>
 <net name="CANL" class="0">
@@
 <label x="279.4" y="139.7" size="1.778" layer="95"/>
 </segment>
+<segment>
+<pinref part="R3" gate="G$1" pin="1"/>
+<wire x1="147.32" y1="38.1" x2="147.32" y2="35.56" width="0.1524" layer="91"/>
+<label x="139.7" y="35.56" size="1.778" layer="95"/>
+</segment>
 </net>
 <net name="CHB_G" class="0">
@@
 <label x="279.4" y="142.24" size="1.778" layer="95"/>
 </segment>
+<segment>
+<pinref part="R4" gate="G$1" pin="1"/>
+<wire x1="152.4" y1="38.1" x2="152.4" y2="35.56" width="0.1524" layer="91"/>
+<label x="152.4" y="35.56" size="1.778" layer="95"/>
+</segment>
 </net>
 <net name="CHA_D" class="0">
@@
 <label x="165.1" y="142.24" size="1.778" layer="95"/>
 </segment>
+<segment>
+<pinref part="R6" gate="G$1" pin="1"/>
+<wire x1="144.78" y1="17.78" x2="144.78" y2="15.24" width="0.1524" layer="91"/>
+<label x="137.16" y="15.24" size="1.778" layer="95"/>
+</segment>
 </net>
 <net name="CHB_D" class="0">
@@
 <label x="165.1" y="139.7" size="1.778" layer="95"/>
 </segment>
-</net>
+<segment>
+<pinref part="R7" gate="G$1" pin="1"/>
+<wire x1="149.86" y1="17.78" x2="149.86" y2="15.24" width="0.1524" layer="91"/>
+<label x="149.86" y="15.24" size="1.778" layer="95"/>
+</segment>
+</net>

Commit message: a envoyer
Parts:
- added M1, M2: SMALL_SERVO, SparkFun-Electromechanical:SMALL_SERVO
Connections:
- new net PWM1: M1.SIG, MBED.P11
- new net PWM2: M2.SIG, MBED.P12
- net +5V: now also M1.V+, M2.V+
- net GND: now also M1.GND, M2.GND
Other:
- moved on the sheet: COMMAND
Changed lines of the file:
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@@
 <part name="R6" library="rcl" deviceset="R-EU_" device="R0805" value="2,7k"/>
 <part name="R7" library="rcl" deviceset="R-EU_" device="R0805" value="2,7k"/>
+<part name="M1" library="SparkFun-Electromechanical" deviceset="SMALL_SERVO" device=""/>
+<part name="M2" library="SparkFun-Electromechanical" deviceset="SMALL_SERVO" device=""/>
 </parts>
 <sheets>
@@
 <frame x1="5.08" y1="114.3" x2="139.7" y2="187.96" columns="8" rows="5" layer="91" border-left="no" border-top="no" border-right="no" border-bottom="no"/>
 <frame x1="5.08" y1="7.62" x2="124.46" y2="111.76" columns="8" rows="5" layer="91" border-left="no" border-top="no" border-right="no" border-bottom="no"/>
-<frame x1="246.38" y1="7.62" x2="360.68" y2="50.8" columns="8" rows="5" layer="91" border-left="no" border-top="no" border-right="no" border-bottom="no"/>
-<text x="261.62" y="22.86" size="5.08" layer="91">CARTE PLAN B
+<text x="271.78" y="10.16" size="5.08" layer="91">CARTE PLAN B
 ARES 2013-14
 Réalisée par Cédric PILLET</text>
@@
 <frame x1="142.24" y1="114.3" x2="363.22" y2="187.96" columns="8" rows="5" layer="91" border-left="no" border-top="no" border-right="no" border-bottom="no"/>
 <frame x1="127" y1="7.62" x2="243.84" y2="111.76" columns="8" rows="5" layer="91" border-left="no" border-top="no" border-right="no" border-bottom="no"/>
-<frame x1="246.38" y1="53.34" x2="363.22" y2="111.76" columns="8" rows="5" layer="91" border-left="no" border-top="no" border-right="no" border-bottom="no"/>
 </plain>
 <instances>
@@
 <instance part="JUMPER" gate="A" x="83.82" y="134.62" rot="MR0"/>
 <instance part="R2" gate="G$1" x="254" y="78.74" rot="R270"/>
-<instance part="COMMAND" gate="G$1" x="330.2" y="87.63"/>
-<instance part="+5V" gate="VCC" x="318.77" y="77.47" rot="R180"/>
-<instance part="GND2" gate="1" x="340.36" y="77.47"/>
+<instance part="COMMAND" gate="G$1" x="327.66" y="92.71"/>
+<instance part="+5V" gate="VCC" x="316.23" y="82.55" rot="R180"/>
+<instance part="GND2" gate="1" x="337.82" y="82.55"/>
 <instance part="R3" gate="G$1" x="147.32" y="43.18" rot="R90"/>
 <instance part="R4" gate="G$1" x="152.4" y="43.18" rot="R90"/>
 <instance part="R6" gate="G$1" x="144.78" y="22.86" rot="R90"/>
 <instance part="R7" gate="G$1" x="149.86" y="22.86" rot="R90"/>
+<instance part="M1" gate="G$1" x="327.66" y="66.04" rot="R180"/>
+<instance part="M2" gate="G$1" x="327.66" y="50.8" rot="R180"/>
 </instances>
 <busses>
@@
 <segment>
 <pinref part="COMMAND" gate="G$1" pin="4"/>
-<wire x1="335.28" y1="85.09" x2="340.36" y2="85.09" width="0.1524" layer="91"/>
-<wire x1="340.36" y1="85.09" x2="340.36" y2="80.01" width="0.1524" layer="91"/>
+<wire x1="332.74" y1="90.17" x2="337.82" y2="90.17" width="0.1524" layer="91"/>
+<wire x1="337.82" y1="90.17" x2="337.82" y2="85.09" width="0.1524" layer="91"/>
 <pinref part="GND2" gate="1" pin="GND"/>
+</segment>
+<segment>
+<pinref part="M1" gate="G$1" pin="GND"/>
+<wire x1="325.12" y1="71.12" x2="317.5" y2="71.12" width="0.1524" layer="91"/>
+</segment>
+<segment>
+<pinref part="M2" gate="G$1" pin="GND"/>
+<wire x1="325.12" y1="55.88" x2="317.5" y2="55.88" width="0.1524" layer="91"/>
 </segment>
 </net>
@@
 <segment>
 <pinref part="COMMAND" gate="G$1" pin="3"/>
-<wire x1="325.12" y1="85.09" x2="318.77" y2="85.09" width="0.1524" layer="91"/>
-<wire x1="318.77" y1="85.09" x2="318.77" y2="80.01" width="0.1524" layer="91"/>
+<wire x1="322.58" y1="90.17" x2="316.23" y2="90.17" width="0.1524" layer="91"/>
+<wire x1="316.23" y1="90.17" x2="316.23" y2="85.09" width="0.1524" layer="91"/>
 <pinref part="+5V" gate="VCC" pin="VCC"/>
 </segment>
@@
 <label x="147.32" y="30.48" size="1.778" layer="95"/>
 </segment>
+<segment>
+<pinref part="M1" gate="G$1" pin="V+"/>
+<wire x1="325.12" y1="68.58" x2="317.5" y2="68.58" width="0.1524" layer="91"/>
+</segment>
+<segment>
+<pinref part="M2" gate="G$1" pin="V+"/>
+<wire x1="325.12" y1="53.34" x2="317.5" y2="53.34" width="0.1524" layer="91"/>
+</segment>
 </net>
 <net name="CANL" class="0">
@@
 <segment>
 <pinref part="COMMAND" gate="G$1" pin="8"/>
-<wire x1="335.28" y1="90.17" x2="340.36" y2="90.17" width="0.1524" layer="91"/>
-<label x="340.36" y="90.17" size="1.778" layer="95"/>
+<wire x1="332.74" y1="95.25" x2="337.82" y2="95.25" width="0.1524" layer="91"/>
+<label x="337.82" y="95.25" size="1.778" layer="95"/>
 </segment>
 </net>
@@
 <segment>
 <pinref part="COMMAND" gate="G$1" pin="7"/>
-<wire x1="325.12" y1="90.17" x2="320.04" y2="90.17" width="0.1524" layer="91"/>
-<label x="320.04" y="90.17" size="1.778" layer="95" rot="R180"/>
+<wire x1="322.58" y1="95.25" x2="317.5" y2="95.25" width="0.1524" layer="91"/>
+<label x="317.5" y="95.25" size="1.778" layer="95" rot="R180"/>
 </segment>
 </net>
@@
 <segment>
 <pinref part="COMMAND" gate="G$1" pin="6"/>
-<wire x1="335.28" y1="87.63" x2="340.36" y2="87.63" width="0.1524" layer="91"/>
-<label x="340.36" y="87.63" size="1.778" layer="95"/>
+<wire x1="332.74" y1="92.71" x2="337.82" y2="92.71" width="0.1524" layer="91"/>
+<label x="337.82" y="92.71" size="1.778" layer="95"/>
 </segment>
 </net>
@@
 <segment>
 <pinref part="COMMAND" gate="G$1" pin="5"/>
-<wire x1="325.12" y1="87.63" x2="320.04" y2="87.63" width="0.1524" layer="91"/>
-<label x="320.04" y="87.63" size="1.778" layer="95" rot="R180"/>
+<wire x1="322.58" y1="92.71" x2="317.5" y2="92.71" width="0.1524" layer="91"/>
+<label x="317.5" y="92.71" size="1.778" layer="95" rot="R180"/>
 </segment>
 </net>
@@
 </segment>
 </net>
+<net name="PWM1" class="0">
+<segment>
+<pinref part="MBED" gate="KIT" pin="P11"/>
+<wire x1="177.8" y1="152.4" x2="170.18" y2="152.4" width="0.1524" layer="91"/>
+<label x="165.1" y="152.4" size="1.778" layer="95"/>
+</segment>
+<segment>
+<pinref part="M1" gate="G$1" pin="SIG"/>
+<wire x1="325.12" y1="66.04" x2="317.5" y2="66.04" width="0.1524" layer="91"/>
+</segment>
+</net>
+<net name="PWM2" class="0">
+<segment>
+<pinref part="MBED" gate="KIT" pin="P12"/>
+<wire x1="177.8" y1="149.86" x2="170.18" y2="149.86" width="0.1524" layer="91"/>
+<label x="165.1" y="149.86" size="1.778" layer="95"/>
+</segment>
+<segment>
+<pinref part="M2" gate="G$1" pin="SIG"/>
+<wire x1="325.12" y1="50.8" x2="317.5" y2="50.8" width="0.1524" layer="91"/>
+</segment>
+</net>
+<net name="N$6" class="0">
+<segment>
+<wire x1="246.38" y1="111.76" x2="363.22" y2="111.76" width="0.3048" layer="91"/>
+<wire x1="363.22" y1="111.76" x2="363.22" y2="43.18" width="0.3048" layer="91"/>
+<wire x1="363.22" y1="43.18" x2="246.38" y2="43.18" width="0.3048" layer="91"/>
+<wire x1="246.38" y1="43.18" x2="246.38" y2="111.76" width="0.3048" layer="91"/>
+</segment>
+</net>
+<net name="N$7" class="0">
+<segment>
+<wire x1="246.38" y1="40.64" x2="363.22" y2="40.64" width="0.3048" layer="91"/>
+<wire x1="363.22" y1="40.64" x2="363.22" y2="5.08" width="0.3048" layer="91"/>
+<wire x1="363.22" y1="5.08" x2="246.38" y2="5.08" width="0.3048" layer="91"/>
+<wire x1="246.38" y1="5.08" x2="246.38" y2="40.64" width="0.3048" layer="91"/>
+</segment>
+</net>
