File: cartes/En dev/pwm_transistor/pwm_nmos_555.brd (EAGLE design)
At the start: 27.6 x 47 mm, 16 parts, among them Q1 MOSFET-NCHANNELFQP30N06L, T1 2N2222

Commit message: carte mos pwm modifié
Parts:
- moved D1 1.27 mm to (17.8, 8.89), flipped to the bottom
- flipped VOUT to the top
Connections:
- net ENABLE_555 renamed GND_555
Routing:
- net GND_555: track 54.6 -> 32.4 mm, vias 0 -> 1
- net SIG: track 38.6 -> 34.2 mm
- net VOUT: track 15.7 -> 12.7 mm
- net V+_MOT: track 14.0 -> 12.5 mm
- net VCC: track 36.5 -> 35.2 mm
- net N$5: track 24.9 -> 25.8 mm, vias 0 -> 1
- net SIG_555: track 22.1 -> 21.3 mm
Other:
- board size 27.6 x 47 mm -> 27.6 x 43.2 mm
- board text added: "ARES 2014"
- board text added: "PWM+MOTEUR"
