File: cartes/Envoyé à dipole/Carte_RF_CAN/nrf_can.brd (EAGLE design)
At the start: 34 x 39.4 mm, 13 parts, among them Q1 16MHz

Commit message: Modif carte rf avec erreur vue par Pak
Parts:
- moved R1 13.3 mm to (29.0, 14.6), turned to 270 degrees
Connections:
- net GND: now also TRANSCEIVER.2; no longer TRANSCEIVER.3
- net VCC: now also TRANSCEIVER.3; no longer TRANSCEIVER.2
Routing:
- net N$5: track 14.1 -> 2.74 mm
- net MISO: track 47.5 -> 53.5 mm, vias 1 -> 0
- net VCC: track 66.4 -> 70.2 mm
- net MOSI: track 43.4 -> 41.7 mm
Changed lines of the file:
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@@
 </element>
 <element name="C2" library="SparkFun-Capacitors" package="0805" value="22pF" x="31.0388" y="41.3766" rot="R270"/>
-<element name="R1" library="SparkFun-Passives" package="0805" value="4,7k" x="16.1798" y="18.0848" rot="MR90"/>
+<element name="R1" library="SparkFun-Passives" package="0805" value="4,7k" x="29.0322" y="14.605" rot="MR270"/>
 <element name="R2" library="SparkFun-Passives" package="0805" value="120" x="31.7246" y="19.1262" rot="MR180"/>
 <element name="CAN_CONTROL" library="MCP2515_MT" package="SO18L" value="MCP2515SO" x="23.8506" y="19.5326" rot="R90"/>
@@
 <contactref element="ARDUINO_MINI" pad="14"/>
 <contactref element="NRF24L01" pad="6"/>
-<wire x1="15.8242" y1="19.3802" x2="18.8468" y2="19.3802" width="0.2" layer="1"/>
-<wire x1="15.8242" y1="20.447" x2="15.8242" y2="19.3802" width="0.2" layer="1"/>
-<wire x1="15.6464" y1="20.6248" x2="15.8242" y2="20.447" width="0.2" layer="16"/>
-<wire x1="15.113" y1="20.6248" x2="15.6464" y2="20.6248" width="0.2" layer="16"/>
-<wire x1="13.6906" y1="19.2024" x2="15.113" y2="20.6248" width="0.2" layer="16"/>
-<wire x1="12.8016" y1="19.2024" x2="13.6906" y2="19.2024" width="0.2" layer="16"/>
-<wire x1="18.8468" y1="19.3802" x2="18.9484" y2="19.5326" width="0.2" layer="1"/>
-<wire x1="12.8016" y1="19.2024" x2="12.7" y2="19.05" width="0.2" layer="16"/>
-<via x="15.8242" y="20.447" extent="1-16" drill="0.3"/>
 <wire x1="14.0462" y1="44.0944" x2="15.2908" y2="42.8498" width="0.2" layer="16"/>
 <wire x1="9.779" y1="44.0944" x2="14.0462" y2="44.0944" width="0.2" layer="16"/>
@@
 <wire x1="15.2908" y1="42.8498" x2="15.3416" y2="42.6974" width="0.2" layer="16"/>
 <wire x1="12.6238" y1="19.2024" x2="12.7" y2="19.05" width="0.2" layer="16"/>
+<wire x1="17.4244" y1="19.3802" x2="18.8468" y2="19.3802" width="0.2" layer="1"/>
+<wire x1="17.2466" y1="19.2024" x2="17.4244" y2="19.3802" width="0.2" layer="16"/>
+<wire x1="12.8016" y1="19.2024" x2="17.2466" y2="19.2024" width="0.2" layer="16"/>
+<wire x1="18.8468" y1="19.3802" x2="18.9484" y2="19.5326" width="0.2" layer="1"/>
+<wire x1="12.8016" y1="19.2024" x2="12.7" y2="19.05" width="0.2" layer="16"/>
+<via x="17.4244" y="19.3802" extent="1-16" drill="0.3"/>
 </signal>
 <signal name="MISO">
@@
 <contactref element="ARDUINO_MINI" pad="15"/>
 <contactref element="NRF24L01" pad="7"/>
-<wire x1="17.4244" y1="18.3134" x2="18.8468" y2="18.3134" width="0.2" layer="1"/>
-<wire x1="17.4244" y1="21.1582" x2="17.4244" y2="18.3134" width="0.2" layer="16"/>
-<wire x1="13.1572" y1="21.1582" x2="17.4244" y2="21.1582" width="0.2" layer="16"/>
-<wire x1="12.8016" y1="21.5138" x2="13.1572" y2="21.1582" width="0.2" layer="16"/>
+<wire x1="15.113" y1="18.3134" x2="18.8468" y2="18.3134" width="0.2" layer="1"/>
+<wire x1="15.113" y1="19.9136" x2="15.113" y2="18.3134" width="0.2" layer="1"/>
+<wire x1="13.5128" y1="21.5138" x2="15.113" y2="19.9136" width="0.2" layer="1"/>
+<wire x1="12.8016" y1="21.5138" x2="13.5128" y2="21.5138" width="0.2" layer="1"/>
 <wire x1="18.8468" y1="18.3134" x2="18.9484" y2="18.2626" width="0.2" layer="1"/>
-<wire x1="12.8016" y1="21.5138" x2="12.7" y2="21.59" width="0.2" layer="16"/>
-<wire x1="28.2702" y1="27.7368" x2="21.0661875" y2="27.7368" width="0.2" layer="16"/>
-<wire x1="21.0661875" y1="27.7368" x2="17.9578" y2="30.8451875" width="0.2" layer="16"/>
-<wire x1="17.9578" y1="30.8451875" x2="17.9578" y2="40.005" width="0.2" layer="16"/>
+<wire x1="12.8016" y1="21.5138" x2="12.7" y2="21.59" width="0.2" layer="1"/>
+<wire x1="17.9578" y1="27.7368" x2="17.9578" y2="40.005" width="0.2" layer="16"/>
+<wire x1="28.2702" y1="27.7368" x2="17.9578" y2="27.7368" width="0.2" layer="16"/>
 <wire x1="28.9814" y1="27.0256" x2="28.2702" y2="27.7368" width="0.2" layer="16"/>
 <wire x1="28.9814" y1="23.114" x2="28.9814" y2="27.0256" width="0.2" layer="16"/>
 <wire x1="19.558" y1="23.114" x2="28.9814" y2="23.114" width="0.2" layer="16"/>
 <wire x1="17.6022" y1="21.1582" x2="19.558" y2="23.114" width="0.2" layer="16"/>
-<wire x1="17.4244" y1="21.1582" x2="17.6022" y2="21.1582" width="0.2" layer="16"/>
+<wire x1="13.1572" y1="21.1582" x2="17.6022" y2="21.1582" width="0.2" layer="16"/>
+<wire x1="12.8016" y1="21.5138" x2="13.1572" y2="21.1582" width="0.2" layer="16"/>
 <wire x1="17.9578" y1="40.005" x2="17.8816" y2="40.1574" width="0.2" layer="16"/>
-<via x="17.4244" y="18.3134" extent="1-16" drill="0.3"/>
+<wire x1="12.8016" y1="21.5138" x2="12.7" y2="21.59" width="0.2" layer="16"/>
 </signal>
 <signal name="SCK">
@@
 <signal name="VCC">
 <contactref element="CAN_CONTROL" pad="18"/>
-<contactref element="TRANSCEIVER" pad="2"/>
 <contactref element="ARDUINO_MINI" pad="VCC"/>
 <contactref element="CAN" pad="7"/>
@@
 <wire x1="24.3586" y1="38.9382" x2="24.318" y2="38.7811" width="0.2" layer="1"/>
 <wire x1="21.6916" y1="46.9392" x2="21.59" y2="46.99" width="0.2" layer="1"/>
-<wire x1="17.4244" y1="15.4686" x2="17.4244" y2="14.5796" width="0.2" layer="1"/>
-<wire x1="17.4244" y1="14.5796" x2="18.8468" y2="14.5796" width="0.2" layer="1"/>
-<wire x1="19.7358" y1="17.78" x2="17.4244" y2="15.4686" width="0.2" layer="16"/>
-<wire x1="21.5138" y1="17.78" x2="19.7358" y2="17.78" width="0.2" layer="16"/>
-<wire x1="18.8468" y1="14.5796" x2="18.9484" y2="14.4526" width="0.2" layer="1"/>
-<wire x1="21.5138" y1="17.78" x2="21.5646" y2="17.8816" width="0.2" layer="16"/>
 <wire x1="28.6258" y1="22.0472" x2="32.3596" y2="25.781" width="0.2" layer="16"/>
 <wire x1="32.3596" y1="25.781" x2="33.8074" y2="27.2288" width="0.2" layer="16"/>
 <wire x1="25.0698" y1="22.0472" x2="28.6258" y2="22.0472" width="0.2" layer="16"/>
 <wire x1="24.003" y1="20.9804" x2="25.0698" y2="22.0472" width="0.2" layer="16"/>
-<wire x1="24.003" y1="17.78" x2="24.003" y2="20.9804" width="0.2" layer="16"/>
+<wire x1="24.003" y1="17.78" x2="24.003" y2="19.2024" width="0.2" layer="16"/>
+<wire x1="24.003" y1="19.2024" x2="24.003" y2="20.9804" width="0.2" layer="16"/>
 <wire x1="21.6916" y1="17.78" x2="24.003" y2="17.78" width="0.2" layer="16"/>
-<wire x1="21.6916" y1="17.78" x2="21.5646" y2="17.8816" width="0.2" layer="16"/>
 <wire x1="36.2712" y1="32.7152" x2="36.2712" y2="33.4264" width="0.2" layer="16"/>
 <wire x1="36.0934" y1="32.7152" x2="36.2712" y2="32.7152" width="0.2" layer="16"/>
@@
 <wire x1="31.6484" y1="29.337" x2="31.6484" y2="33.782" width="0.2" layer="16"/>
 <wire x1="31.8262" y1="29.337" x2="31.6484" y2="29.337" width="0.2" layer="16"/>
-<via x="17.4244" y="15.4686" extent="1-16" drill="0.3"/>
 <via x="25.6032" y="40.1828" extent="1-16" drill="0.3"/>
+<contactref element="TRANSCEIVER" pad="3"/>
+<wire x1="21.6916" y1="19.2024" x2="21.6916" y2="19.15158125" width="0.2" layer="16"/>
+<wire x1="24.003" y1="19.2024" x2="21.6916" y2="19.2024" width="0.2" layer="16"/>
+<wire x1="21.6916" y1="19.2024" x2="21.5646" y2="19.1516" width="0.2" layer="16"/>
+<wire x1="19.0246" y1="13.5128" x2="19.0246" y2="14.4018" width="0.2" layer="1"/>
+<wire x1="19.0246" y1="19.0246" x2="19.0246" y2="13.5128" width="0.2" layer="16"/>
+<wire x1="21.5138" y1="19.0246" x2="19.0246" y2="19.0246" width="0.2" layer="16"/>
+<wire x1="19.0246" y1="14.4018" x2="18.9484" y2="14.4526" width="0.2" layer="1"/>
+<wire x1="21.5138" y1="19.0246" x2="21.5646" y2="19.1516" width="0.2" layer="16"/>
+<via x="19.0246" y="13.5128" extent="1-16" drill="0.3"/>
 </signal>
 <signal name="GND">
 <contactref element="CAN_CONTROL" pad="9"/>
-<contactref element="TRANSCEIVER" pad="3"/>
 <contactref element="R1" pad="2"/>
 <contactref element="C1" pad="1"/>
@@
 <contactref element="3.3V" pad="2"/>
 <wire x1="19.3802" y1="45.5168" x2="19.35819375" y2="45.4406" width="0.2" layer="16"/>
-<wire x1="21.6916" y1="19.2024" x2="21.5646" y2="19.1516" width="0.2" layer="16"/>
-<wire x1="21.6916" y1="19.2024" x2="21.6916" y2="19.15158125" width="0.2" layer="16"/>
-<via x="14.7955" y="18.3388" extent="1-16" drill="0.5"/>
-<wire x1="21.5646" y1="19.1516" x2="16.1798" y2="18.9848" width="0" layer="19" extent="16-16"/>
+<contactref element="TRANSCEIVER" pad="2"/>
+<via x="21.2725" y="14.8717" extent="1-16" drill="0.5"/>
 </signal>
 <signal name="CAN_TXD">
@@
 <wire x1="22.0472" y1="16.875846875" x2="20.995553125" y2="15.8242" width="0.2" layer="1"/>
 <wire x1="20.995553125" y1="15.8242" x2="19.0246" y2="15.8242" width="0.2" layer="1"/>
-<wire x1="24.3586" y1="24.003" x2="22.0472" y2="21.6916" width="0.2" layer="1"/>
+<wire x1="25.6032" y1="25.2476" x2="22.0472" y2="21.6916" width="0.2" layer="1"/>
 <wire x1="25.6032" y1="36.2712" x2="25.6032" y2="25.2476" width="0.2" layer="1"/>
-<wire x1="25.6032" y1="25.2476" x2="24.3586" y2="24.003" width="0.2" layer="1"/>
 <wire x1="27.9146" y1="38.5826" x2="25.6032" y2="36.2712" width="0.2" layer="1"/>
 <wire x1="27.9146" y1="39.2938" x2="27.9146" y2="38.5826" width="0.2" layer="1"/>
@@
 <contactref element="TRANSCEIVER" pad="8"/>
 <contactref element="R1" pad="1"/>
-<wire x1="17.78" y1="14.7574" x2="16.65904375" y2="14.7574" width="0.2" layer="16"/>
-<wire x1="16.65904375" y1="14.7574" x2="16.1798" y2="15.23664375" width="0.2" layer="16"/>
-<wire x1="16.1798" y1="15.23664375" x2="16.1798" y2="17.1848" width="0.2" layer="16"/>
-<wire x1="20.2692" y1="17.2466" x2="17.78" y2="14.7574" width="0.2" layer="16"/>
-<wire x1="22.9362" y1="17.2466" x2="20.2692" y2="17.2466" width="0.2" layer="16"/>
-<wire x1="23.6474" y1="16.5354" x2="22.9362" y2="17.2466" width="0.2" layer="16"/>
-<wire x1="26.67" y1="16.5354" x2="23.6474" y2="16.5354" width="0.2" layer="16"/>
-<wire x1="26.67" y1="16.5354" x2="26.797" y2="16.6116" width="0.2" layer="16"/>
+<wire x1="28.0924" y1="16.5354" x2="28.9814" y2="15.6464" width="0.2" layer="16"/>
+<wire x1="26.8478" y1="16.5354" x2="28.0924" y2="16.5354" width="0.2" layer="16"/>
+<wire x1="28.9814" y1="15.6464" x2="29.0322" y2="15.505" width="0.2" layer="16"/>
+<wire x1="26.8478" y1="16.5354" x2="26.797" y2="16.6116" width="0.2" layer="16"/>
 </signal>
 <signal name="CANH">
