File: cartes/En dev/servo_shield/servo_1.sch (EAGLE design)
At the start: 33 parts, among them X1 5V_INPUT, X2 12V_INPUT

Commit message: Fix du bug #5 avec l'ajout d'un treansceiver RS485 pour l'ax12
Parts:
- removed JP6: RX_TX_Connxion, SparkFun-Passives:JUMPER-2PTH
- added U1: SN65HVD08D, Texas Instruments_By_element14_Batch_1:SN65HVD08D
Connections:
- net RXTX_OUT renamed RXTX_DIRTY
- new net RXTX: ADUM1250.SCL1, U1.A
- net GND: now also U1.GND
- net N$4: now also LED_12V.A; no longer LED_5V.A
- net N$6: now also LED_5V.A; no longer LED_12V.A
- net OUT4: now also U1.DE, U1.~RE
- net RXI: now also U1.R; no longer JP6.2
- net TXO: now also U1.D; no longer ADUM1250.SCL1, JP6.1
- net VCC: now also U1.VCC
Other:
- moved on the sheet: LED_12V, LED_5V

Commit message: Modif carte sharp et carte servo avec probleme transceiver
Connections:
- net GND: now also TRANSCEIVER.VSS; no longer TRANSCEIVER.VDD
- net VCC: now also TRANSCEIVER.VDD; no longer TRANSCEIVER.VSS
Changed lines of the file:
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@@
 <?xml version="1.0" encoding="utf-8"?>
 <!DOCTYPE eagle SYSTEM "eagle.dtd">
-<eagle version="6.5.0">
+<eagle version="6.4">
 <drawing>
 <settings>
@@
 </segment>
 <segment>
-<pinref part="TRANSCEIVER" gate="G$1" pin="VSS"/>
-<wire x1="144.78" y1="45.72" x2="157.48" y2="45.72" width="0.1524" layer="91"/>
-<label x="144.78" y="45.72" size="1.778" layer="95"/>
-</segment>
-<segment>
 <pinref part="ARDUINO" gate="G$1" pin="VCC"/>
 <wire x1="0" y1="73.66" x2="7.62" y2="73.66" width="0.1524" layer="91"/>
@@
 <label x="-55.88" y="-91.44" size="1.778" layer="95"/>
 </segment>
+<segment>
+<pinref part="TRANSCEIVER" gate="G$1" pin="VDD"/>
+<wire x1="157.48" y1="43.18" x2="149.86" y2="43.18" width="0.1524" layer="91"/>
+<label x="144.78" y="43.18" size="1.778" layer="95"/>
+</segment>
 </net>
 <net name="GND" class="0">
@@
 <label x="83.82" y="45.72" size="1.778" layer="95"/>
 <pinref part="CONTROLLER" gate="G$1" pin="GND"/>
-</segment>
-<segment>
-<pinref part="TRANSCEIVER" gate="G$1" pin="VDD"/>
-<wire x1="157.48" y1="43.18" x2="149.86" y2="43.18" width="0.1524" layer="91"/>
-<label x="144.78" y="43.18" size="1.778" layer="95"/>
 </segment>
 <segment>
@@
 <label x="-58.42" y="-111.76" size="1.778" layer="95"/>
 </segment>
+<segment>
+<pinref part="TRANSCEIVER" gate="G$1" pin="VSS"/>
+<wire x1="144.78" y1="45.72" x2="157.48" y2="45.72" width="0.1524" layer="91"/>
+<label x="144.78" y="45.72" size="1.778" layer="95"/>
+</segment>
 </net>
