File: cartes/En dev/Carte ascenseur/carte_ascenseur.sch (EAGLE design)
At the start: 35 parts, among them U1 MCP2551, U2 ADUM1250ARZ, U3 ADUM1400ARWZ, X1 12V Dirty, X2 5V Dirty

Commit message: Carte ascenseur
Correction d'une erreur dans la schéma, début du routage.
Parts:
- removed U$5: L7805TO263, st-microelectronics:L7805TO263
- added IC1: (no value), SparkFun-PowerIC:V_REG_78XX-TO-220
- JP2: value 'Servo' lanceur -> Servo doigt
- JP4: value Servo doigt -> 'Servo' lanceur
Connections:
- removed net 5V: CAN.2
- removed net GND: CAN.8
- removed net N$5: LED_12V.C, LED_5V.C
- net +12V: now also IC1.IN; no longer U$5.IN
- net DOIGT: now also U3.VIC; no longer U3.VIB
- net GND1: now also CAN.8
- net GND2: now also IC1.GND, LED_12V.C, LED_5V.C; no longer U$5.GND
- net N$6: now also IC1.OUT; no longer U$5.OUT
- net PANNIER: now also U3.VIB; no longer U3.VIC
- net VCC: now also CAN.2
Changed lines of the file:
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@@
 <part name="SUPPLY15" library="supply2" deviceset="GND2" device=""/>
 <part name="P+13" library="supply1" deviceset="+5V" device=""/>
-<part name="JP2" library="SparkFun-Connectors" deviceset="M03" device="PTH" value="'Servo' lanceur"/>
+<part name="JP2" library="SparkFun-Connectors" deviceset="M03" device="PTH" value="Servo doigt"/>
 <part name="Q2" library="crystal" deviceset="CRYSTAL" device="HC49S"/>
 <part name="SUPPLY17" library="supply2" deviceset="GND1" device=""/>
@@
 <part name="P+6" library="supply1" deviceset="VCC" device=""/>
 <part name="JP3" library="SparkFun-Connectors" deviceset="M03" device="PTH" value="Servo pannier"/>
-<part name="JP4" library="SparkFun-Connectors" deviceset="M03" device="PTH" value="Servo doigt"/>
+<part name="JP4" library="SparkFun-Connectors" deviceset="M03" device="PTH" value="'Servo' lanceur"/>
 <part name="P+10" library="supply1" deviceset="+5V" device=""/>
 <part name="SUPPLY8" library="supply2" deviceset="GND2" device=""/>
@@
 <part name="JP5" library="SparkFun-Connectors" deviceset="M03" device="POLAR" value="AX12"/>
 <part name="P+3" library="supply1" deviceset="VCC" device=""/>
-<part name="U$5" library="st-microelectronics" deviceset="L7805" device="TO263"/>
 <part name="C9" library="rcl" deviceset="C-EU" device="C0805" value="100nF"/>
 <part name="C10" library="rcl" deviceset="C-EU" device="C0805" value="330nF"/>
@@
 <part name="P+20" library="supply1" deviceset="VCC" device=""/>
 <part name="SUPPLY18" library="supply2" deviceset="GND1" device=""/>
+<part name="IC1" library="SparkFun-PowerIC" deviceset="V_REG_78XX" device="-TO-220"/>
 </parts>
 <sheets>
@@
 <instance part="JP5" gate="G$1" x="256.54" y="91.44" rot="R180"/>
 <instance part="P+3" gate="VCC" x="0" y="60.96"/>
-<instance part="U$5" gate="G$1" x="256.54" y="149.86"/>
 <instance part="C9" gate="G$1" x="276.86" y="142.24" rot="R180"/>
 <instance part="C10" gate="G$1" x="238.76" y="142.24" rot="R180"/>
@@
 </instance>
 <instance part="P+18" gate="1" x="317.5" y="134.62"/>
-<instance part="SUPPLY16" gate="G$1" x="317.5" y="99.06"/>
+<instance part="SUPPLY16" gate="G$1" x="317.5" y="96.52"/>
 <instance part="LED_12V" gate="G$1" x="330.2" y="111.76"/>
 <instance part="R7" gate="G$1" x="330.2" y="121.92" rot="R270">
@@
 <instance part="P+20" gate="VCC" x="-104.14" y="68.58"/>
 <instance part="SUPPLY18" gate="G$1" x="-104.14" y="38.1"/>
+<instance part="IC1" gate="G$1" x="256.54" y="152.4"/>
 </instances>
 <busses>
@@
 </segment>
 </net>
-<net name="GND" class="0">
-<segment>
-<pinref part="CAN" gate="G$1" pin="8"/>
-<wire x1="-60.96" y1="58.42" x2="-53.34" y2="58.42" width="0.1524" layer="91"/>
-<label x="-58.42" y="58.42" size="1.778" layer="95"/>
-</segment>
-</net>
 <net name="PGC" class="0">
 <segment>
@@
 <pinref part="PIC" gate="A" pin="!MCLR!"/>
 <wire x1="40.64" y1="33.02" x2="38.1" y2="33.02" width="0.1524" layer="91"/>
-</segment>
-</net>
-<net name="5V" class="0">
-<segment>
-<pinref part="CAN" gate="G$1" pin="2"/>
-<wire x1="-60.96" y1="50.8" x2="-53.34" y2="50.8" width="0.1524" layer="91"/>
-<label x="-58.42" y="50.8" size="1.778" layer="95"/>
 </segment>
 </net>
@@
 <pinref part="SUPPLY18" gate="G$1" pin="GND1"/>
 </segment>
+<segment>
+<pinref part="CAN" gate="G$1" pin="8"/>
+<wire x1="-60.96" y1="58.42" x2="-53.34" y2="58.42" width="0.1524" layer="91"/>
+<label x="-58.42" y="58.42" size="1.778" layer="95"/>
+</segment>
 </net>
 <net name="GND2" class="0">
@@
 <wire x1="276.86" y1="139.7" x2="276.86" y2="137.16" width="0.1524" layer="91"/>
 <wire x1="276.86" y1="137.16" x2="256.54" y2="137.16" width="0.1524" layer="91"/>
-<pinref part="U$5" gate="G$1" pin="GND"/>
-<wire x1="256.54" y1="139.7" x2="256.54" y2="137.16" width="0.1524" layer="91"/>
 <pinref part="C10" gate="G$1" pin="1"/>
 <wire x1="256.54" y1="137.16" x2="238.76" y2="137.16" width="0.1524" layer="91"/>
@@
 <junction x="238.76" y="137.16"/>
 <pinref part="SUPPLY9" gate="G$1" pin="GND2"/>
+<pinref part="IC1" gate="G$1" pin="GND"/>
+<wire x1="256.54" y1="144.78" x2="256.54" y2="137.16" width="0.1524" layer="91"/>
 </segment>
 <segment>
@@
 <wire x1="182.88" y1="132.08" x2="182.88" y2="129.54" width="0.1524" layer="91"/>
 <pinref part="SUPPLY12" gate="G$1" pin="GND2"/>
+</segment>
+<segment>
+<pinref part="LED_5V" gate="G$1" pin="C"/>
+<wire x1="317.5" y1="106.68" x2="317.5" y2="104.14" width="0.1524" layer="91"/>
+<pinref part="SUPPLY16" gate="G$1" pin="GND2"/>
+<pinref part="LED_12V" gate="G$1" pin="C"/>
+<wire x1="317.5" y1="104.14" x2="317.5" y2="99.06" width="0.1524" layer="91"/>
+<wire x1="317.5" y1="104.14" x2="330.2" y2="104.14" width="0.1524" layer="91"/>
+<wire x1="330.2" y1="104.14" x2="330.2" y2="106.68" width="0.1524" layer="91"/>
 </segment>
 </net>
@@
 <pinref part="R8" gate="G$1" pin="1"/>
 <wire x1="-104.14" y1="66.04" x2="-104.14" y2="63.5" width="0.1524" layer="91"/>
+</segment>
+<segment>
+<pinref part="CAN" gate="G$1" pin="2"/>
+<wire x1="-60.96" y1="50.8" x2="-53.34" y2="50.8" width="0.1524" layer="91"/>
+<label x="-58.42" y="50.8" size="1.778" layer="95"/>
 </segment>
 </net>
@@
 </segment>
 <segment>
-<label x="167.64" y="40.64" size="1.778" layer="96"/>
-<pinref part="U3" gate="A" pin="VIB"/>
-<wire x1="167.64" y1="40.64" x2="180.34" y2="40.64" width="0.1524" layer="91"/>
+<pinref part="U3" gate="A" pin="VIC"/>
+<wire x1="167.64" y1="38.1" x2="180.34" y2="38.1" width="0.1524" layer="91"/>
+<label x="167.64" y="38.1" size="1.778" layer="95"/>
 </segment>
 </net>
@@
 </segment>
 <segment>
-<pinref part="U3" gate="A" pin="VIC"/>
-<wire x1="167.64" y1="38.1" x2="180.34" y2="38.1" width="0.1524" layer="91"/>
-<label x="167.64" y="38.1" size="1.778" layer="95"/>
+<label x="167.64" y="40.64" size="1.778" layer="96"/>
+<pinref part="U3" gate="A" pin="VIB"/>
+<wire x1="167.64" y1="40.64" x2="180.34" y2="40.64" width="0.1524" layer="91"/>
 </segment>
 </net>
@@
 </segment>
 <segment>
-<pinref part="U$5" gate="G$1" pin="IN"/>
-<wire x1="241.3" y1="152.4" x2="238.76" y2="152.4" width="0.1524" layer="91"/>
 <pinref part="C10" gate="G$1" pin="2"/>
 <wire x1="238.76" y1="152.4" x2="215.9" y2="152.4" width="0.1524" layer="91"/>
@@
 <pinref part="P+14" gate="1" pin="+12V"/>
 <wire x1="213.36" y1="154.94" x2="213.36" y2="152.4" width="0.1524" layer="91"/>
+<pinref part="IC1" gate="G$1" pin="IN"/>
+<wire x1="238.76" y1="152.4" x2="248.92" y2="152.4" width="0.1524" layer="91"/>
 </segment>
 <segment>
@@
 <net name="N$6" class="0">
 <segment>
-<pinref part="U$5" gate="G$1" pin="OUT"/>
-<wire x1="271.78" y1="152.4" x2="276.86" y2="152.4" width="0.1524" layer="91"/>
 <pinref part="C9" gate="G$1" pin="2"/>
 <wire x1="276.86" y1="152.4" x2="287.02" y2="152.4" width="0.1524" layer="91"/>
@@
 <junction x="276.86" y="152.4"/>
 <pinref part="JP6" gate="A" pin="1"/>
+<pinref part="IC1" gate="G$1" pin="OUT"/>
+<wire x1="264.16" y1="152.4" x2="276.86" y2="152.4" width="0.1524" layer="91"/>
 </segment>
 </net>
@@
 </segment>
 </net>
-<net name="N$5" class="0">
-<segment>
-<pinref part="LED_5V" gate="G$1" pin="C"/>
-<wire x1="317.5" y1="106.68" x2="317.5" y2="104.14" width="0.1524" layer="91"/>
-<pinref part="SUPPLY16" gate="G$1" pin="GND2"/>
-<pinref part="LED_12V" gate="G$1" pin="C"/>
-<wire x1="317.5" y1="104.14" x2="317.5" y2="101.6" width="0.1524" layer="91"/>
-<wire x1="317.5" y1="104.14" x2="330.2" y2="104.14" width="0.1524" layer="91"/>
-<wire x1="330.2" y1="104.14" x2="330.2" y2="106.68" width="0.1524" layer="91"/>
-</segment>
-</net>

Commit message: Maj ascenseur
Parts:
- removed IC1: (no value), SparkFun-PowerIC:V_REG_78XX-TO-220
- added IC2: 7805TV, linear:7805TV
- SV2: device con-lstb:MA03-1 -> con-lstb:MA05-1
Connections:
- new net C_S2: PIC.OC4/RD3, SV2.5
- new net C_S3: PIC.EMUD2/OC2/IC2/INT2/RD1, SV2.4
- net +12V: now also IC2.VI; no longer IC1.IN
- net GND2: now also IC2.GND; no longer IC1.GND
- net N$6: now also IC2.VO; no longer IC1.OUT
Changed lines of the file:
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@@
 <part name="P+7" library="supply1" deviceset="VCC" device=""/>
 <part name="P+8" library="supply1" deviceset="+5V" device=""/>
-<part name="SV2" library="con-lstb" deviceset="MA03-1" device="" value="Carte couleur"/>
+<part name="SV2" library="con-lstb" deviceset="MA05-1" device="" value="Carte couleur"/>
 <part name="P+9" library="supply1" deviceset="VCC" device=""/>
 <part name="SUPPLY11" library="supply2" deviceset="GND1" device=""/>
@@
 <part name="P+20" library="supply1" deviceset="VCC" device=""/>
 <part name="SUPPLY18" library="supply2" deviceset="GND1" device=""/>
-<part name="IC1" library="SparkFun-PowerIC" deviceset="V_REG_78XX" device="-TO-220"/>
+<part name="IC2" library="linear" deviceset="78*" device="TV" technology="05"/>
 </parts>
 <sheets>
@@
 <instance part="P+8" gate="1" x="170.18" y="58.42"/>
 <instance part="SV2" gate="G$1" x="99.06" y="129.54"/>
-<instance part="P+9" gate="VCC" x="127" y="134.62"/>
-<instance part="SUPPLY11" gate="G$1" x="114.3" y="134.62"/>
+<instance part="P+9" gate="VCC" x="139.7" y="132.08"/>
+<instance part="SUPPLY11" gate="G$1" x="127" y="132.08"/>
 <instance part="JP1" gate="G$1" x="256.54" y="109.22" rot="R180"/>
 <instance part="R5" gate="G$1" x="233.68" y="109.22"/>
@@
 <instance part="P+20" gate="VCC" x="-104.14" y="68.58"/>
 <instance part="SUPPLY18" gate="G$1" x="-104.14" y="38.1"/>
-<instance part="IC1" gate="G$1" x="256.54" y="152.4"/>
+<instance part="IC2" gate="A1" x="256.54" y="152.4"/>
 </instances>
 <busses>
@@
 <segment>
 <pinref part="SV2" gate="G$1" pin="3"/>
-<wire x1="106.68" y1="132.08" x2="109.22" y2="132.08" width="0.1524" layer="91"/>
-<wire x1="109.22" y1="132.08" x2="109.22" y2="139.7" width="0.1524" layer="91"/>
-<wire x1="109.22" y1="139.7" x2="114.3" y2="139.7" width="0.1524" layer="91"/>
-<wire x1="114.3" y1="139.7" x2="114.3" y2="137.16" width="0.1524" layer="91"/>
+<wire x1="106.68" y1="129.54" x2="121.92" y2="129.54" width="0.1524" layer="91"/>
+<wire x1="121.92" y1="129.54" x2="121.92" y2="137.16" width="0.1524" layer="91"/>
+<wire x1="121.92" y1="137.16" x2="127" y2="137.16" width="0.1524" layer="91"/>
+<wire x1="127" y1="137.16" x2="127" y2="134.62" width="0.1524" layer="91"/>
 <pinref part="SUPPLY11" gate="G$1" pin="GND1"/>
 </segment>
@@
 <junction x="238.76" y="137.16"/>
 <pinref part="SUPPLY9" gate="G$1" pin="GND2"/>
-<pinref part="IC1" gate="G$1" pin="GND"/>
 <wire x1="256.54" y1="144.78" x2="256.54" y2="137.16" width="0.1524" layer="91"/>
+<pinref part="IC2" gate="A1" pin="GND"/>
 </segment>
 <segment>
@@
 <segment>
 <pinref part="SV2" gate="G$1" pin="2"/>
-<wire x1="106.68" y1="129.54" x2="127" y2="129.54" width="0.1524" layer="91"/>
-<wire x1="127" y1="129.54" x2="127" y2="132.08" width="0.1524" layer="91"/>
+<wire x1="106.68" y1="127" x2="139.7" y2="127" width="0.1524" layer="91"/>
+<wire x1="139.7" y1="127" x2="139.7" y2="129.54" width="0.1524" layer="91"/>
 <pinref part="P+9" gate="VCC" pin="VCC"/>
 </segment>
@@
 <segment>
 <pinref part="SV2" gate="G$1" pin="1"/>
-<wire x1="106.68" y1="127" x2="127" y2="127" width="0.1524" layer="91"/>
-<label x="114.3" y="127" size="1.778" layer="96"/>
+<wire x1="106.68" y1="124.46" x2="139.7" y2="124.46" width="0.1524" layer="91"/>
+<label x="127" y="124.46" size="1.778" layer="96"/>
 </segment>
 <segment>
@@
 <pinref part="P+14" gate="1" pin="+12V"/>
 <wire x1="213.36" y1="154.94" x2="213.36" y2="152.4" width="0.1524" layer="91"/>
-<pinref part="IC1" gate="G$1" pin="IN"/>
-<wire x1="238.76" y1="152.4" x2="248.92" y2="152.4" width="0.1524" layer="91"/>
+<wire x1="238.76" y1="152.4" x2="246.38" y2="152.4" width="0.1524" layer="91"/>
+<pinref part="IC2" gate="A1" pin="VI"/>
 </segment>
 <segment>
@@
 <junction x="276.86" y="152.4"/>
 <pinref part="JP6" gate="A" pin="1"/>
-<pinref part="IC1" gate="G$1" pin="OUT"/>
-<wire x1="264.16" y1="152.4" x2="276.86" y2="152.4" width="0.1524" layer="91"/>
+<pinref part="IC2" gate="A1" pin="VO"/>
+<wire x1="266.7" y1="152.4" x2="276.86" y2="152.4" width="0.1524" layer="91"/>
 </segment>
 </net>
@@
 </segment>
 </net>
+<net name="C_S2" class="0">
+<segment>
+<pinref part="SV2" gate="G$1" pin="5"/>
+<wire x1="106.68" y1="134.62" x2="116.84" y2="134.62" width="0.1524" layer="91"/>
+<label x="109.22" y="134.62" size="1.778" layer="95"/>
+</segment>
+<segment>
+<pinref part="PIC" gate="A" pin="OC4/RD3"/>
+<wire x1="119.38" y1="60.96" x2="127" y2="60.96" width="0.1524" layer="91"/>
+<label x="121.92" y="60.96" size="1.778" layer="95"/>
+</segment>
+</net>
+<net name="C_S3" class="0">
+<segment>
+<pinref part="SV2" gate="G$1" pin="4"/>
+<wire x1="106.68" y1="132.08" x2="116.84" y2="132.08" width="0.1524" layer="91"/>
+<label x="109.22" y="132.08" size="1.778" layer="95"/>
+</segment>
+<segment>
+<pinref part="PIC" gate="A" pin="EMUD2/OC2/IC2/INT2/RD1"/>
+<wire x1="119.38" y1="58.42" x2="127" y2="58.42" width="0.1524" layer="91"/>
+<label x="121.92" y="58.42" size="1.778" layer="95"/>
+</segment>
+</net>
