File: cartes/robot/Carte ascenseur/v2/carte_ascenseur_v2.sch (EAGLE design)
At the start: 41 parts, among them IC2 7805TV, U1 MCP2551, U2 ADUM1250ARZ, U3 ADUM1400ARWZ, X1 12V Dirty, X2 5V Dirty

Commit message: Maj carte ascenseur
Fusible, condo d'alim, jumper triple pour l'alim 5V, LED pour le PIC,
sortie UART
Parts:
- removed JP6: (no value), jumper:JP1E
- added JP7: (no value), jumper:JP2E
- added LED_INFO: (no value), adafruit:LEDCHIPLED_0805
- added R9: 200, SparkFun-Passives:RESISTOR0805-RES
- added RESET: SWITCH-MOMENTARY-2PTH, SparkFun-Electromechanical:SWITCH-MOMENTARY-2PTH
- R6, R8: value 1k -> 200
Connections:
- removed net 5V_FUSE: F2.1A, U2.VDD2, U3.VDD2, U3.VE2
- removed net UART_RX: PIC.EMUC1/SOSCO/T1CK/U1ARX/CN0/RC14, UART.3
- removed net UART_TX: PIC.EMUD1/SOSCI/T2CK/U1ATX/CN1/RC13, UART.2
- removed net VCC_FUSE: F1.1A, U2.VDD1, U3.VDD1
- new net N$25: PIC.SCK1/RF6, R9.1
- new net N$27: F2.2A, X1.2, X2.2
- new net N$29: CAN.1, CAN.8, F1.2A, UART.4
- new net N$30: PIC.!MCLR!, R3.1
- new net N$31: JP7.3, X2.1
- new net N$32: C10.2, IC2.VI
- new net N$5: LED_INFO.A, R9.2
- net !MCLR!: no longer PIC.!MCLR!, R3.1
- net +12V: no longer C10.2, IC2.VI
- net +5V: now also JP7.2, U2.VDD2, U3.VDD2, U3.VE2; no longer F2.2A, JP6.2, X2.1
- net GND1: now also F1.1A, LED_INFO.C, RESET.1; no longer CAN.1, CAN.8, UART.4
- net GND2: now also F2.1A; no longer X1.2, X2.2
- net N$6: now also JP7.1; no longer JP6.1
- net PGC: now also UART.3
- net PGD: now also UART.2
- net VCC: now also RESET.2, U2.VDD1, U3.VDD1; no longer F1.2A
Other:
- moved on the sheet: C10, C11, C9, F1, F2, IC2, UART, X1, X2
