File: cartes/robot/supportS_carte_asserv/support_4N25V/adaptateur_fusible_4N25V.sch (EAGLE design)
At the start: 19 parts

Commit message: nouvelle carte sans ne555
Parts:
- F3: device fuse:SHK20Q -> fuse:SHK20L
Connections:
- net C_DIR1: now also OK1.A
- net FUSE_5V: now also OK1.COL, OK2.COL, OK3.COL, OK4.COL
Other:
- moved on the sheet: OK1, OK2, OK4
Changed lines of the file:
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@@
 <?xml version="1.0" encoding="utf-8"?>
 <!DOCTYPE eagle SYSTEM "eagle.dtd">
-<eagle version="6.4">
+<eagle version="6.5.0">
 <drawing>
 <settings>
@@
 <setting verticaltext="up"/>
 </settings>
-<grid distance="0.05" unitdist="inch" unit="inch" style="lines" multiple="1" display="no" altdistance="0.01" altunitdist="inch" altunit="inch"/>
+<grid distance="0.1" unitdist="inch" unit="inch" style="lines" multiple="1" display="no" altdistance="0.01" altunitdist="inch" altunit="inch"/>
 <layers>
 <layer number="1" name="Top" color="4" fill="1" visible="no" active="no"/>
@@
 <part name="P+2" library="supply1" deviceset="+5V" device=""/>
 <part name="GND3" library="supply1" deviceset="GNDA" device=""/>
-<part name="F3" library="fuse" deviceset="SHK20Q" device=""/>
+<part name="F3" library="fuse" deviceset="SHK20L" device=""/>
 <part name="OK1" library="optocoupler" deviceset="4N*?M" device="S" technology="25"/>
 <part name="OK2" library="optocoupler" deviceset="4N*?M" device="S" technology="25"/>
@@
 <instance part="GND3" gate="1" x="31.75" y="46.355" rot="R180"/>
 <instance part="F3" gate="G$1" x="-2.54" y="-5.08"/>
-<instance part="OK1" gate="G$1" x="-60.96" y="-38.1"/>
-<instance part="OK2" gate="G$1" x="-60.96" y="-58.42"/>
+<instance part="OK1" gate="G$1" x="-55.88" y="-38.1"/>
+<instance part="OK2" gate="G$1" x="-58.42" y="-58.42"/>
 <instance part="OK3" gate="G$1" x="-60.96" y="-76.2"/>
-<instance part="OK4" gate="G$1" x="-60.96" y="-96.52"/>
+<instance part="OK4" gate="G$1" x="-58.42" y="-96.52"/>
 <instance part="GND7" gate="1" x="-85.09" y="-45.72"/>
 <instance part="R11" gate="G$1" x="-77.47" y="-43.18" rot="R180"/>
@@
 <segment>
 <pinref part="OK4" gate="G$1" pin="A"/>
-<wire x1="-71.12" y1="-93.98" x2="-83.82" y2="-93.98" width="0.1524" layer="91"/>
+<wire x1="-68.58" y1="-93.98" x2="-83.82" y2="-93.98" width="0.1524" layer="91"/>
 <label x="-81.28" y="-96.52" size="1.778" layer="95"/>
 </segment>
@@
 <segment>
 <pinref part="OK2" gate="G$1" pin="A"/>
-<wire x1="-71.12" y1="-55.88" x2="-78.74" y2="-55.88" width="0.1524" layer="91"/>
+<wire x1="-68.58" y1="-55.88" x2="-78.74" y2="-55.88" width="0.1524" layer="91"/>
 <label x="-78.74" y="-58.42" size="1.778" layer="95"/>
 </segment>
@@
 <junction x="-172.72" y="30.48"/>
 <wire x1="-172.72" y1="30.48" x2="-177.165" y2="30.48" width="0.1524" layer="91"/>
+</segment>
+<segment>
+<pinref part="OK1" gate="G$1" pin="A"/>
+<wire x1="-66.04" y1="-35.56" x2="-83.82" y2="-35.56" width="0.1524" layer="91"/>
+<label x="-83.82" y="-35.56" size="1.778" layer="95"/>
 </segment>
 </net>
@@
 </segment>
 <segment>
-<wire x1="-38.1" y1="-38.1" x2="-53.34" y2="-38.1" width="0.1524" layer="91"/>
+<wire x1="-38.1" y1="-38.1" x2="-48.26" y2="-38.1" width="0.1524" layer="91"/>
 <label x="-40.64" y="-37.465" size="1.778" layer="95"/>
-</segment>
-<segment>
-<wire x1="-38.1" y1="-58.42" x2="-53.34" y2="-58.42" width="0.1524" layer="91"/>
+<pinref part="OK1" gate="G$1" pin="COL"/>
+</segment>
+<segment>
+<wire x1="-38.1" y1="-58.42" x2="-50.8" y2="-58.42" width="0.1524" layer="91"/>
 <label x="-40.64" y="-57.785" size="1.778" layer="95"/>
+<pinref part="OK2" gate="G$1" pin="COL"/>
+<wire x1="-50.8" y1="-58.42" x2="-53.34" y2="-58.42" width="0.1524" layer="91"/>
+<junction x="-50.8" y="-58.42"/>
 </segment>
 <segment>
 <wire x1="-38.1" y1="-76.2" x2="-53.34" y2="-76.2" width="0.1524" layer="91"/>
 <label x="-40.64" y="-75.565" size="1.778" layer="95"/>
-</segment>
-<segment>
-<wire x1="-38.1" y1="-96.52" x2="-53.34" y2="-96.52" width="0.1524" layer="91"/>
+<pinref part="OK3" gate="G$1" pin="COL"/>
+</segment>
+<segment>
+<wire x1="-38.1" y1="-96.52" x2="-50.8" y2="-96.52" width="0.1524" layer="91"/>
 <label x="-40.64" y="-95.885" size="1.778" layer="95"/>
+<pinref part="OK4" gate="G$1" pin="COL"/>
 </segment>
 </net>
@@
 <segment>
 <pinref part="R16" gate="G$1" pin="2"/>
-<wire x1="-48.895" y1="-43.18" x2="-53.34" y2="-43.18" width="0.1524" layer="91"/>
+<wire x1="-48.895" y1="-43.18" x2="-48.26" y2="-43.18" width="0.1524" layer="91"/>
 <pinref part="OK1" gate="G$1" pin="EMI"/>
-<junction x="-53.34" y="-43.18"/>
+<junction x="-48.26" y="-43.18"/>
 </segment>
 </net>
@@
 <segment>
 <pinref part="R17" gate="G$1" pin="2"/>
-<wire x1="-48.895" y1="-63.5" x2="-53.34" y2="-63.5" width="0.1524" layer="91"/>
+<wire x1="-48.895" y1="-63.5" x2="-50.8" y2="-63.5" width="0.1524" layer="91"/>
 <pinref part="OK2" gate="G$1" pin="EMI"/>
-<junction x="-53.34" y="-63.5"/>
+<junction x="-50.8" y="-63.5"/>
 </segment>
 </net>
@@
 <segment>
 <pinref part="R19" gate="G$1" pin="2"/>
-<wire x1="-48.895" y1="-101.6" x2="-53.34" y2="-101.6" width="0.1524" layer="91"/>
+<wire x1="-48.895" y1="-101.6" x2="-50.8" y2="-101.6" width="0.1524" layer="91"/>
 <pinref part="OK4" gate="G$1" pin="EMI"/>
-<junction x="-53.34" y="-101.6"/>
-</segment>
-</net>
-<net name="C_DIR" class="0">
-<segment>
-<wire x1="-68.58" y1="-35.56" x2="-78.74" y2="-35.56" width="0.1524" layer="91"/>
-<label x="-78.74" y="-38.1" size="1.778" layer="95"/>
+<junction x="-50.8" y="-101.6"/>
 </segment>
 </net>
@@
 <pinref part="OK1" gate="G$1" pin="C"/>
 <pinref part="R11" gate="G$1" pin="1"/>
-<wire x1="-72.39" y1="-43.18" x2="-71.12" y2="-43.18" width="0.1524" layer="91"/>
+<wire x1="-72.39" y1="-43.18" x2="-66.04" y2="-43.18" width="0.1524" layer="91"/>
 </segment>
 </net>
@@
 <pinref part="OK2" gate="G$1" pin="C"/>
 <pinref part="R12" gate="G$1" pin="1"/>
-<wire x1="-72.39" y1="-63.5" x2="-71.12" y2="-63.5" width="0.1524" layer="91"/>
+<wire x1="-72.39" y1="-63.5" x2="-68.58" y2="-63.5" width="0.1524" layer="91"/>
 </segment>
 </net>
@@
 <pinref part="OK4" gate="G$1" pin="C"/>
 <pinref part="R15" gate="G$1" pin="1"/>
-<wire x1="-73.66" y1="-101.6" x2="-71.12" y2="-101.6" width="0.1524" layer="91"/>
-</segment>
-</net>
+<wire x1="-73.66" y1="-101.6" x2="-68.58" y2="-101.6" width="0.1524" layer="91"/>
+</segment>
+</net>
